Commit message: multiple person controller

File: urdf/person.urdf (robot description, URDF)
Before this commit: robot person, 2 links, 1 joints
Links:
- link body: mass 49.077 -> 58.927; geometry collision cylinder length=1.723 radius=0.287; visual cylinder length=1.723 radius=0.287
- link head: mass 8.174 -> 9.815; geometry collision cylinder length=0.287 radius=0.144; visual cylinder length=0.287 radius=0.144
Joints:
- joint joint: origin xyz=0 0 1.5545 rpy=0 0 0 -> xyz=0 0 1.8665 rpy=0 0 0

Commit message: fixed person controller

File: urdf/person.urdf (robot description, URDF)
Before this commit: robot person, 2 links, 1 joints
Links:
- link body: mass 58.927 -> 56.327; geometry collision cylinder length=1.647 radius=0.274; visual cylinder length=1.647 radius=0.274
- link head: mass 9.815 -> 9.371; geometry collision cylinder length=0.274 radius=0.137; visual cylinder length=0.274 radius=0.137
Joints:
- joint joint: origin xyz=0 0 1.8665 rpy=0 0 0 -> xyz=0 0 1.784 rpy=0 0 0

Commit message: made executable

File: urdf/person.urdf (robot description, URDF)
Before this commit: robot person, 2 links, 1 joints
Links:
- added link base_footprint; visual box size=0.001 0.001 0.001
- link body: mass 56.327 -> 48.359; geometry collision cylinder length=1.414 radius=0.236; visual cylinder length=1.414 radius=0.236
- link head: mass 9.371 -> 8.071; geometry collision cylinder length=0.236 radius=0.118; visual cylinder length=0.236 radius=0.118
Joints:
- removed joint joint
- added joint joint_body: type fixed, parent base_footprint, child body, origin xyz=0 0 0.707 rpy=0 0 0
- added joint joint_head: type fixed, parent base_footprint, child head, origin xyz=0 0 1.532 rpy=0 0 0

Commit message: creates hall and robot text files for post processing

File: urdf/person.urdf (robot description, URDF)
Before this commit: robot person, 3 links, 2 joints
Links:
- link body: mass 48.359 -> 47.572; geometry collision cylinder length=1.391 radius=0.232; visual cylinder length=1.391 radius=0.232
- link head: mass 8.071 -> 7.934; geometry collision cylinder length=0.232 radius=0.116; visual cylinder length=0.232 radius=0.116
Joints:
- joint joint_body: origin xyz=0 0 0.707 rpy=0 0 0 -> xyz=0 0 0.6955 rpy=0 0 0
- joint joint_head: origin xyz=0 0 1.532 rpy=0 0 0 -> xyz=0 0 1.507 rpy=0 0 0

File: urdf/random_hall.urdf (robot description, URDF)
Before this commit: robot hallway, 88 links, 87 joints
Links:
- removed link 5_int_side_2
- added link 4_sec_4_left_conn; collision box size=0.82 0.2 3.0; visual box size=0.82 0.2 3.0
- added link 4_sec_4_right_conn; collision box size=0.82 0.2 3.0; visual box size=0.82 0.2 3.0
- added link 4_sec_5_left_conn; collision box size=0.87 0.2 3.0; visual box size=0.87 0.2 3.0
- added link 4_sec_5_left_wall; collision box size=0.2 4.45 3.0; visual box size=0.2 4.45 3.0
- added link 4_sec_5_right_conn; collision box size=0.87 0.2 3.0; visual box size=0.87 0.2 3.0
- added link 4_sec_5_right_wall; collision box size=0.2 4.45 3.0; visual box size=0.2 4.45 3.0
- added link 4_sec_6_left_conn; collision box size=0.39 0.2 3.0; visual box size=0.39 0.2 3.0
- added link 4_sec_6_left_wall; collision box size=0.2 5.29 3.0; visual box size=0.2 5.29 3.0
- added link 4_sec_6_right_conn; collision box size=0.39 0.2 3.0; visual box size=0.39 0.2 3.0
- added link 4_sec_6_right_wall; collision box size=0.2 5.29 3.0; visual box size=0.2 5.29 3.0
- added link 4_sec_7_left_conn; collision box size=1.045 0.2 3.0; visual box size=1.045 0.2 3.0
- added link 4_sec_7_left_wall; collision box size=0.2 4.19 3.0; visual box size=0.2 4.19 3.0
- added link 4_sec_7_right_conn; collision box size=1.045 0.2 3.0; visual box size=1.045 0.2 3.0
- added link 4_sec_7_right_wall; collision box size=0.2 4.19 3.0; visual box size=0.2 4.19 3.0
- added link 4_sec_8_left_conn; collision box size=1.36 0.2 3.0; visual box size=1.36 0.2 3.0
- added link 4_sec_8_left_wall; collision box size=0.2 5.18 3.0; visual box size=0.2 5.18 3.0
- added link 4_sec_8_right_conn; collision box size=1.36 0.2 3.0; visual box size=1.36 0.2 3.0
- added link 4_sec_8_right_wall; collision box size=0.2 5.18 3.0; visual box size=0.2 5.18 3.0
- added link 4_sec_9_left_wall; collision box size=0.2 4.0 3.0; visual box size=0.2 4.0 3.0
- added link 4_sec_9_right_wall; collision box size=0.2 4.0 3.0; visual box size=0.2 4.0 3.0
- added link 5_int_side_2_left; collision box size=0.2 1.2 3.0; visual box size=0.2 1.2 3.0
- added link 5_int_side_2_right; collision box size=0.2 1.2 3.0; visual box size=0.2 1.2 3.0
- added link 7_sec_1_left_conn; collision box size=0.2 1.16 3.0; visual box size=0.2 1.16 3.0
- added link 7_sec_1_left_wall; collision box size=4.0 0.2 3.0; visual box size=4.0 0.2 3.0
- added link 7_sec_1_right_conn; collision box size=0.2 1.16 3.0; visual box size=0.2 1.16 3.0
- added link 7_sec_1_right_wall; collision box size=4.0 0.2 3.0; visual box size=4.0 0.2 3.0
- added link 7_sec_2_left_conn; collision box size=0.2 0.74 3.0; visual box size=0.2 0.74 3.0
- added link 7_sec_2_left_wall; collision box size=2.88 0.2 3.0; visual box size=2.88 0.2 3.0
- added link 7_sec_2_right_conn; collision box size=0.2 0.74 3.0; visual box size=0.2 0.74 3.0
- added link 7_sec_2_right_wall; collision box size=2.88 0.2 3.0; visual box size=2.88 0.2 3.0
- added link 7_sec_3_left_conn; collision box size=0.2 0.68 3.0; visual box size=0.2 0.68 3.0
- added link 7_sec_3_left_wall; collision box size=5.01 0.2 3.0; visual box size=5.01 0.2 3.0
- added link 7_sec_3_right_conn; collision box size=0.2 0.68 3.0; visual box size=0.2 0.68 3.0
- added link 7_sec_3_right_wall; collision box size=5.01 0.2 3.0; visual box size=5.01 0.2 3.0
- added link 7_sec_4_left_conn; collision box size=0.2 1.145 3.0; visual box size=0.2 1.145 3.0
- added link 7_sec_4_left_wall; collision box size=3.03 0.2 3.0; visual box size=3.03 0.2 3.0
- added link 7_sec_4_right_conn; collision box size=0.2 1.145 3.0; visual box size=0.2 1.145 3.0
- added link 7_sec_4_right_wall; collision box size=3.03 0.2 3.0; visual box size=3.03 0.2 3.0
- added link 7_sec_5_left_conn; collision box size=0.2 0.265 3.0; visual box size=0.2 0.265 3.0
- added link 7_sec_5_left_wall; collision box size=4.18 0.2 3.0; visual box size=4.18 0.2 3.0
- added link 7_sec_5_right_conn; collision box size=0.2 0.265 3.0; visual box size=0.2 0.265 3.0
- added link 7_sec_5_right_wall; collision box size=4.18 0.2 3.0; visual box size=4.18 0.2 3.0
- added link 7_sec_6_left_conn; collision box size=0.2 0.78 3.0; visual box size=0.2 0.78 3.0
- added link 7_sec_6_left_wall; collision box size=5.48 0.2 3.0; visual box size=5.48 0.2 3.0
- added link 7_sec_6_right_conn; collision box size=0.2 0.78 3.0; visual box size=0.2 0.78 3.0
- added link 7_sec_6_right_wall; collision box size=5.48 0.2 3.0; visual box size=5.48 0.2 3.0
- added link 7_sec_7_left_conn; collision box size=0.2 0.455 3.0; visual box size=0.2 0.455 3.0
- added link 7_sec_7_left_wall; collision box size=4.26 0.2 3.0; visual box size=4.26 0.2 3.0
- added link 7_sec_7_right_conn; collision box size=0.2 0.455 3.0; visual box size=0.2 0.455 3.0
- added link 7_sec_7_right_wall; collision box size=4.26 0.2 3.0; visual box size=4.26 0.2 3.0
- added link 7_sec_8_left_conn; collision box size=0.2 0.695 3.0; visual box size=0.2 0.695 3.0
- added link 7_sec_8_left_wall; collision box size=3.86 0.2 3.0; visual box size=3.86 0.2 3.0
- added link 7_sec_8_right_conn; collision box size=0.2 0.695 3.0; visual box size=0.2 0.695 3.0
- added link 7_sec_8_right_wall; collision box size=3.86 0.2 3.0; visual box size=3.86 0.2 3.0
- added link 7_sec_9_left_wall; collision box size=4.0 0.2 3.0; visual box size=4.0 0.2 3.0
- added link 7_sec_9_right_wall; collision box size=4.0 0.2 3.0; visual box size=4.0 0.2 3.0
- link 2_sec_1_left_conn: geometry collision box size=0.2 0.905 3.0; visual box size=0.2 0.905 3.0
- link 2_sec_1_right_conn: geometry collision box size=0.2 0.905 3.0; visual box size=0.2 0.905 3.0
- link 2_sec_2_left_conn: geometry collision box size=0.2 0.745 3.0; visual box size=0.2 0.745 3.0
- link 2_sec_2_left_wall: geometry collision box size=5.27 0.2 3.0; visual box size=5.27 0.2 3.0
- link 2_sec_2_right_conn: geometry collision box size=0.2 0.745 3.0; visual box size=0.2 0.745 3.0
- link 2_sec_2_right_wall: geometry collision box size=5.27 0.2 3.0; visual box size=5.27 0.2 3.0
- link 2_sec_3_left_conn: geometry collision box size=0.2 0.83 3.0; visual box size=0.2 0.83 3.0
- link 2_sec_3_left_wall: geometry collision box size=3.97 0.2 3.0; visual box size=3.97 0.2 3.0
- link 2_sec_3_right_conn: geometry collision box size=0.2 0.83 3.0; visual box size=0.2 0.83 3.0
- link 2_sec_3_right_wall: geometry collision box size=3.97 0.2 3.0; visual box size=3.97 0.2 3.0
- link 2_sec_4_left_conn: geometry collision box size=0.2 0.505 3.0; visual box size=0.2 0.505 3.0
- link 2_sec_4_left_wall: geometry collision box size=3.75 0.2 3.0; visual box size=3.75 0.2 3.0
- link 2_sec_4_right_conn: geometry collision box size=0.2 0.505 3.0; visual box size=0.2 0.505 3.0
- link 2_sec_4_right_wall: geometry collision box size=3.75 0.2 3.0; visual box size=3.75 0.2 3.0
- link 2_sec_5_left_conn: geometry collision box size=0.2 0.7 3.0; visual box size=0.2 0.7 3.0
- link 2_sec_5_left_wall: geometry collision box size=3.15 0.2 3.0; visual box size=3.15 0.2 3.0
- link 2_sec_5_right_conn: geometry collision box size=0.2 0.7 3.0; visual box size=0.2 0.7 3.0
- link 2_sec_5_right_wall: geometry collision box size=3.15 0.2 3.0; visual box size=3.15 0.2 3.0
- link 2_sec_6_left_conn: geometry collision box size=0.2 0.29 3.0; visual box size=0.2 0.29 3.0
- link 2_sec_6_left_wall: geometry collision box size=2.39 0.2 3.0; visual box size=2.39 0.2 3.0
- link 2_sec_6_right_conn: geometry collision box size=0.2 0.29 3.0; visual box size=0.2 0.29 3.0
- link 2_sec_6_right_wall: geometry collision box size=2.39 0.2 3.0; visual box size=2.39 0.2 3.0
- link 2_sec_7_left_conn: geometry collision box size=0.2 0.38 3.0; visual box size=0.2 0.38 3.0
- link 2_sec_7_left_wall: geometry collision box size=3.84 0.2 3.0; visual box size=3.84 0.2 3.0
- link 2_sec_7_right_conn: geometry collision box size=0.2 0.38 3.0; visual box size=0.2 0.38 3.0
- link 2_sec_7_right_wall: geometry collision box size=3.84 0.2 3.0; visual box size=3.84 0.2 3.0
- link 2_sec_8_left_conn: geometry collision box size=0.2 0.31 3.0; visual box size=0.2 0.31 3.0
- link 2_sec_8_left_wall: geometry collision box size=3.49 0.2 3.0; visual box size=3.49 0.2 3.0
- link 2_sec_8_right_conn: geometry collision box size=0.2 0.31 3.0; visual box size=0.2 0.31 3.0
- link 2_sec_8_right_wall: geometry collision box size=3.49 0.2 3.0; visual box size=3.49 0.2 3.0
- link 2_sec_9_left_conn: geometry collision box size=0.2 0.595 3.0; visual box size=0.2 0.595 3.0
- link 2_sec_9_left_wall: geometry collision box size=5.83 0.2 3.0; visual box size=5.83 0.2 3.0
- link 2_sec_9_right_conn: geometry collision box size=0.2 0.595 3.0; visual box size=0.2 0.595 3.0
- link 2_sec_9_right_wall: geometry collision box size=5.83 0.2 3.0; visual box size=5.83 0.2 3.0
- link 4_sec_1_left_conn: geometry collision box size=1.315 0.2 3.0; visual box size=1.315 0.2 3.0
- link 4_sec_1_right_conn: geometry collision box size=1.315 0.2 3.0; visual box size=1.315 0.2 3.0
- link 4_sec_2_left_conn: geometry collision box size=0.635 0.2 3.0; visual box size=0.635 0.2 3.0
- link 4_sec_2_left_wall: geometry collision box size=0.2 4.66 3.0; visual box size=0.2 4.66 3.0
- link 4_sec_2_right_conn: geometry collision box size=0.635 0.2 3.0; visual box size=0.635 0.2 3.0
- link 4_sec_2_right_wall: geometry collision box size=0.2 4.66 3.0; visual box size=0.2 4.66 3.0
- link 4_sec_3_left_conn: geometry collision box size=0.425 0.2 3.0; visual box size=0.425 0.2 3.0
- link 4_sec_3_left_wall: geometry collision box size=0.2 2.88 3.0; visual box size=0.2 2.88 3.0
- link 4_sec_3_right_conn: geometry collision box size=0.425 0.2 3.0; visual box size=0.425 0.2 3.0
- link 4_sec_3_right_wall: geometry collision box size=0.2 2.88 3.0; visual box size=0.2 2.88 3.0
- link 4_sec_4_left_wall: geometry collision box size=0.2 2.73 3.0; visual box size=0.2 2.73 3.0
- link 4_sec_4_right_wall: geometry collision box size=0.2 2.73 3.0; visual box size=0.2 2.73 3.0
- link 6_sec_1_left_conn: geometry collision box size=-0.2 -1.7 3.0; visual box size=-0.2 -1.7 3.0
- link 6_sec_1_right_conn: geometry collision box size=-0.2 -1.7 3.0; visual box size=-0.2 -1.7 3.0
- link 6_sec_2_left_conn: geometry collision box size=-0.2 -1.45 3.0; visual box size=-0.2 -1.45 3.0
- link 6_sec_2_left_wall: geometry collision box size=-3.04 -0.2 3.0; visual box size=-3.04 -0.2 3.0
- link 6_sec_2_right_conn: geometry collision box size=-0.2 -1.45 3.0; visual box size=-0.2 -1.45 3.0
- link 6_sec_2_right_wall: geometry collision box size=-3.04 -0.2 3.0; visual box size=-3.04 -0.2 3.0
- link 6_sec_3_left_conn: geometry collision box size=-0.2 -0.305 3.0; visual box size=-0.2 -0.305 3.0
- link 6_sec_3_left_wall: geometry collision box size=-4.39 -0.2 3.0; visual box size=-4.39 -0.2 3.0
- link 6_sec_3_right_conn: geometry collision box size=-0.2 -0.305 3.0; visual box size=-0.2 -0.305 3.0
- link 6_sec_3_right_wall: geometry collision box size=-4.39 -0.2 3.0; visual box size=-4.39 -0.2 3.0
- link 6_sec_4_left_conn: geometry collision box size=-0.2 -0.345 3.0; visual box size=-0.2 -0.345 3.0
- link 6_sec_4_left_wall: geometry collision box size=-5.31 -0.2 3.0; visual box size=-5.31 -0.2 3.0
- link 6_sec_4_right_conn: geometry collision box size=-0.2 -0.345 3.0; visual box size=-0.2 -0.345 3.0
- link 6_sec_4_right_wall: geometry collision box size=-5.31 -0.2 3.0; visual box size=-5.31 -0.2 3.0
- link base: geometry collision box size=500 500 0.2; visual box size=500 500 0.2
Joints:
- removed joint joint_5_int_side_2
- added joint joint_4_sec_4_left_conn: type fixed, parent base, child 4_sec_4_left_conn, origin xyz=0 0 0 rpy=0 0 0
- added joint joint_4_sec_4_right_conn: type fixed, parent base, child 4_sec_4_right_conn, origin xyz=0 0 0 rpy=0 0 0
- added joint joint_4_sec_5_left_conn: type fixed, parent base, child 4_sec_5_left_conn, origin xyz=0 0 0 rpy=0 0 0
- added joint joint_4_sec_5_left_wall: type fixed, parent base, child 4_sec_5_left_wall, origin xyz=0 0 0 rpy=0 0 0
- added joint joint_4_sec_5_right_conn: type fixed, parent base, child 4_sec_5_right_conn, origin xyz=0 0 0 rpy=0 0 0
- added joint joint_4_sec_5_right_wall: type fixed, parent base, child 4_sec_5_right_wall, origin xyz=0 0 0 rpy=0 0 0
- added joint joint_4_sec_6_left_conn: type fixed, parent base, child 4_sec_6_left_conn, origin xyz=0 0 0 rpy=0 0 0
- added joint joint_4_sec_6_left_wall: type fixed, parent base, child 4_sec_6_left_wall, origin xyz=0 0 0 rpy=0 0 0
- added joint joint_4_sec_6_right_conn: type fixed, parent base, child 4_sec_6_right_conn, origin xyz=0 0 0 rpy=0 0 0
- added joint joint_4_sec_6_right_wall: type fixed, parent base, child 4_sec_6_right_wall, origin xyz=0 0 0 rpy=0 0 0
- added joint joint_4_sec_7_left_conn: type fixed, parent base, child 4_sec_7_left_conn, origin xyz=0 0 0 rpy=0 0 0
- added joint joint_4_sec_7_left_wall: type fixed, parent base, child 4_sec_7_left_wall, origin xyz=0 0 0 rpy=0 0 0
- added joint joint_4_sec_7_right_conn: type fixed, parent base, child 4_sec_7_right_conn, origin xyz=0 0 0 rpy=0 0 0
- added joint joint_4_sec_7_right_wall: type fixed, parent base, child 4_sec_7_right_wall, origin xyz=0 0 0 rpy=0 0 0
- added joint joint_4_sec_8_left_conn: type fixed, parent base, child 4_sec_8_left_conn, origin xyz=0 0 0 rpy=0 0 0
- added joint joint_4_sec_8_left_wall: type fixed, parent base, child 4_sec_8_left_wall, origin xyz=0 0 0 rpy=0 0 0
- added joint joint_4_sec_8_right_conn: type fixed, parent base, child 4_sec_8_right_conn, origin xyz=0 0 0 rpy=0 0 0
- added joint joint_4_sec_8_right_wall: type fixed, parent base, child 4_sec_8_right_wall, origin xyz=0 0 0 rpy=0 0 0
- added joint joint_4_sec_9_left_wall: type fixed, parent base, child 4_sec_9_left_wall, origin xyz=0 0 0 rpy=0 0 0
- added joint joint_4_sec_9_right_wall: type fixed, parent base, child 4_sec_9_right_wall, origin xyz=0 0 0 rpy=0 0 0
- added joint joint_5_int_side_2_left: type fixed, parent base, child 5_int_side_2_left, origin xyz=0 0 0 rpy=0 0 0
- added joint joint_5_int_side_2_right: type fixed, parent base, child 5_int_side_2_right, origin xyz=0 0 0 rpy=0 0 0
- added joint joint_7_sec_1_left_conn: type fixed, parent base, child 7_sec_1_left_conn, origin xyz=0 0 0 rpy=0 0 0
- added joint joint_7_sec_1_left_wall: type fixed, parent base, child 7_sec_1_left_wall, origin xyz=0 0 0 rpy=0 0 0
- added joint joint_7_sec_1_right_conn: type fixed, parent base, child 7_sec_1_right_conn, origin xyz=0 0 0 rpy=0 0 0
- added joint joint_7_sec_1_right_wall: type fixed, parent base, child 7_sec_1_right_wall, origin xyz=0 0 0 rpy=0 0 0
- added joint joint_7_sec_2_left_conn: type fixed, parent base, child 7_sec_2_left_conn, origin xyz=0 0 0 rpy=0 0 0
- added joint joint_7_sec_2_left_wall: type fixed, parent base, child 7_sec_2_left_wall, origin xyz=0 0 0 rpy=0 0 0
- added joint joint_7_sec_2_right_conn: type fixed, parent base, child 7_sec_2_right_conn, origin xyz=0 0 0 rpy=0 0 0
- added joint joint_7_sec_2_right_wall: type fixed, parent base, child 7_sec_2_right_wall, origin xyz=0 0 0 rpy=0 0 0
- added joint joint_7_sec_3_left_conn: type fixed, parent base, child 7_sec_3_left_conn, origin xyz=0 0 0 rpy=0 0 0
- added joint joint_7_sec_3_left_wall: type fixed, parent base, child 7_sec_3_left_wall, origin xyz=0 0 0 rpy=0 0 0
- added joint joint_7_sec_3_right_conn: type fixed, parent base, child 7_sec_3_right_conn, origin xyz=0 0 0 rpy=0 0 0
- added joint joint_7_sec_3_right_wall: type fixed, parent base, child 7_sec_3_right_wall, origin xyz=0 0 0 rpy=0 0 0
- added joint joint_7_sec_4_left_conn: type fixed, parent base, child 7_sec_4_left_conn, origin xyz=0 0 0 rpy=0 0 0
- added joint joint_7_sec_4_left_wall: type fixed, parent base, child 7_sec_4_left_wall, origin xyz=0 0 0 rpy=0 0 0
- added joint joint_7_sec_4_right_conn: type fixed, parent base, child 7_sec_4_right_conn, origin xyz=0 0 0 rpy=0 0 0
- added joint joint_7_sec_4_right_wall: type fixed, parent base, child 7_sec_4_right_wall, origin xyz=0 0 0 rpy=0 0 0
- added joint joint_7_sec_5_left_conn: type fixed, parent base, child 7_sec_5_left_conn, origin xyz=0 0 0 rpy=0 0 0
- added joint joint_7_sec_5_left_wall: type fixed, parent base, child 7_sec_5_left_wall, origin xyz=0 0 0 rpy=0 0 0
- added joint joint_7_sec_5_right_conn: type fixed, parent base, child 7_sec_5_right_conn, origin xyz=0 0 0 rpy=0 0 0
- added joint joint_7_sec_5_right_wall: type fixed, parent base, child 7_sec_5_right_wall, origin xyz=0 0 0 rpy=0 0 0
- added joint joint_7_sec_6_left_conn: type fixed, parent base, child 7_sec_6_left_conn, origin xyz=0 0 0 rpy=0 0 0
- added joint joint_7_sec_6_left_wall: type fixed, parent base, child 7_sec_6_left_wall, origin xyz=0 0 0 rpy=0 0 0
- added joint joint_7_sec_6_right_conn: type fixed, parent base, child 7_sec_6_right_conn, origin xyz=0 0 0 rpy=0 0 0
- added joint joint_7_sec_6_right_wall: type fixed, parent base, child 7_sec_6_right_wall, origin xyz=0 0 0 rpy=0 0 0
- added joint joint_7_sec_7_left_conn: type fixed, parent base, child 7_sec_7_left_conn, origin xyz=0 0 0 rpy=0 0 0
- added joint joint_7_sec_7_left_wall: type fixed, parent base, child 7_sec_7_left_wall, origin xyz=0 0 0 rpy=0 0 0
- added joint joint_7_sec_7_right_conn: type fixed, parent base, child 7_sec_7_right_conn, origin xyz=0 0 0 rpy=0 0 0
- added joint joint_7_sec_7_right_wall: type fixed, parent base, child 7_sec_7_right_wall, origin xyz=0 0 0 rpy=0 0 0
- added joint joint_7_sec_8_left_conn: type fixed, parent base, child 7_sec_8_left_conn, origin xyz=0 0 0 rpy=0 0 0
- added joint joint_7_sec_8_left_wall: type fixed, parent base, child 7_sec_8_left_wall, origin xyz=0 0 0 rpy=0 0 0
- added joint joint_7_sec_8_right_conn: type fixed, parent base, child 7_sec_8_right_conn, origin xyz=0 0 0 rpy=0 0 0
- added joint joint_7_sec_8_right_wall: type fixed, parent base, child 7_sec_8_right_wall, origin xyz=0 0 0 rpy=0 0 0
- added joint joint_7_sec_9_left_wall: type fixed, parent base, child 7_sec_9_left_wall, origin xyz=0 0 0 rpy=0 0 0
- added joint joint_7_sec_9_right_wall: type fixed, parent base, child 7_sec_9_right_wall, origin xyz=0 0 0 rpy=0 0 0
