Commit message: Update elevator.urdf

File: urdf/elevator.urdf (robot description, URDF)
Before this commit: robot elevator, 7 links, 6 joints
Joints:
- joint back_ground_joint: parent ground -> floor
- joint door_ground_joint: parent ground -> floor
- joint front_exterior_ground_joint: parent ground -> floor
- joint front_interior_ground_joint: parent ground -> floor
- joint left_ground_joint: parent ground -> floor
- joint right_ground_joint: parent ground -> floor

Commit message: Update elevator.urdf

File: urdf/elevator.urdf (robot description, URDF)
Before this commit: robot elevator, 7 links, 6 joints
Links:
- removed link back_wall
- removed link door
- removed link front_wall_exterior
- removed link front_wall_interior
- removed link left_wall
- removed link right_wall
Joints:
- removed joint back_ground_joint
- removed joint door_ground_joint
- removed joint front_exterior_ground_joint
- removed joint front_interior_ground_joint
- removed joint left_ground_joint
- removed joint right_ground_joint

Commit message: Update elevator.urdf

File: urdf/elevator.urdf (robot description, URDF)
Before this commit: robot elevator, 1 links, 0 joints
Links:
- added link front_wall_exterior; collision box size=1.5 0.125 3; visual box size=1.5 0.125 3
Joints:
- added joint front_exterior_ground_joint: type fixed, parent floor, child front_wall_exterior, origin xyz=0 0 0 rpy=0 0 0

Commit message: Update elevator.urdf

File: urdf/elevator.urdf (robot description, URDF)
Before this commit: robot elevator, 2 links, 1 joints
Links:
- added link front_wall_interior; collision box size=1.5 0.125 3; visual box size=1.5 0.125 3
Joints:
- added joint front_interior_ground_joint: type fixed, parent floor, child front_wall_interior, origin xyz=0 0 0 rpy=0 0 0

Commit message: Update elevator.urdf

File: urdf/elevator.urdf (robot description, URDF)
Before this commit: robot elevator, 3 links, 2 joints
Links:
- added link back_wall; collision box size=3 0.25 3; visual box size=3 0.25 3
Joints:
- added joint back_ground_joint: type fixed, parent floor, child back_wall, origin xyz=0 0 0 rpy=0 0 0

Commit message: Update elevator.urdf

File: urdf/elevator.urdf (robot description, URDF)
Before this commit: robot elevator, 4 links, 3 joints
Links:
- added link right_wall; collision box size=0.25 2.75 3; visual box size=0.25 2.75 3
Joints:
- added joint right_ground_joint: type fixed, parent floor, child right_wall, origin xyz=0 0 0 rpy=0 0 0

Commit message: Update elevator.urdf

File: urdf/elevator.urdf (robot description, URDF)
Before this commit: robot elevator, 5 links, 4 joints
Links:
- added link left_wall; collision box size=0.25 2.75 3; visual box size=0.25 2.75 3
Joints:
- added joint left_ground_joint: type fixed, parent floor, child left_wall, origin xyz=0 0 0 rpy=0 0 0

Commit message: Update elevator.urdf

File: urdf/elevator.urdf (robot description, URDF)
Before this commit: robot elevator, 6 links, 5 joints
Links:
- added link door; collision box size=1.75 0.25 3; visual box size=1.75 0.25 3
Joints:
- added joint door_ground_joint: type prismatic, parent floor, child door, origin xyz=0 0 0 rpy=0 0 0, axis 1 0 0, limit lower=-1.25 upper=1.25 effort=1000.0 velocity=0.1

Commit message: Update elevator.urdf

File: urdf/elevator.urdf (robot description, URDF)
Before this commit: robot elevator, 7 links, 6 joints
Joints:
- joint door_ground_joint: axis 1 0 0 -> 0 1 0

Commit message: Update elevator.urdf

File: urdf/elevator.urdf (robot description, URDF)
Before this commit: robot elevator, 7 links, 6 joints
Joints:
- joint door_ground_joint: axis 0 1 0 -> (none); limit lower=-1.25 upper=1.25 effort=1000.0 velocity=0.1 -> (none); type prismatic -> fixed

Commit message: Update elevator.urdf

File: urdf/elevator.urdf (robot description, URDF)
Before this commit: robot elevator, 7 links, 6 joints
Links:
- link door: geometry collision box size=1.75 0.25 3; visual box size=1.75 0.125 3

Commit message: Update elevator.urdf

File: urdf/elevator.urdf (robot description, URDF)
Before this commit: robot elevator, 7 links, 6 joints
Links:
- link door: geometry collision box size=1.75 0.25 3; visual box size=1.75 0.25 3

Commit message: Update elevator.urdf

File: urdf/elevator.urdf (robot description, URDF)
Before this commit: robot elevator, 7 links, 6 joints
Links:
- link door: geometry collision box size=1.25 0.25 3; visual box size=1.25 0.25 3
Joints:
- joint door_ground_joint: axis (none) -> 1 0 0; limit (none) -> lower=-0.625 upper=0.625 effort=1000.0 velocity=0.1; type fixed -> prismatic

Commit message: Update elevator.urdf

File: urdf/elevator.urdf (robot description, URDF)
Before this commit: robot elevator, 7 links, 6 joints
Joints:
- removed joint door_ground_joint
- added joint door_joint: type prismatic, parent front_wall_exterior, child door, origin xyz=0 0 0 rpy=0 0 0, axis 1 0 0, limit lower=-0.625 upper=0.625 effort=1000.0 velocity=0.1

Commit message: Update elevator.urdf

File: urdf/elevator.urdf (robot description, URDF)
Before this commit: robot elevator, 7 links, 6 joints
Joints:
- joint door_joint: origin xyz=0 0 0 rpy=0 0 0 -> xyz=0 1.125 1.5 rpy=0 0 0

Commit message: Update elevator.urdf

File: urdf/elevator.urdf (robot description, URDF)
Before this commit: robot elevator, 7 links, 6 joints
Joints:
- joint door_joint: axis 1 0 0 -> (none); origin xyz=0 1.125 1.5 rpy=0 0 0 -> xyz=0 1.125 0 rpy=0 0 0

Commit message: Update elevator.urdf

File: urdf/elevator.urdf (robot description, URDF)
Before this commit: robot elevator, 7 links, 6 joints
Joints:
- joint door_joint: axis (none) -> 1 0 0; origin xyz=0 1.125 0 rpy=0 0 0 -> xyz=0 0 0 rpy=0 0 0

Commit message: Update elevator.urdf

File: urdf/elevator.urdf (robot description, URDF)
Before this commit: robot elevator, 7 links, 6 joints
Links:
- removed link back_wall
- removed link floor
- removed link front_wall_interior
- removed link left_wall
- removed link right_wall
Joints:
- removed joint back_ground_joint
- removed joint front_exterior_ground_joint
- removed joint front_interior_ground_joint
- removed joint left_ground_joint
- removed joint right_ground_joint
- joint door_joint: origin xyz=0 0 0 rpy=0 0 0 -> xyz=0 -0.125 1.5 rpy=0 0 0

Commit message: Update elevator.urdf

File: urdf/elevator.urdf (robot description, URDF)
Before this commit: robot elevator, 2 links, 1 joints
Links:
- removed link front_wall_exterior
- added link front; visual box size=2 2 2
- link door: geometry visual box size=1 1 1
Joints:
- removed joint door_joint
- added joint front_to_door: type fixed, parent front, child door, origin xyz=0 -2 1

Commit message: Update elevator.urdf

File: urdf/elevator.urdf (robot description, URDF)
Before this commit: robot elevator, 2 links, 1 joints
Links:
- removed link front
- added link back_wall; collision box size=3 0.25 3; visual box size=3 0.25 3
- added link floor, mass 50; collision box size=3 2.75 0.5; visual box size=3 2.75 0.5
- added link front_wall_exterior; collision box size=1.5 0.125 3; visual box size=1.5 0.125 3
- added link front_wall_interior; collision box size=1.5 0.125 3; visual box size=1.5 0.125 3
- added link left_wall; collision box size=0.25 2.75 3; visual box size=0.25 2.75 3
- added link right_wall; collision box size=0.25 2.75 3; visual box size=0.25 2.75 3
- link door: geometry collision box size=1.25 0.25 3; visual box size=1.25 0.25 3
Joints:
- removed joint front_to_door
- added joint back_ground_joint: type fixed, parent floor, child back_wall, origin xyz=0 0 0 rpy=0 0 0
- added joint door_joint: type prismatic, parent front_wall_exterior, child door, origin xyz=0 0 0 rpy=0 0 0, axis 1 0 0, limit lower=-0.625 upper=0.625 effort=1000.0 velocity=0.1
- added joint front_exterior_ground_joint: type fixed, parent floor, child front_wall_exterior, origin xyz=0 0 0 rpy=0 0 0
- added joint front_interior_ground_joint: type fixed, parent floor, child front_wall_interior, origin xyz=0 0 0 rpy=0 0 0
- added joint left_ground_joint: type fixed, parent floor, child left_wall, origin xyz=0 0 0 rpy=0 0 0
- added joint right_ground_joint: type fixed, parent floor, child right_wall, origin xyz=0 0 0 rpy=0 0 0

Commit message: Update elevator.urdf

File: urdf/elevator.urdf (robot description, URDF)
Before this commit: robot elevator, 6 links, 5 joints
Links:
- added link door; collision box size=0.25 1.25 3; visual box size=0.25 1.25 3
Joints:
- added joint door_ground_joint: type fixed, parent floor, child door, origin xyz=0 0 0 rpy=0 0 0

Commit message: Update elevator.urdf

File: urdf/elevator.urdf (robot description, URDF)
Before this commit: robot elevator, 7 links, 6 joints
Links:
- link door: geometry collision box size=1.25 0.25 3; visual box size=1.25 0.25 3

Commit message: Update elevator.urdf

File: urdf/elevator.urdf (robot description, URDF)
Before this commit: robot elevator, 7 links, 6 joints
Links:
- link back_wall: mass None -> 50
- link door: mass None -> 50
- link front_wall_exterior: mass None -> 50
- link front_wall_interior: mass None -> 50
- link left_wall: mass None -> 50
- link right_wall: mass None -> 50
Joints:
- joint door_ground_joint: axis (none) -> 1 0 0; limit (none) -> lower=-0.625 upper=0.625 effort=1000.0 velocity=0.1; type fixed -> prismatic

Commit message: Update elevator.urdf

File: urdf/elevator.urdf (robot description, URDF)
Before this commit: robot elevator, 7 links, 6 joints
Links:
- added link left_panel, mass 50; collision box size=1 0.25 3; visual box size=1 0.25 3
- added link panel_floor_left, mass 50; collision box size=1 0.25 0.5; visual box size=1 0.25 0.5
- added link panel_floor_right, mass 50; collision box size=1 0.25 0.5; visual box size=1 0.25 0.5

Commit message: Update elevator.urdf

File: urdf/elevator.urdf (robot description, URDF)
Before this commit: robot elevator, 10 links, 6 joints
Links:
- added link right_panel, mass 50; collision box size=1 0.25 3; visual box sizw=1 0.25 3
Joints:
- added joint ground_panel_floor_left_joint: type fixed, parent floor, child panel_floor_left, origin xyz=0 0 0 rpy=0 0 0
- added joint ground_panel_floor_right_joint: type fixed, parent floor, child panel_floor_right, origin xyz=0 0 0 rpy=0 0 0
- added joint left_panel_floor_joint: type fixed, parent panel_floor_left, child left_panel, origin xyz=0 0 0 rpy=0 0 0
- added joint right_panel_floor_joint: type fixed, parent panel_floor_right, child right_panel, origin xyz=0 0 0 rpy=0 0 0

Commit message: Update elevator.urdf

File: urdf/elevator.urdf (robot description, URDF)
Before this commit: robot elevator, 11 links, 10 joints
Links:
- link right_panel: geometry collision box size=1 0.25 3; visual box size=1 0.25 3

Commit message: Update elevator.urdf

File: urdf/elevator.urdf (robot description, URDF)
Before this commit: robot elevator, 11 links, 10 joints
Links:
- added link Inner_Button, mass 0.00001; collision sphere radius=0.02; visual sphere radius=0.02
- added link Outer_Button, mass 0.00001; collision sphere radius=0.02; visual sphere radius=0.02
Joints:
- added joint inner_button_wall_joint: type fixed, parent front_wall_interior, child Inner_Button, origin xyz=0 0 0 rpy=0 0 0
- added joint outer_button_panel_joint: type fixed, parent left_panel, child Outer_Button, origin xyz=0 0 0 rpy=0 0 0

Commit message: Update elevator.urdf

File: urdf/elevator.urdf (robot description, URDF)
Before this commit: robot elevator, 13 links, 12 joints
Joints:
- joint inner_button_wall_joint: axis (none) -> 1 0 0; limit (none) -> lower=0.0 upper=0.0 effort=1000000000000000000000.0 velocity=0.0; type fixed -> revolute
- joint outer_button_panel_joint: axis (none) -> 1 0 0; limit (none) -> lower=0.0 upper=0.0 effort=1000000000000000000000.0 velocity=0.0; type fixed -> revolute

Commit message: Update elevator.urdf

File: urdf/elevator.urdf (robot description, URDF)
Before this commit: robot elevator, 13 links, 12 joints
Links:
- link door: mass 50 -> 0.5
