Commit message: add generation script

File: urdf/random_hall.urdf (robot description, URDF)
Before this commit: robot hallway, 39 links, 38 joints
Links:
- link base: mass None -> 50; geometry collision box size=22.0 6.0 0.2; visual box size=22.0 6.0 0.2
- link sec_10_left_wall: geometry collision box size=2.56 0.2 3.0; visual box size=2.56 0.2 3.0
- link sec_10_right_wall: geometry collision box size=2.56 0.2 3.0; visual box size=2.56 0.2 3.0
- link sec_1_left_conn: geometry collision box size=0.2 1.34 3.0; visual box size=0.2 1.34 3.0
- link sec_1_left_wall: geometry collision box size=1.95 0.2 3.0; visual box size=1.95 0.2 3.0
- link sec_1_right_conn: geometry collision box size=0.2 1.34 3.0; visual box size=0.2 1.34 3.0
- link sec_1_right_wall: geometry collision box size=1.95 0.2 3.0; visual box size=1.95 0.2 3.0
- link sec_2_left_conn: geometry collision box size=0.2 0.69 3.0; visual box size=0.2 0.69 3.0
- link sec_2_left_wall: geometry collision box size=2.13 0.2 3.0; visual box size=2.13 0.2 3.0
- link sec_2_right_conn: geometry collision box size=0.2 0.69 3.0; visual box size=0.2 0.69 3.0
- link sec_2_right_wall: geometry collision box size=2.13 0.2 3.0; visual box size=2.13 0.2 3.0
- link sec_3_left_conn: geometry collision box size=0.2 0.295 3.0; visual box size=0.2 0.295 3.0
- link sec_3_left_wall: geometry collision box size=2.2 0.2 3.0; visual box size=2.2 0.2 3.0
- link sec_3_right_conn: geometry collision box size=0.2 0.295 3.0; visual box size=0.2 0.295 3.0
- link sec_3_right_wall: geometry collision box size=2.2 0.2 3.0; visual box size=2.2 0.2 3.0
- link sec_4_left_conn: geometry collision box size=0.2 0.99 3.0; visual box size=0.2 0.99 3.0
- link sec_4_left_wall: geometry collision box size=1.69 0.2 3.0; visual box size=1.69 0.2 3.0
- link sec_4_right_conn: geometry collision box size=0.2 0.99 3.0; visual box size=0.2 0.99 3.0
- link sec_4_right_wall: geometry collision box size=1.69 0.2 3.0; visual box size=1.69 0.2 3.0
- link sec_5_left_conn: geometry collision box size=0.2 1.12 3.0; visual box size=0.2 1.12 3.0
- link sec_5_left_wall: geometry collision box size=2.15 0.2 3.0; visual box size=2.15 0.2 3.0
- link sec_5_right_conn: geometry collision box size=0.2 1.12 3.0; visual box size=0.2 1.12 3.0
- link sec_5_right_wall: geometry collision box size=2.15 0.2 3.0; visual box size=2.15 0.2 3.0
- link sec_6_left_conn: geometry collision box size=0.2 0.985 3.0; visual box size=0.2 0.985 3.0
- link sec_6_left_wall: geometry collision box size=2.38 0.2 3.0; visual box size=2.38 0.2 3.0
- link sec_6_right_conn: geometry collision box size=0.2 0.985 3.0; visual box size=0.2 0.985 3.0
- link sec_6_right_wall: geometry collision box size=2.38 0.2 3.0; visual box size=2.38 0.2 3.0
- link sec_7_left_conn: geometry collision box size=0.2 1.07 3.0; visual box size=0.2 1.07 3.0
- link sec_7_left_wall: geometry collision box size=2.72 0.2 3.0; visual box size=2.72 0.2 3.0
- link sec_7_right_conn: geometry collision box size=0.2 1.07 3.0; visual box size=0.2 1.07 3.0
- link sec_7_right_wall: geometry collision box size=2.72 0.2 3.0; visual box size=2.72 0.2 3.0
- link sec_8_left_conn: geometry collision box size=0.2 0.55 3.0; visual box size=0.2 0.55 3.0
- link sec_8_left_wall: geometry collision box size=2.05 0.2 3.0; visual box size=2.05 0.2 3.0
- link sec_8_right_conn: geometry collision box size=0.2 0.55 3.0; visual box size=0.2 0.55 3.0
- link sec_8_right_wall: geometry collision box size=2.05 0.2 3.0; visual box size=2.05 0.2 3.0
- link sec_9_left_conn: geometry collision box size=0.2 1.15 3.0; visual box size=0.2 1.15 3.0
- link sec_9_left_wall: geometry collision box size=2.17 0.2 3.0; visual box size=2.17 0.2 3.0
- link sec_9_right_conn: geometry collision box size=0.2 1.15 3.0; visual box size=0.2 1.15 3.0
- link sec_9_right_wall: geometry collision box size=2.17 0.2 3.0; visual box size=2.17 0.2 3.0
Joints:
- joint joint_sec_10_left_wall: origin xyz=17.635 1.985 1.5 rpy=0 0 0 -> xyz=20.72 1.295 1.5 rpy=0 0 0
- joint joint_sec_10_right_wall: origin xyz=17.635 -1.985 1.5 rpy=0 0 0 -> xyz=20.72 -1.295 1.5 rpy=0 0 0
- joint joint_sec_1_left_conn: origin xyz=1.78 1.965 1.5 rpy=0 0 0 -> xyz=1.95 2.185 1.5 rpy=0 0 0
- joint joint_sec_1_left_wall: origin xyz=0.89 1.82 1.5 rpy=0 0 0 -> xyz=0.975 2.855 1.5 rpy=0 0 0
- joint joint_sec_1_right_conn: origin xyz=1.78 -1.965 1.5 rpy=0 0 0 -> xyz=1.95 -2.185 1.5 rpy=0 0 0
- joint joint_sec_1_right_wall: origin xyz=0.89 -1.82 1.5 rpy=0 0 0 -> xyz=0.975 -2.855 1.5 rpy=0 0 0
- joint joint_sec_2_left_conn: origin xyz=3.85 1.83 1.5 rpy=0 0 0 -> xyz=4.08 1.86 1.5 rpy=0 0 0
- joint joint_sec_2_left_wall: origin xyz=2.815 2.31 1.5 rpy=0 0 0 -> xyz=3.015 1.715 1.5 rpy=0 0 0
- joint joint_sec_2_right_conn: origin xyz=3.85 -1.83 1.5 rpy=0 0 0 -> xyz=4.08 -1.86 1.5 rpy=0 0 0
- joint joint_sec_2_right_wall: origin xyz=2.815 -2.31 1.5 rpy=0 0 0 -> xyz=3.015 -1.715 1.5 rpy=0 0 0
- joint joint_sec_3_left_conn: origin xyz=5.22 2.02 1.5 rpy=0 0 0 -> xyz=6.28 2.0575 1.5 rpy=0 0 0
- joint joint_sec_3_left_wall: origin xyz=4.535 1.55 1.5 rpy=0 0 0 -> xyz=5.18 2.205 1.5 rpy=0 0 0
- joint joint_sec_3_right_conn: origin xyz=5.22 -2.02 1.5 rpy=0 0 0 -> xyz=6.28 -2.0575 1.5 rpy=0 0 0
- joint joint_sec_3_right_wall: origin xyz=4.535 -1.55 1.5 rpy=0 0 0 -> xyz=5.18 -2.205 1.5 rpy=0 0 0
- joint joint_sec_4_left_conn: origin xyz=5.72 2.32 1.5 rpy=0 0 0 -> xyz=7.97 2.405 1.5 rpy=0 0 0
- joint joint_sec_4_left_wall: origin xyz=5.47 2.69 1.5 rpy=0 0 0 -> xyz=7.125 2.11 1.5 rpy=0 0 0
- joint joint_sec_4_right_conn: origin xyz=5.72 -2.32 1.5 rpy=0 0 0 -> xyz=7.97 -2.405 1.5 rpy=0 0 0
- joint joint_sec_4_right_wall: origin xyz=5.47 -2.69 1.5 rpy=0 0 0 -> xyz=7.125 -2.11 1.5 rpy=0 0 0
- joint joint_sec_5_left_conn: origin xyz=6.97 2.5525 1.5 rpy=0 0 0 -> xyz=10.12 2.34 1.5 rpy=0 0 0
- joint joint_sec_5_left_wall: origin xyz=6.345 2.15 1.5 rpy=0 0 0 -> xyz=9.045 2.9 1.5 rpy=0 0 0
- joint joint_sec_5_right_conn: origin xyz=6.97 -2.5525 1.5 rpy=0 0 0 -> xyz=10.12 -2.34 1.5 rpy=0 0 0
- joint joint_sec_5_right_wall: origin xyz=6.345 -2.15 1.5 rpy=0 0 0 -> xyz=9.045 -2.9 1.5 rpy=0 0 0
- joint joint_sec_6_left_conn: origin xyz=8.93 2.98 1.5 rpy=0 0 0 -> xyz=12.5 2.2725 1.5 rpy=0 0 0
- joint joint_sec_6_left_wall: origin xyz=7.95 3.155 1.5 rpy=0 0 0 -> xyz=11.31 1.98 1.5 rpy=0 0 0
- joint joint_sec_6_right_conn: origin xyz=8.93 -2.98 1.5 rpy=0 0 0 -> xyz=12.5 -2.2725 1.5 rpy=0 0 0
- joint joint_sec_6_right_wall: origin xyz=7.95 -3.155 1.5 rpy=0 0 0 -> xyz=11.31 -1.98 1.5 rpy=0 0 0
- joint joint_sec_7_left_conn: origin xyz=11.73 2.4525 1.5 rpy=0 0 0 -> xyz=15.22 2.23 1.5 rpy=0 0 0
- joint joint_sec_7_left_wall: origin xyz=10.33 3.005 1.5 rpy=0 0 0 -> xyz=13.86 2.765 1.5 rpy=0 0 0
- joint joint_sec_7_right_conn: origin xyz=11.73 -2.4525 1.5 rpy=0 0 0 -> xyz=15.22 -2.23 1.5 rpy=0 0 0
- joint joint_sec_7_right_wall: origin xyz=10.33 -3.005 1.5 rpy=0 0 0 -> xyz=13.86 -2.765 1.5 rpy=0 0 0
- joint joint_sec_8_left_conn: origin xyz=13.73 1.55 1.5 rpy=0 0 0 -> xyz=17.27 1.97 1.5 rpy=0 0 0
- joint joint_sec_8_left_wall: origin xyz=12.73 2.1 1.5 rpy=0 0 0 -> xyz=16.245 1.895 1.5 rpy=0 0 0
- joint joint_sec_8_right_conn: origin xyz=13.73 -1.55 1.5 rpy=0 0 0 -> xyz=17.27 -1.97 1.5 rpy=0 0 0
- joint joint_sec_8_right_wall: origin xyz=12.73 -2.1 1.5 rpy=0 0 0 -> xyz=16.245 -1.895 1.5 rpy=0 0 0
- joint joint_sec_9_left_conn: origin xyz=16.28 1.4925 1.5 rpy=0 0 0 -> xyz=19.44 1.67 1.5 rpy=0 0 0
- joint joint_sec_9_left_wall: origin xyz=15.005 1.2 1.5 rpy=0 0 0 -> xyz=18.355 2.245 1.5 rpy=0 0 0
- joint joint_sec_9_right_conn: origin xyz=16.28 -1.4925 1.5 rpy=0 0 0 -> xyz=19.44 -1.67 1.5 rpy=0 0 0
- joint joint_sec_9_right_wall: origin xyz=15.005 -1.2 1.5 rpy=0 0 0 -> xyz=18.355 -2.245 1.5 rpy=0 0 0

Commit message: added node

File: urdf/random_hall.urdf (robot description, URDF)
Before this commit: robot hallway, 39 links, 38 joints
Links:
- link base: geometry collision box size=48.17 5.15 0.2; visual box size=48.17 5.15 0.2
- link sec_10_left_wall: geometry collision box size=6.2 0.2 3.0; visual box size=6.2 0.2 3.0
- link sec_10_right_wall: geometry collision box size=6.2 0.2 3.0; visual box size=6.2 0.2 3.0
- link sec_1_left_conn: geometry collision box size=0.2 0.355 3.0; visual box size=0.2 0.355 3.0
- link sec_1_left_wall: geometry collision box size=4.74 0.2 3.0; visual box size=4.74 0.2 3.0
- link sec_1_right_conn: geometry collision box size=0.2 0.355 3.0; visual box size=0.2 0.355 3.0
- link sec_1_right_wall: geometry collision box size=4.74 0.2 3.0; visual box size=4.74 0.2 3.0
- link sec_2_left_conn: geometry collision box size=0.2 0.52 3.0; visual box size=0.2 0.52 3.0
- link sec_2_left_wall: geometry collision box size=3.92 0.2 3.0; visual box size=3.92 0.2 3.0
- link sec_2_right_conn: geometry collision box size=0.2 0.52 3.0; visual box size=0.2 0.52 3.0
- link sec_2_right_wall: geometry collision box size=3.92 0.2 3.0; visual box size=3.92 0.2 3.0
- link sec_3_left_conn: geometry collision box size=0.2 0.36 3.0; visual box size=0.2 0.36 3.0
- link sec_3_left_wall: geometry collision box size=3.42 0.2 3.0; visual box size=3.42 0.2 3.0
- link sec_3_right_conn: geometry collision box size=0.2 0.36 3.0; visual box size=0.2 0.36 3.0
- link sec_3_right_wall: geometry collision box size=3.42 0.2 3.0; visual box size=3.42 0.2 3.0
- link sec_4_left_conn: geometry collision box size=0.2 0.205 3.0; visual box size=0.2 0.205 3.0
- link sec_4_left_wall: geometry collision box size=6.09 0.2 3.0; visual box size=6.09 0.2 3.0
- link sec_4_right_conn: geometry collision box size=0.2 0.205 3.0; visual box size=0.2 0.205 3.0
- link sec_4_right_wall: geometry collision box size=6.09 0.2 3.0; visual box size=6.09 0.2 3.0
- link sec_5_left_conn: geometry collision box size=0.2 0.34 3.0; visual box size=0.2 0.34 3.0
- link sec_5_left_wall: geometry collision box size=5.45 0.2 3.0; visual box size=5.45 0.2 3.0
- link sec_5_right_conn: geometry collision box size=0.2 0.34 3.0; visual box size=0.2 0.34 3.0
- link sec_5_right_wall: geometry collision box size=5.45 0.2 3.0; visual box size=5.45 0.2 3.0
- link sec_6_left_conn: geometry collision box size=0.2 0.365 3.0; visual box size=0.2 0.365 3.0
- link sec_6_left_wall: geometry collision box size=4.12 0.2 3.0; visual box size=4.12 0.2 3.0
- link sec_6_right_conn: geometry collision box size=0.2 0.365 3.0; visual box size=0.2 0.365 3.0
- link sec_6_right_wall: geometry collision box size=4.12 0.2 3.0; visual box size=4.12 0.2 3.0
- link sec_7_left_conn: geometry collision box size=0.2 0.9 3.0; visual box size=0.2 0.9 3.0
- link sec_7_left_wall: geometry collision box size=4.2 0.2 3.0; visual box size=4.2 0.2 3.0
- link sec_7_right_conn: geometry collision box size=0.2 0.9 3.0; visual box size=0.2 0.9 3.0
- link sec_7_right_wall: geometry collision box size=4.2 0.2 3.0; visual box size=4.2 0.2 3.0
- link sec_8_left_conn: geometry collision box size=0.2 1.17 3.0; visual box size=0.2 1.17 3.0
- link sec_8_left_wall: geometry collision box size=6.18 0.2 3.0; visual box size=6.18 0.2 3.0
- link sec_8_right_conn: geometry collision box size=0.2 1.17 3.0; visual box size=0.2 1.17 3.0
- link sec_8_right_wall: geometry collision box size=6.18 0.2 3.0; visual box size=6.18 0.2 3.0
- link sec_9_left_conn: geometry collision box size=0.2 0.73 3.0; visual box size=0.2 0.73 3.0
- link sec_9_left_wall: geometry collision box size=3.85 0.2 3.0; visual box size=3.85 0.2 3.0
- link sec_9_right_conn: geometry collision box size=0.2 0.73 3.0; visual box size=0.2 0.73 3.0
- link sec_9_right_wall: geometry collision box size=3.85 0.2 3.0; visual box size=3.85 0.2 3.0
Joints:
- joint joint_sec_10_left_wall: origin xyz=20.72 1.295 1.5 rpy=0 0 0 -> xyz=45.07 1.945 0 rpy=0 0 0
- joint joint_sec_10_right_wall: origin xyz=20.72 -1.295 1.5 rpy=0 0 0 -> xyz=45.07 -1.945 0 rpy=0 0 0
- joint joint_sec_1_left_conn: origin xyz=1.95 2.185 1.5 rpy=0 0 0 -> xyz=4.74 1.6825 0 rpy=0 0 0
- joint joint_sec_1_left_wall: origin xyz=0.975 2.855 1.5 rpy=0 0 0 -> xyz=2.37 1.86 0 rpy=0 0 0
- joint joint_sec_1_right_conn: origin xyz=1.95 -2.185 1.5 rpy=0 0 0 -> xyz=4.74 -1.6825 0 rpy=0 0 0
- joint joint_sec_1_right_wall: origin xyz=0.975 -2.855 1.5 rpy=0 0 0 -> xyz=2.37 -1.86 0 rpy=0 0 0
- joint joint_sec_2_left_conn: origin xyz=4.08 1.86 1.5 rpy=0 0 0 -> xyz=8.66 1.765 0 rpy=0 0 0
- joint joint_sec_2_left_wall: origin xyz=3.015 1.715 1.5 rpy=0 0 0 -> xyz=6.7 1.705 0 rpy=0 0 0
- joint joint_sec_2_right_conn: origin xyz=4.08 -1.86 1.5 rpy=0 0 0 -> xyz=8.66 -1.765 0 rpy=0 0 0
- joint joint_sec_2_right_wall: origin xyz=3.015 -1.715 1.5 rpy=0 0 0 -> xyz=6.7 -1.705 0 rpy=0 0 0
- joint joint_sec_3_left_conn: origin xyz=6.28 2.0575 1.5 rpy=0 0 0 -> xyz=12.08 2.005 0 rpy=0 0 0
- joint joint_sec_3_left_wall: origin xyz=5.18 2.205 1.5 rpy=0 0 0 -> xyz=10.37 2.025 0 rpy=0 0 0
- joint joint_sec_3_right_conn: origin xyz=6.28 -2.0575 1.5 rpy=0 0 0 -> xyz=12.08 -2.005 0 rpy=0 0 0
- joint joint_sec_3_right_wall: origin xyz=5.18 -2.205 1.5 rpy=0 0 0 -> xyz=10.37 -2.025 0 rpy=0 0 0
- joint joint_sec_4_left_conn: origin xyz=7.97 2.405 1.5 rpy=0 0 0 -> xyz=18.17 2.0825 0 rpy=0 0 0
- joint joint_sec_4_left_wall: origin xyz=7.125 2.11 1.5 rpy=0 0 0 -> xyz=15.125 2.185 0 rpy=0 0 0
- joint joint_sec_4_right_conn: origin xyz=7.97 -2.405 1.5 rpy=0 0 0 -> xyz=18.17 -2.0825 0 rpy=0 0 0
- joint joint_sec_4_right_wall: origin xyz=7.125 -2.11 1.5 rpy=0 0 0 -> xyz=15.125 -2.185 0 rpy=0 0 0
- joint joint_sec_5_left_conn: origin xyz=10.12 2.34 1.5 rpy=0 0 0 -> xyz=23.62 2.01 0 rpy=0 0 0
- joint joint_sec_5_left_wall: origin xyz=9.045 2.9 1.5 rpy=0 0 0 -> xyz=20.895 2.18 0 rpy=0 0 0
- joint joint_sec_5_right_conn: origin xyz=10.12 -2.34 1.5 rpy=0 0 0 -> xyz=23.62 -2.01 0 rpy=0 0 0
- joint joint_sec_5_right_wall: origin xyz=9.045 -2.9 1.5 rpy=0 0 0 -> xyz=20.895 -2.18 0 rpy=0 0 0
- joint joint_sec_6_left_conn: origin xyz=12.5 2.2725 1.5 rpy=0 0 0 -> xyz=27.74 2.0225 0 rpy=0 0 0
- joint joint_sec_6_left_wall: origin xyz=11.31 1.98 1.5 rpy=0 0 0 -> xyz=25.68 2.04 0 rpy=0 0 0
- joint joint_sec_6_right_conn: origin xyz=12.5 -2.2725 1.5 rpy=0 0 0 -> xyz=27.74 -2.0225 0 rpy=0 0 0
- joint joint_sec_6_right_wall: origin xyz=11.31 -1.98 1.5 rpy=0 0 0 -> xyz=25.68 -2.04 0 rpy=0 0 0
- joint joint_sec_7_left_conn: origin xyz=15.22 2.23 1.5 rpy=0 0 0 -> xyz=31.94 1.755 0 rpy=0 0 0
- joint joint_sec_7_left_wall: origin xyz=13.86 2.765 1.5 rpy=0 0 0 -> xyz=29.84 2.205 0 rpy=0 0 0
- joint joint_sec_7_right_conn: origin xyz=15.22 -2.23 1.5 rpy=0 0 0 -> xyz=31.94 -1.755 0 rpy=0 0 0
- joint joint_sec_7_right_wall: origin xyz=13.86 -2.765 1.5 rpy=0 0 0 -> xyz=29.84 -2.205 0 rpy=0 0 0
- joint joint_sec_8_left_conn: origin xyz=17.27 1.97 1.5 rpy=0 0 0 -> xyz=38.12 1.89 0 rpy=0 0 0
- joint joint_sec_8_left_wall: origin xyz=16.245 1.895 1.5 rpy=0 0 0 -> xyz=35.03 1.505 0 rpy=0 0 0
- joint joint_sec_8_right_conn: origin xyz=17.27 -1.97 1.5 rpy=0 0 0 -> xyz=38.12 -1.89 0 rpy=0 0 0
- joint joint_sec_8_right_wall: origin xyz=16.245 -1.895 1.5 rpy=0 0 0 -> xyz=35.03 -1.505 0 rpy=0 0 0
- joint joint_sec_9_left_conn: origin xyz=19.44 1.67 1.5 rpy=0 0 0 -> xyz=41.97 2.11 0 rpy=0 0 0
- joint joint_sec_9_left_wall: origin xyz=18.355 2.245 1.5 rpy=0 0 0 -> xyz=40.045 2.475 0 rpy=0 0 0
- joint joint_sec_9_right_conn: origin xyz=19.44 -1.67 1.5 rpy=0 0 0 -> xyz=41.97 -2.11 0 rpy=0 0 0
- joint joint_sec_9_right_wall: origin xyz=18.355 -2.245 1.5 rpy=0 0 0 -> xyz=40.045 -2.475 0 rpy=0 0 0

Commit message: made executable

File: urdf/random_hall.urdf (robot description, URDF)
Before this commit: robot hallway, 39 links, 38 joints
Links:
- link base: geometry collision box size=51.11 5.12 0.2; visual box size=51.11 5.12 0.2
- link sec_10_left_wall: geometry collision box size=3.59 0.2 3.0; visual box size=3.59 0.2 3.0
- link sec_10_right_wall: geometry collision box size=3.59 0.2 3.0; visual box size=3.59 0.2 3.0
- link sec_1_left_conn: geometry collision box size=0.2 1.03 3.0; visual box size=0.2 1.03 3.0
- link sec_1_left_wall: geometry collision box size=5.29 0.2 3.0; visual box size=5.29 0.2 3.0
- link sec_1_right_conn: geometry collision box size=0.2 1.03 3.0; visual box size=0.2 1.03 3.0
- link sec_1_right_wall: geometry collision box size=5.29 0.2 3.0; visual box size=5.29 0.2 3.0
- link sec_2_left_conn: geometry collision box size=0.2 0.285 3.0; visual box size=0.2 0.285 3.0
- link sec_2_left_wall: geometry collision box size=3.31 0.2 3.0; visual box size=3.31 0.2 3.0
- link sec_2_right_conn: geometry collision box size=0.2 0.285 3.0; visual box size=0.2 0.285 3.0
- link sec_2_right_wall: geometry collision box size=3.31 0.2 3.0; visual box size=3.31 0.2 3.0
- link sec_3_left_conn: geometry collision box size=0.2 0.235 3.0; visual box size=0.2 0.235 3.0
- link sec_3_left_wall: geometry collision box size=3.48 0.2 3.0; visual box size=3.48 0.2 3.0
- link sec_3_right_conn: geometry collision box size=0.2 0.235 3.0; visual box size=0.2 0.235 3.0
- link sec_3_right_wall: geometry collision box size=3.48 0.2 3.0; visual box size=3.48 0.2 3.0
- link sec_4_left_conn: geometry collision box size=0.2 0.36 3.0; visual box size=0.2 0.36 3.0
- link sec_4_left_wall: geometry collision box size=7.38 0.2 3.0; visual box size=7.38 0.2 3.0
- link sec_4_right_conn: geometry collision box size=0.2 0.36 3.0; visual box size=0.2 0.36 3.0
- link sec_4_right_wall: geometry collision box size=7.38 0.2 3.0; visual box size=7.38 0.2 3.0
- link sec_5_left_conn: geometry collision box size=0.2 0.52 3.0; visual box size=0.2 0.52 3.0
- link sec_5_left_wall: geometry collision box size=4.8 0.2 3.0; visual box size=4.8 0.2 3.0
- link sec_5_right_conn: geometry collision box size=0.2 0.52 3.0; visual box size=0.2 0.52 3.0
- link sec_5_right_wall: geometry collision box size=4.8 0.2 3.0; visual box size=4.8 0.2 3.0
- link sec_6_left_conn: geometry collision box size=0.2 0.57 3.0; visual box size=0.2 0.57 3.0
- link sec_6_left_wall: geometry collision box size=5.3 0.2 3.0; visual box size=5.3 0.2 3.0
- link sec_6_right_conn: geometry collision box size=0.2 0.57 3.0; visual box size=0.2 0.57 3.0
- link sec_6_right_wall: geometry collision box size=5.3 0.2 3.0; visual box size=5.3 0.2 3.0
- link sec_7_left_conn: geometry collision box size=0.2 0.5 3.0; visual box size=0.2 0.5 3.0
- link sec_7_left_wall: geometry collision box size=5.2 0.2 3.0; visual box size=5.2 0.2 3.0
- link sec_7_right_conn: geometry collision box size=0.2 0.5 3.0; visual box size=0.2 0.5 3.0
- link sec_7_right_wall: geometry collision box size=5.2 0.2 3.0; visual box size=5.2 0.2 3.0
- link sec_8_left_conn: geometry collision box size=0.2 0.215 3.0; visual box size=0.2 0.215 3.0
- link sec_8_left_wall: geometry collision box size=6.91 0.2 3.0; visual box size=6.91 0.2 3.0
- link sec_8_right_conn: geometry collision box size=0.2 0.215 3.0; visual box size=0.2 0.215 3.0
- link sec_8_right_wall: geometry collision box size=6.91 0.2 3.0; visual box size=6.91 0.2 3.0
- link sec_9_left_conn: geometry collision box size=0.2 0.755 3.0; visual box size=0.2 0.755 3.0
- link sec_9_left_wall: geometry collision box size=5.85 0.2 3.0; visual box size=5.85 0.2 3.0
- link sec_9_right_conn: geometry collision box size=0.2 0.755 3.0; visual box size=0.2 0.755 3.0
- link sec_9_right_wall: geometry collision box size=5.85 0.2 3.0; visual box size=5.85 0.2 3.0
Joints:
- joint joint_sec_10_left_wall: origin xyz=45.07 1.945 0 rpy=0 0 0 -> xyz=47.52 1.59 1.5 rpy=0 0 0
- joint joint_sec_10_right_wall: origin xyz=45.07 -1.945 0 rpy=0 0 0 -> xyz=47.52 -1.59 1.5 rpy=0 0 0
- joint joint_sec_1_left_conn: origin xyz=4.74 1.6825 0 rpy=0 0 0 -> xyz=5.29 1.945 1.5 rpy=0 0 0
- joint joint_sec_1_left_wall: origin xyz=2.37 1.86 0 rpy=0 0 0 -> xyz=0.0 2.46 1.5 rpy=0 0 0
- joint joint_sec_1_right_conn: origin xyz=4.74 -1.6825 0 rpy=0 0 0 -> xyz=5.29 -1.945 1.5 rpy=0 0 0
- joint joint_sec_1_right_wall: origin xyz=2.37 -1.86 0 rpy=0 0 0 -> xyz=0.0 -2.46 1.5 rpy=0 0 0
- joint joint_sec_2_left_conn: origin xyz=8.66 1.765 0 rpy=0 0 0 -> xyz=8.6 1.4875 1.5 rpy=0 0 0
- joint joint_sec_2_left_wall: origin xyz=6.7 1.705 0 rpy=0 0 0 -> xyz=5.29 1.63 1.5 rpy=0 0 0
- joint joint_sec_2_right_conn: origin xyz=8.66 -1.765 0 rpy=0 0 0 -> xyz=8.6 -1.4875 1.5 rpy=0 0 0
- joint joint_sec_2_right_wall: origin xyz=6.7 -1.705 0 rpy=0 0 0 -> xyz=5.29 -1.63 1.5 rpy=0 0 0
- joint joint_sec_3_left_conn: origin xyz=12.08 2.005 0 rpy=0 0 0 -> xyz=12.08 1.4625 1.5 rpy=0 0 0
- joint joint_sec_3_left_wall: origin xyz=10.37 2.025 0 rpy=0 0 0 -> xyz=8.6 1.545 1.5 rpy=0 0 0
- joint joint_sec_3_right_conn: origin xyz=12.08 -2.005 0 rpy=0 0 0 -> xyz=12.08 -1.4625 1.5 rpy=0 0 0
- joint joint_sec_3_right_wall: origin xyz=10.37 -2.025 0 rpy=0 0 0 -> xyz=8.6 -1.545 1.5 rpy=0 0 0
- joint joint_sec_4_left_conn: origin xyz=18.17 2.0825 0 rpy=0 0 0 -> xyz=19.46 1.56 1.5 rpy=0 0 0
- joint joint_sec_4_left_wall: origin xyz=15.125 2.185 0 rpy=0 0 0 -> xyz=12.08 1.58 1.5 rpy=0 0 0
- joint joint_sec_4_right_conn: origin xyz=18.17 -2.0825 0 rpy=0 0 0 -> xyz=19.46 -1.56 1.5 rpy=0 0 0
- joint joint_sec_4_right_wall: origin xyz=15.125 -2.185 0 rpy=0 0 0 -> xyz=12.08 -1.58 1.5 rpy=0 0 0
- joint joint_sec_5_left_conn: origin xyz=23.62 2.01 0 rpy=0 0 0 -> xyz=24.26 1.8 1.5 rpy=0 0 0
- joint joint_sec_5_left_wall: origin xyz=20.895 2.18 0 rpy=0 0 0 -> xyz=19.46 1.74 1.5 rpy=0 0 0
- joint joint_sec_5_right_conn: origin xyz=23.62 -2.01 0 rpy=0 0 0 -> xyz=24.26 -1.8 1.5 rpy=0 0 0
- joint joint_sec_5_right_wall: origin xyz=20.895 -2.18 0 rpy=0 0 0 -> xyz=19.46 -1.74 1.5 rpy=0 0 0
- joint joint_sec_6_left_conn: origin xyz=27.74 2.0225 0 rpy=0 0 0 -> xyz=29.56 2.145 1.5 rpy=0 0 0
- joint joint_sec_6_left_wall: origin xyz=25.68 2.04 0 rpy=0 0 0 -> xyz=24.26 2.06 1.5 rpy=0 0 0
- joint joint_sec_6_right_conn: origin xyz=27.74 -2.0225 0 rpy=0 0 0 -> xyz=29.56 -2.145 1.5 rpy=0 0 0
- joint joint_sec_6_right_wall: origin xyz=25.68 -2.04 0 rpy=0 0 0 -> xyz=24.26 -2.06 1.5 rpy=0 0 0
- joint joint_sec_7_left_conn: origin xyz=31.94 1.755 0 rpy=0 0 0 -> xyz=34.76 2.18 1.5 rpy=0 0 0
- joint joint_sec_7_left_wall: origin xyz=29.84 2.205 0 rpy=0 0 0 -> xyz=29.56 2.43 1.5 rpy=0 0 0
- joint joint_sec_7_right_conn: origin xyz=31.94 -1.755 0 rpy=0 0 0 -> xyz=34.76 -2.18 1.5 rpy=0 0 0
- joint joint_sec_7_right_wall: origin xyz=29.84 -2.205 0 rpy=0 0 0 -> xyz=29.56 -2.43 1.5 rpy=0 0 0
- joint joint_sec_8_left_conn: origin xyz=38.12 1.89 0 rpy=0 0 0 -> xyz=41.67 2.0375 1.5 rpy=0 0 0
- joint joint_sec_8_left_wall: origin xyz=35.03 1.505 0 rpy=0 0 0 -> xyz=34.76 2.13 1.5 rpy=0 0 0
- joint joint_sec_8_right_conn: origin xyz=38.12 -1.89 0 rpy=0 0 0 -> xyz=41.67 -2.0375 1.5 rpy=0 0 0
- joint joint_sec_8_right_wall: origin xyz=35.03 -1.505 0 rpy=0 0 0 -> xyz=34.76 -2.13 1.5 rpy=0 0 0
- joint joint_sec_9_left_conn: origin xyz=41.97 2.11 0 rpy=0 0 0 -> xyz=47.52 1.7675 1.5 rpy=0 0 0
- joint joint_sec_9_left_wall: origin xyz=40.045 2.475 0 rpy=0 0 0 -> xyz=41.67 2.145 1.5 rpy=0 0 0
- joint joint_sec_9_right_conn: origin xyz=41.97 -2.11 0 rpy=0 0 0 -> xyz=47.52 -1.7675 1.5 rpy=0 0 0
- joint joint_sec_9_right_wall: origin xyz=40.045 -2.475 0 rpy=0 0 0 -> xyz=41.67 -2.145 1.5 rpy=0 0 0
