Commit message: working hallway

File: urdf/random_hall.urdf (robot description, URDF)
Before this commit: robot hallway, 39 links, 38 joints
Links:
- link base: geometry collision box size=55.16 4.82 0.2; visual box size=55.16 4.82 0.2
- link sec_10_left_wall: geometry collision box size=5.39 0.2 3.0; visual box size=5.39 0.2 3.0
- link sec_10_right_wall: geometry collision box size=5.39 0.2 3.0; visual box size=5.39 0.2 3.0
- link sec_1_left_conn: geometry collision box size=0.2 0.925 3.0; visual box size=0.2 0.925 3.0
- link sec_1_left_wall: geometry collision box size=5.84 0.2 3.0; visual box size=5.84 0.2 3.0
- link sec_1_right_conn: geometry collision box size=0.2 0.925 3.0; visual box size=0.2 0.925 3.0
- link sec_1_right_wall: geometry collision box size=5.84 0.2 3.0; visual box size=5.84 0.2 3.0
- link sec_2_left_conn: geometry collision box size=0.2 0.595 3.0; visual box size=0.2 0.595 3.0
- link sec_2_left_wall: geometry collision box size=4.25 0.2 3.0; visual box size=4.25 0.2 3.0
- link sec_2_right_conn: geometry collision box size=0.2 0.595 3.0; visual box size=0.2 0.595 3.0
- link sec_2_right_wall: geometry collision box size=4.25 0.2 3.0; visual box size=4.25 0.2 3.0
- link sec_3_left_conn: geometry collision box size=0.2 0.455 3.0; visual box size=0.2 0.455 3.0
- link sec_3_left_wall: geometry collision box size=5.31 0.2 3.0; visual box size=5.31 0.2 3.0
- link sec_3_right_conn: geometry collision box size=0.2 0.455 3.0; visual box size=0.2 0.455 3.0
- link sec_3_right_wall: geometry collision box size=5.31 0.2 3.0; visual box size=5.31 0.2 3.0
- link sec_4_left_conn: geometry collision box size=0.2 0.51 3.0; visual box size=0.2 0.51 3.0
- link sec_4_left_wall: geometry collision box size=6.54 0.2 3.0; visual box size=6.54 0.2 3.0
- link sec_4_right_conn: geometry collision box size=0.2 0.51 3.0; visual box size=0.2 0.51 3.0
- link sec_4_right_wall: geometry collision box size=6.54 0.2 3.0; visual box size=6.54 0.2 3.0
- link sec_5_left_conn: geometry collision box size=0.2 0.475 3.0; visual box size=0.2 0.475 3.0
- link sec_5_left_wall: geometry collision box size=6.35 0.2 3.0; visual box size=6.35 0.2 3.0
- link sec_5_right_conn: geometry collision box size=0.2 0.475 3.0; visual box size=0.2 0.475 3.0
- link sec_5_right_wall: geometry collision box size=6.35 0.2 3.0; visual box size=6.35 0.2 3.0
- link sec_6_left_conn: geometry collision box size=0.2 0.225 3.0; visual box size=0.2 0.225 3.0
- link sec_6_left_wall: geometry collision box size=3.8 0.2 3.0; visual box size=3.8 0.2 3.0
- link sec_6_right_conn: geometry collision box size=0.2 0.225 3.0; visual box size=0.2 0.225 3.0
- link sec_6_right_wall: geometry collision box size=3.8 0.2 3.0; visual box size=3.8 0.2 3.0
- link sec_7_left_conn: geometry collision box size=0.2 0.41 3.0; visual box size=0.2 0.41 3.0
- link sec_7_left_wall: geometry collision box size=6.1 0.2 3.0; visual box size=6.1 0.2 3.0
- link sec_7_right_conn: geometry collision box size=0.2 0.41 3.0; visual box size=0.2 0.41 3.0
- link sec_7_right_wall: geometry collision box size=6.1 0.2 3.0; visual box size=6.1 0.2 3.0
- link sec_8_left_conn: geometry collision box size=0.2 0.435 3.0; visual box size=0.2 0.435 3.0
- link sec_8_left_wall: geometry collision box size=5.61 0.2 3.0; visual box size=5.61 0.2 3.0
- link sec_8_right_conn: geometry collision box size=0.2 0.435 3.0; visual box size=0.2 0.435 3.0
- link sec_8_right_wall: geometry collision box size=5.61 0.2 3.0; visual box size=5.61 0.2 3.0
- link sec_9_left_conn: geometry collision box size=0.2 0.365 3.0; visual box size=0.2 0.365 3.0
- link sec_9_left_wall: geometry collision box size=5.97 0.2 3.0; visual box size=5.97 0.2 3.0
- link sec_9_right_conn: geometry collision box size=0.2 0.365 3.0; visual box size=0.2 0.365 3.0
- link sec_9_right_wall: geometry collision box size=5.97 0.2 3.0; visual box size=5.97 0.2 3.0
Joints:
- joint joint_sec_10_left_wall: origin xyz=47.52 1.59 1.5 rpy=0 0 0 -> xyz=0 0 0 rpy=0 0 0
- joint joint_sec_10_right_wall: origin xyz=47.52 -1.59 1.5 rpy=0 0 0 -> xyz=0 0 0 rpy=0 0 0
- joint joint_sec_1_left_conn: origin xyz=5.29 1.945 1.5 rpy=0 0 0 -> xyz=0 0 0 rpy=0 0 0
- joint joint_sec_1_left_wall: origin xyz=0.0 2.46 1.5 rpy=0 0 0 -> xyz=0 0 0 rpy=0 0 0
- joint joint_sec_1_right_conn: origin xyz=5.29 -1.945 1.5 rpy=0 0 0 -> xyz=0 0 0 rpy=0 0 0
- joint joint_sec_1_right_wall: origin xyz=0.0 -2.46 1.5 rpy=0 0 0 -> xyz=0 0 0 rpy=0 0 0
- joint joint_sec_2_left_conn: origin xyz=8.6 1.4875 1.5 rpy=0 0 0 -> xyz=0 0 0 rpy=0 0 0
- joint joint_sec_2_left_wall: origin xyz=5.29 1.63 1.5 rpy=0 0 0 -> xyz=0 0 0 rpy=0 0 0
- joint joint_sec_2_right_conn: origin xyz=8.6 -1.4875 1.5 rpy=0 0 0 -> xyz=0 0 0 rpy=0 0 0
- joint joint_sec_2_right_wall: origin xyz=5.29 -1.63 1.5 rpy=0 0 0 -> xyz=0 0 0 rpy=0 0 0
- joint joint_sec_3_left_conn: origin xyz=12.08 1.4625 1.5 rpy=0 0 0 -> xyz=0 0 0 rpy=0 0 0
- joint joint_sec_3_left_wall: origin xyz=8.6 1.545 1.5 rpy=0 0 0 -> xyz=0 0 0 rpy=0 0 0
- joint joint_sec_3_right_conn: origin xyz=12.08 -1.4625 1.5 rpy=0 0 0 -> xyz=0 0 0 rpy=0 0 0
- joint joint_sec_3_right_wall: origin xyz=8.6 -1.545 1.5 rpy=0 0 0 -> xyz=0 0 0 rpy=0 0 0
- joint joint_sec_4_left_conn: origin xyz=19.46 1.56 1.5 rpy=0 0 0 -> xyz=0 0 0 rpy=0 0 0
- joint joint_sec_4_left_wall: origin xyz=12.08 1.58 1.5 rpy=0 0 0 -> xyz=0 0 0 rpy=0 0 0
- joint joint_sec_4_right_conn: origin xyz=19.46 -1.56 1.5 rpy=0 0 0 -> xyz=0 0 0 rpy=0 0 0
- joint joint_sec_4_right_wall: origin xyz=12.08 -1.58 1.5 rpy=0 0 0 -> xyz=0 0 0 rpy=0 0 0
- joint joint_sec_5_left_conn: origin xyz=24.26 1.8 1.5 rpy=0 0 0 -> xyz=0 0 0 rpy=0 0 0
- joint joint_sec_5_left_wall: origin xyz=19.46 1.74 1.5 rpy=0 0 0 -> xyz=0 0 0 rpy=0 0 0
- joint joint_sec_5_right_conn: origin xyz=24.26 -1.8 1.5 rpy=0 0 0 -> xyz=0 0 0 rpy=0 0 0
- joint joint_sec_5_right_wall: origin xyz=19.46 -1.74 1.5 rpy=0 0 0 -> xyz=0 0 0 rpy=0 0 0
- joint joint_sec_6_left_conn: origin xyz=29.56 2.145 1.5 rpy=0 0 0 -> xyz=0 0 0 rpy=0 0 0
- joint joint_sec_6_left_wall: origin xyz=24.26 2.06 1.5 rpy=0 0 0 -> xyz=0 0 0 rpy=0 0 0
- joint joint_sec_6_right_conn: origin xyz=29.56 -2.145 1.5 rpy=0 0 0 -> xyz=0 0 0 rpy=0 0 0
- joint joint_sec_6_right_wall: origin xyz=24.26 -2.06 1.5 rpy=0 0 0 -> xyz=0 0 0 rpy=0 0 0
- joint joint_sec_7_left_conn: origin xyz=34.76 2.18 1.5 rpy=0 0 0 -> xyz=0 0 0 rpy=0 0 0
- joint joint_sec_7_left_wall: origin xyz=29.56 2.43 1.5 rpy=0 0 0 -> xyz=0 0 0 rpy=0 0 0
- joint joint_sec_7_right_conn: origin xyz=34.76 -2.18 1.5 rpy=0 0 0 -> xyz=0 0 0 rpy=0 0 0
- joint joint_sec_7_right_wall: origin xyz=29.56 -2.43 1.5 rpy=0 0 0 -> xyz=0 0 0 rpy=0 0 0
- joint joint_sec_8_left_conn: origin xyz=41.67 2.0375 1.5 rpy=0 0 0 -> xyz=0 0 0 rpy=0 0 0
- joint joint_sec_8_left_wall: origin xyz=34.76 2.13 1.5 rpy=0 0 0 -> xyz=0 0 0 rpy=0 0 0
- joint joint_sec_8_right_conn: origin xyz=41.67 -2.0375 1.5 rpy=0 0 0 -> xyz=0 0 0 rpy=0 0 0
- joint joint_sec_8_right_wall: origin xyz=34.76 -2.13 1.5 rpy=0 0 0 -> xyz=0 0 0 rpy=0 0 0
- joint joint_sec_9_left_conn: origin xyz=47.52 1.7675 1.5 rpy=0 0 0 -> xyz=0 0 0 rpy=0 0 0
- joint joint_sec_9_left_wall: origin xyz=41.67 2.145 1.5 rpy=0 0 0 -> xyz=0 0 0 rpy=0 0 0
- joint joint_sec_9_right_conn: origin xyz=47.52 -1.7675 1.5 rpy=0 0 0 -> xyz=0 0 0 rpy=0 0 0
- joint joint_sec_9_right_wall: origin xyz=41.67 -2.145 1.5 rpy=0 0 0 -> xyz=0 0 0 rpy=0 0 0

File: urdf/room.urdf (robot description, URDF)
Before this commit: robot room, 5 links, 4 joints
Links:
- link ground: mass None -> 50; geometry collision box size=10 10 0.5; visual box size=10 10 0.5
Joints:
- joint back_joint: origin xyz=-5 0 1.5 rpy=0 0 0 -> xyz=0 0 0 rpy=0 0 0
- joint front_joint: origin xyz=5 0 1.5 rpy=0 0 0 -> xyz=0 0 0 rpy=0 0 0
- joint left_joint: origin xyz=0 -5 1.5 rpy=0 0 0 -> xyz=0 0 0 rpy=0 0 0
- joint right_joint: origin xyz=0 5 1.5 rpy=0 0 0 -> xyz=0 0 0 rpy=0 0 0

Commit message: fixed hallway shift

File: urdf/random_hall.urdf (robot description, URDF)
Before this commit: robot hallway, 39 links, 38 joints
Links:
- link base: geometry collision box size=51.14 5.51 0.2; visual box size=51.14 5.51 0.2
- link sec_10_left_wall: geometry collision box size=4.89 0.2 3.0; visual box size=4.89 0.2 3.0
- link sec_10_right_wall: geometry collision box size=4.89 0.2 3.0; visual box size=4.89 0.2 3.0
- link sec_1_left_conn: geometry collision box size=0.2 0.505 3.0; visual box size=0.2 0.505 3.0
- link sec_1_left_wall: geometry collision box size=5.29 0.2 3.0; visual box size=5.29 0.2 3.0
- link sec_1_right_conn: geometry collision box size=0.2 0.505 3.0; visual box size=0.2 0.505 3.0
- link sec_1_right_wall: geometry collision box size=5.29 0.2 3.0; visual box size=5.29 0.2 3.0
- link sec_2_left_conn: geometry collision box size=0.2 0.245 3.0; visual box size=0.2 0.245 3.0
- link sec_2_left_wall: geometry collision box size=3.98 0.2 3.0; visual box size=3.98 0.2 3.0
- link sec_2_right_conn: geometry collision box size=0.2 0.245 3.0; visual box size=0.2 0.245 3.0
- link sec_2_right_wall: geometry collision box size=3.98 0.2 3.0; visual box size=3.98 0.2 3.0
- link sec_3_left_conn: geometry collision box size=0.2 0.3 3.0; visual box size=0.2 0.3 3.0
- link sec_3_left_wall: geometry collision box size=6.07 0.2 3.0; visual box size=6.07 0.2 3.0
- link sec_3_right_conn: geometry collision box size=0.2 0.3 3.0; visual box size=0.2 0.3 3.0
- link sec_3_right_wall: geometry collision box size=6.07 0.2 3.0; visual box size=6.07 0.2 3.0
- link sec_4_left_conn: geometry collision box size=0.2 0.945 3.0; visual box size=0.2 0.945 3.0
- link sec_4_left_wall: geometry collision box size=5.82 0.2 3.0; visual box size=5.82 0.2 3.0
- link sec_4_right_conn: geometry collision box size=0.2 0.945 3.0; visual box size=0.2 0.945 3.0
- link sec_4_right_wall: geometry collision box size=5.82 0.2 3.0; visual box size=5.82 0.2 3.0
- link sec_5_left_conn: geometry collision box size=0.2 0.93 3.0; visual box size=0.2 0.93 3.0
- link sec_5_left_wall: geometry collision box size=4.83 0.2 3.0; visual box size=4.83 0.2 3.0
- link sec_5_right_conn: geometry collision box size=0.2 0.93 3.0; visual box size=0.2 0.93 3.0
- link sec_5_right_wall: geometry collision box size=4.83 0.2 3.0; visual box size=4.83 0.2 3.0
- link sec_6_left_conn: geometry collision box size=0.2 0.295 3.0; visual box size=0.2 0.295 3.0
- link sec_6_left_wall: geometry collision box size=3.94 0.2 3.0; visual box size=3.94 0.2 3.0
- link sec_6_right_conn: geometry collision box size=0.2 0.295 3.0; visual box size=0.2 0.295 3.0
- link sec_6_right_wall: geometry collision box size=3.94 0.2 3.0; visual box size=3.94 0.2 3.0
- link sec_7_left_conn: geometry collision box size=0.2 0.73 3.0; visual box size=0.2 0.73 3.0
- link sec_7_left_wall: geometry collision box size=4.56 0.2 3.0; visual box size=4.56 0.2 3.0
- link sec_7_right_conn: geometry collision box size=0.2 0.73 3.0; visual box size=0.2 0.73 3.0
- link sec_7_right_wall: geometry collision box size=4.56 0.2 3.0; visual box size=4.56 0.2 3.0
- link sec_8_left_conn: geometry collision box size=0.2 0.685 3.0; visual box size=0.2 0.685 3.0
- link sec_8_left_wall: geometry collision box size=5.44 0.2 3.0; visual box size=5.44 0.2 3.0
- link sec_8_right_conn: geometry collision box size=0.2 0.685 3.0; visual box size=0.2 0.685 3.0
- link sec_8_right_wall: geometry collision box size=5.44 0.2 3.0; visual box size=5.44 0.2 3.0
- link sec_9_left_conn: geometry collision box size=0.2 0.38 3.0; visual box size=0.2 0.38 3.0
- link sec_9_left_wall: geometry collision box size=6.32 0.2 3.0; visual box size=6.32 0.2 3.0
- link sec_9_right_conn: geometry collision box size=0.2 0.38 3.0; visual box size=0.2 0.38 3.0
- link sec_9_right_wall: geometry collision box size=6.32 0.2 3.0; visual box size=6.32 0.2 3.0

Commit message: add static tag

File: urdf/random_hall.urdf (robot description, URDF)
Before this commit: robot hallway, 39 links, 38 joints
Links:
- link base: geometry collision box size=54.58 5.04 0.2; visual box size=54.58 5.04 0.2
- link sec_10_left_wall: geometry collision box size=5.33 0.2 3.0; visual box size=5.33 0.2 3.0
- link sec_10_right_wall: geometry collision box size=5.33 0.2 3.0; visual box size=5.33 0.2 3.0
- link sec_1_left_conn: geometry collision box size=0.2 0.27 3.0; visual box size=0.2 0.27 3.0
- link sec_1_left_wall: geometry collision box size=6.95 0.2 3.0; visual box size=6.95 0.2 3.0
- link sec_1_right_conn: geometry collision box size=0.2 0.27 3.0; visual box size=0.2 0.27 3.0
- link sec_1_right_wall: geometry collision box size=6.95 0.2 3.0; visual box size=6.95 0.2 3.0
- link sec_2_left_conn: geometry collision box size=0.2 0.62 3.0; visual box size=0.2 0.62 3.0
- link sec_2_left_wall: geometry collision box size=5.98 0.2 3.0; visual box size=5.98 0.2 3.0
- link sec_2_right_conn: geometry collision box size=0.2 0.62 3.0; visual box size=0.2 0.62 3.0
- link sec_2_right_wall: geometry collision box size=5.98 0.2 3.0; visual box size=5.98 0.2 3.0
- link sec_3_left_conn: geometry collision box size=0.2 0.685 3.0; visual box size=0.2 0.685 3.0
- link sec_3_left_wall: geometry collision box size=4.35 0.2 3.0; visual box size=4.35 0.2 3.0
- link sec_3_right_conn: geometry collision box size=0.2 0.685 3.0; visual box size=0.2 0.685 3.0
- link sec_3_right_wall: geometry collision box size=4.35 0.2 3.0; visual box size=4.35 0.2 3.0
- link sec_4_left_conn: geometry collision box size=0.2 0.36 3.0; visual box size=0.2 0.36 3.0
- link sec_4_left_wall: geometry collision box size=5.2 0.2 3.0; visual box size=5.2 0.2 3.0
- link sec_4_right_conn: geometry collision box size=0.2 0.36 3.0; visual box size=0.2 0.36 3.0
- link sec_4_right_wall: geometry collision box size=5.2 0.2 3.0; visual box size=5.2 0.2 3.0
- link sec_5_left_conn: geometry collision box size=0.2 0.305 3.0; visual box size=0.2 0.305 3.0
- link sec_5_left_wall: geometry collision box size=5.03 0.2 3.0; visual box size=5.03 0.2 3.0
- link sec_5_right_conn: geometry collision box size=0.2 0.305 3.0; visual box size=0.2 0.305 3.0
- link sec_5_right_wall: geometry collision box size=5.03 0.2 3.0; visual box size=5.03 0.2 3.0
- link sec_6_left_conn: geometry collision box size=0.2 0.47 3.0; visual box size=0.2 0.47 3.0
- link sec_6_left_wall: geometry collision box size=6.94 0.2 3.0; visual box size=6.94 0.2 3.0
- link sec_6_right_conn: geometry collision box size=0.2 0.47 3.0; visual box size=0.2 0.47 3.0
- link sec_6_right_wall: geometry collision box size=6.94 0.2 3.0; visual box size=6.94 0.2 3.0
- link sec_7_left_conn: geometry collision box size=0.2 0.28 3.0; visual box size=0.2 0.28 3.0
- link sec_7_left_wall: geometry collision box size=4.03 0.2 3.0; visual box size=4.03 0.2 3.0
- link sec_7_right_conn: geometry collision box size=0.2 0.28 3.0; visual box size=0.2 0.28 3.0
- link sec_7_right_wall: geometry collision box size=4.03 0.2 3.0; visual box size=4.03 0.2 3.0
- link sec_8_left_conn: geometry collision box size=0.2 0.215 3.0; visual box size=0.2 0.215 3.0
- link sec_8_left_wall: geometry collision box size=4.42 0.2 3.0; visual box size=4.42 0.2 3.0
- link sec_8_right_conn: geometry collision box size=0.2 0.215 3.0; visual box size=0.2 0.215 3.0
- link sec_8_right_wall: geometry collision box size=4.42 0.2 3.0; visual box size=4.42 0.2 3.0
- link sec_9_left_conn: geometry collision box size=0.2 0.4 3.0; visual box size=0.2 0.4 3.0
- link sec_9_left_wall: geometry collision box size=6.35 0.2 3.0; visual box size=6.35 0.2 3.0
- link sec_9_right_conn: geometry collision box size=0.2 0.4 3.0; visual box size=0.2 0.4 3.0
- link sec_9_right_wall: geometry collision box size=6.35 0.2 3.0; visual box size=6.35 0.2 3.0

Commit message: random hallway generation from launch file!

File: urdf/random_hall.urdf (robot description, URDF)
Before this commit: robot hallway, 39 links, 38 joints
Links:
- link base: geometry collision box size=45.36 5.07 0.2; visual box size=45.36 5.07 0.2
- link sec_10_left_wall: geometry collision box size=3.71 0.2 3.0; visual box size=3.71 0.2 3.0
- link sec_10_right_wall: geometry collision box size=3.71 0.2 3.0; visual box size=3.71 0.2 3.0
- link sec_1_left_conn: geometry collision box size=0.2 0.87 3.0; visual box size=0.2 0.87 3.0
- link sec_1_left_wall: geometry collision box size=4.53 0.2 3.0; visual box size=4.53 0.2 3.0
- link sec_1_right_conn: geometry collision box size=0.2 0.87 3.0; visual box size=0.2 0.87 3.0
- link sec_1_right_wall: geometry collision box size=4.53 0.2 3.0; visual box size=4.53 0.2 3.0
- link sec_2_left_conn: geometry collision box size=0.2 0.5 3.0; visual box size=0.2 0.5 3.0
- link sec_2_left_wall: geometry collision box size=4.36 0.2 3.0; visual box size=4.36 0.2 3.0
- link sec_2_right_conn: geometry collision box size=0.2 0.5 3.0; visual box size=0.2 0.5 3.0
- link sec_2_right_wall: geometry collision box size=4.36 0.2 3.0; visual box size=4.36 0.2 3.0
- link sec_3_left_conn: geometry collision box size=0.2 0.78 3.0; visual box size=0.2 0.78 3.0
- link sec_3_left_wall: geometry collision box size=6.1 0.2 3.0; visual box size=6.1 0.2 3.0
- link sec_3_right_conn: geometry collision box size=0.2 0.78 3.0; visual box size=0.2 0.78 3.0
- link sec_3_right_wall: geometry collision box size=6.1 0.2 3.0; visual box size=6.1 0.2 3.0
- link sec_4_left_conn: geometry collision box size=0.2 1.075 3.0; visual box size=0.2 1.075 3.0
- link sec_4_left_wall: geometry collision box size=3.55 0.2 3.0; visual box size=3.55 0.2 3.0
- link sec_4_right_conn: geometry collision box size=0.2 1.075 3.0; visual box size=0.2 1.075 3.0
- link sec_4_right_wall: geometry collision box size=3.55 0.2 3.0; visual box size=3.55 0.2 3.0
- link sec_5_left_conn: geometry collision box size=0.2 0.26 3.0; visual box size=0.2 0.26 3.0
- link sec_5_left_wall: geometry collision box size=5.51 0.2 3.0; visual box size=5.51 0.2 3.0
- link sec_5_right_conn: geometry collision box size=0.2 0.26 3.0; visual box size=0.2 0.26 3.0
- link sec_5_right_wall: geometry collision box size=5.51 0.2 3.0; visual box size=5.51 0.2 3.0
- link sec_6_left_conn: geometry collision box size=0.2 0.975 3.0; visual box size=0.2 0.975 3.0
- link sec_6_left_wall: geometry collision box size=4.72 0.2 3.0; visual box size=4.72 0.2 3.0
- link sec_6_right_conn: geometry collision box size=0.2 0.975 3.0; visual box size=0.2 0.975 3.0
- link sec_6_right_wall: geometry collision box size=4.72 0.2 3.0; visual box size=4.72 0.2 3.0
- link sec_7_left_conn: geometry collision box size=0.2 0.725 3.0; visual box size=0.2 0.725 3.0
- link sec_7_left_wall: geometry collision box size=4.0 0.2 3.0; visual box size=4.0 0.2 3.0
- link sec_7_right_conn: geometry collision box size=0.2 0.725 3.0; visual box size=0.2 0.725 3.0
- link sec_7_right_wall: geometry collision box size=4.0 0.2 3.0; visual box size=4.0 0.2 3.0
- link sec_8_left_conn: geometry collision box size=0.2 0.52 3.0; visual box size=0.2 0.52 3.0
- link sec_8_left_wall: geometry collision box size=4.19 0.2 3.0; visual box size=4.19 0.2 3.0
- link sec_8_right_conn: geometry collision box size=0.2 0.52 3.0; visual box size=0.2 0.52 3.0
- link sec_8_right_wall: geometry collision box size=4.19 0.2 3.0; visual box size=4.19 0.2 3.0
- link sec_9_left_conn: geometry collision box size=0.2 0.77 3.0; visual box size=0.2 0.77 3.0
- link sec_9_left_wall: geometry collision box size=4.69 0.2 3.0; visual box size=4.69 0.2 3.0
- link sec_9_right_conn: geometry collision box size=0.2 0.77 3.0; visual box size=0.2 0.77 3.0
- link sec_9_right_wall: geometry collision box size=4.69 0.2 3.0; visual box size=4.69 0.2 3.0
