Commit message: added functionality for hallway intersections

File: urdf/random_hall.urdf (robot description, URDF)
Before this commit: robot hallway, 39 links, 38 joints
Links:
- removed link sec_10_left_wall
- removed link sec_10_right_wall
- removed link sec_1_left_conn
- removed link sec_1_left_wall
- removed link sec_1_right_conn
- removed link sec_1_right_wall
- removed link sec_2_left_conn
- removed link sec_2_left_wall
- removed link sec_2_right_conn
- removed link sec_2_right_wall
- removed link sec_3_left_conn
- removed link sec_3_left_wall
- removed link sec_3_right_conn
- removed link sec_3_right_wall
- removed link sec_4_left_conn
- removed link sec_4_left_wall
- removed link sec_4_right_conn
- removed link sec_4_right_wall
- removed link sec_5_left_conn
- removed link sec_5_left_wall
- removed link sec_5_right_conn
- removed link sec_5_right_wall
- removed link sec_6_left_conn
- removed link sec_6_left_wall
- removed link sec_6_right_conn
- removed link sec_6_right_wall
- removed link sec_7_left_conn
- removed link sec_7_left_wall
- removed link sec_7_right_conn
- removed link sec_7_right_wall
- removed link sec_8_left_conn
- removed link sec_8_left_wall
- removed link sec_8_right_conn
- removed link sec_8_right_wall
- removed link sec_9_left_conn
- removed link sec_9_left_wall
- removed link sec_9_right_conn
- removed link sec_9_right_wall
- added link 1_int_side_0; collision box size=0.2 5.9 3.0; visual box size=0.2 5.9 3.0
- added link 1_int_side_1; collision box size=5.9 0.2 3.0; visual box size=5.9 0.2 3.0
- added link 1_int_side_2_left; collision box size=0.2 0.7 3.0; visual box size=0.2 0.7 3.0
- added link 1_int_side_2_right; collision box size=0.2 0.7 3.0; visual box size=0.2 0.7 3.0
- added link 1_int_side_3; collision box size=5.9 0.2 3.0; visual box size=5.9 0.2 3.0
- added link 2_sec_10_left_wall; collision box size=5.0 0.2 3.0; visual box size=5.0 0.2 3.0
- added link 2_sec_10_right_wall; collision box size=5.0 0.2 3.0; visual box size=5.0 0.2 3.0
- added link 2_sec_1_left_conn; collision box size=0.2 0.6 3.0; visual box size=0.2 0.6 3.0
- added link 2_sec_1_left_wall; collision box size=5.0 0.2 3.0; visual box size=5.0 0.2 3.0
- added link 2_sec_1_right_conn; collision box size=0.2 0.6 3.0; visual box size=0.2 0.6 3.0
- added link 2_sec_1_right_wall; collision box size=5.0 0.2 3.0; visual box size=5.0 0.2 3.0
- added link 2_sec_2_left_conn; collision box size=0.2 0.37 3.0; visual box size=0.2 0.37 3.0
- added link 2_sec_2_left_wall; collision box size=6.26 0.2 3.0; visual box size=6.26 0.2 3.0
- added link 2_sec_2_right_conn; collision box size=0.2 0.37 3.0; visual box size=0.2 0.37 3.0
- added link 2_sec_2_right_wall; collision box size=6.26 0.2 3.0; visual box size=6.26 0.2 3.0
- added link 2_sec_3_left_conn; collision box size=0.2 0.305 3.0; visual box size=0.2 0.305 3.0
- added link 2_sec_3_left_wall; collision box size=5.4 0.2 3.0; visual box size=5.4 0.2 3.0
- added link 2_sec_3_right_conn; collision box size=0.2 0.305 3.0; visual box size=0.2 0.305 3.0
- added link 2_sec_3_right_wall; collision box size=5.4 0.2 3.0; visual box size=5.4 0.2 3.0
- added link 2_sec_4_left_conn; collision box size=0.2 0.385 3.0; visual box size=0.2 0.385 3.0
- added link 2_sec_4_left_wall; collision box size=4.53 0.2 3.0; visual box size=4.53 0.2 3.0
- added link 2_sec_4_right_conn; collision box size=0.2 0.385 3.0; visual box size=0.2 0.385 3.0
- added link 2_sec_4_right_wall; collision box size=4.53 0.2 3.0; visual box size=4.53 0.2 3.0
- added link 2_sec_5_left_conn; collision box size=0.2 0.345 3.0; visual box size=0.2 0.345 3.0
- added link 2_sec_5_left_wall; collision box size=6.08 0.2 3.0; visual box size=6.08 0.2 3.0
- added link 2_sec_5_right_conn; collision box size=0.2 0.345 3.0; visual box size=0.2 0.345 3.0
- added link 2_sec_5_right_wall; collision box size=6.08 0.2 3.0; visual box size=6.08 0.2 3.0
- added link 2_sec_6_left_conn; collision box size=0.2 0.465 3.0; visual box size=0.2 0.465 3.0
- added link 2_sec_6_left_wall; collision box size=5.49 0.2 3.0; visual box size=5.49 0.2 3.0
- added link 2_sec_6_right_conn; collision box size=0.2 0.465 3.0; visual box size=0.2 0.465 3.0
- added link 2_sec_6_right_wall; collision box size=5.49 0.2 3.0; visual box size=5.49 0.2 3.0
- added link 2_sec_7_left_conn; collision box size=0.2 0.62 3.0; visual box size=0.2 0.62 3.0
- added link 2_sec_7_left_wall; collision box size=5.46 0.2 3.0; visual box size=5.46 0.2 3.0
- added link 2_sec_7_right_conn; collision box size=0.2 0.62 3.0; visual box size=0.2 0.62 3.0
- added link 2_sec_7_right_wall; collision box size=5.46 0.2 3.0; visual box size=5.46 0.2 3.0
- added link 2_sec_8_left_conn; collision box size=0.2 0.315 3.0; visual box size=0.2 0.315 3.0
- added link 2_sec_8_left_wall; collision box size=5.19 0.2 3.0; visual box size=5.19 0.2 3.0
- added link 2_sec_8_right_conn; collision box size=0.2 0.315 3.0; visual box size=0.2 0.315 3.0
- added link 2_sec_8_right_wall; collision box size=5.19 0.2 3.0; visual box size=5.19 0.2 3.0
- added link 2_sec_9_left_conn; collision box size=0.2 0.265 3.0; visual box size=0.2 0.265 3.0
- added link 2_sec_9_left_wall; collision box size=5.23 0.2 3.0; visual box size=5.23 0.2 3.0
- added link 2_sec_9_right_conn; collision box size=0.2 0.265 3.0; visual box size=0.2 0.265 3.0
- added link 2_sec_9_right_wall; collision box size=5.23 0.2 3.0; visual box size=5.23 0.2 3.0
- added link 3_int_side_0_left; collision box size=0.2 0.7 3.0; visual box size=0.2 0.7 3.0
- added link 3_int_side_0_right; collision box size=0.2 0.7 3.0; visual box size=0.2 0.7 3.0
- added link 3_int_side_1_left; collision box size=0.7 0.2 3.0; visual box size=0.7 0.2 3.0
- added link 3_int_side_1_right; collision box size=0.7 0.2 3.0; visual box size=0.7 0.2 3.0
- added link 3_int_side_2; collision box size=0.2 5.9 3.0; visual box size=0.2 5.9 3.0
- added link 3_int_side_3_left; collision box size=0.7 0.2 3.0; visual box size=0.7 0.2 3.0
- added link 3_int_side_3_right; collision box size=0.7 0.2 3.0; visual box size=0.7 0.2 3.0
- added link 4_sec_10_left_wall; collision box size=0.2 5.0 3.0; visual box size=0.2 5.0 3.0
- added link 4_sec_10_right_wall; collision box size=0.2 5.0 3.0; visual box size=0.2 5.0 3.0
- added link 4_sec_1_left_conn; collision box size=0.65 0.2 3.0; visual box size=0.65 0.2 3.0
- added link 4_sec_1_left_wall; collision box size=0.2 5.0 3.0; visual box size=0.2 5.0 3.0
- added link 4_sec_1_right_conn; collision box size=0.65 0.2 3.0; visual box size=0.65 0.2 3.0
- added link 4_sec_1_right_wall; collision box size=0.2 5.0 3.0; visual box size=0.2 5.0 3.0
- added link 4_sec_2_left_conn; collision box size=0.7 0.2 3.0; visual box size=0.7 0.2 3.0
- added link 4_sec_2_left_wall; collision box size=0.2 5.43 3.0; visual box size=0.2 5.43 3.0
- added link 4_sec_2_right_conn; collision box size=0.7 0.2 3.0; visual box size=0.7 0.2 3.0
- added link 4_sec_2_right_wall; collision box size=0.2 5.43 3.0; visual box size=0.2 5.43 3.0
- added link 4_sec_3_left_conn; collision box size=0.43 0.2 3.0; visual box size=0.43 0.2 3.0
- added link 4_sec_3_left_wall; collision box size=0.2 4.11 3.0; visual box size=0.2 4.11 3.0
- added link 4_sec_3_right_conn; collision box size=0.43 0.2 3.0; visual box size=0.43 0.2 3.0
- added link 4_sec_3_right_wall; collision box size=0.2 4.11 3.0; visual box size=0.2 4.11 3.0
- added link 4_sec_4_left_conn; collision box size=0.78 0.2 3.0; visual box size=0.78 0.2 3.0
- added link 4_sec_4_left_wall; collision box size=0.2 4.76 3.0; visual box size=0.2 4.76 3.0
- added link 4_sec_4_right_conn; collision box size=0.78 0.2 3.0; visual box size=0.78 0.2 3.0
- added link 4_sec_4_right_wall; collision box size=0.2 4.76 3.0; visual box size=0.2 4.76 3.0
- added link 4_sec_5_left_conn; collision box size=0.45 0.2 3.0; visual box size=0.45 0.2 3.0
- added link 4_sec_5_left_wall; collision box size=0.2 3.73 3.0; visual box size=0.2 3.73 3.0
- added link 4_sec_5_right_conn; collision box size=0.45 0.2 3.0; visual box size=0.45 0.2 3.0
- added link 4_sec_5_right_wall; collision box size=0.2 3.73 3.0; visual box size=0.2 3.73 3.0
- added link 4_sec_6_left_conn; collision box size=0.4 0.2 3.0; visual box size=0.4 0.2 3.0
- added link 4_sec_6_left_wall; collision box size=0.2 5.79 3.0; visual box size=0.2 5.79 3.0
- added link 4_sec_6_right_conn; collision box size=0.4 0.2 3.0; visual box size=0.4 0.2 3.0
- added link 4_sec_6_right_wall; collision box size=0.2 5.79 3.0; visual box size=0.2 5.79 3.0
- added link 4_sec_7_left_conn; collision box size=0.22 0.2 3.0; visual box size=0.22 0.2 3.0
- added link 4_sec_7_left_wall; collision box size=0.2 2.24 3.0; visual box size=0.2 2.24 3.0
- added link 4_sec_7_right_conn; collision box size=0.22 0.2 3.0; visual box size=0.22 0.2 3.0
- added link 4_sec_7_right_wall; collision box size=0.2 2.24 3.0; visual box size=0.2 2.24 3.0
- added link 4_sec_8_left_conn; collision box size=0.415 0.2 3.0; visual box size=0.415 0.2 3.0
- added link 4_sec_8_left_wall; collision box size=0.2 5.25 3.0; visual box size=0.2 5.25 3.0
- added link 4_sec_8_right_conn; collision box size=0.415 0.2 3.0; visual box size=0.415 0.2 3.0
- added link 4_sec_8_right_wall; collision box size=0.2 5.25 3.0; visual box size=0.2 5.25 3.0
- added link 4_sec_9_left_conn; collision box size=0.615 0.2 3.0; visual box size=0.615 0.2 3.0
- added link 4_sec_9_left_wall; collision box size=0.2 3.29 3.0; visual box size=0.2 3.29 3.0
- added link 4_sec_9_right_conn; collision box size=0.615 0.2 3.0; visual box size=0.615 0.2 3.0
- added link 4_sec_9_right_wall; collision box size=0.2 3.29 3.0; visual box size=0.2 3.29 3.0
- link base: mass 50 -> 50,0; geometry collision box size=119.08 101.0 0.2; visual box size=119.08 101.0 0.2
Joints:
- removed joint joint_sec_10_left_wall
- removed joint joint_sec_10_right_wall
- removed joint joint_sec_1_left_conn
- removed joint joint_sec_1_left_wall
- removed joint joint_sec_1_right_conn
- removed joint joint_sec_1_right_wall
- removed joint joint_sec_2_left_conn
- removed joint joint_sec_2_left_wall
- removed joint joint_sec_2_right_conn
- removed joint joint_sec_2_right_wall
- removed joint joint_sec_3_left_conn
- removed joint joint_sec_3_left_wall
- removed joint joint_sec_3_right_conn
- removed joint joint_sec_3_right_wall
- removed joint joint_sec_4_left_conn
- removed joint joint_sec_4_left_wall
- removed joint joint_sec_4_right_conn
- removed joint joint_sec_4_right_wall
- removed joint joint_sec_5_left_conn
- removed joint joint_sec_5_left_wall
- removed joint joint_sec_5_right_conn
- removed joint joint_sec_5_right_wall
- removed joint joint_sec_6_left_conn
- removed joint joint_sec_6_left_wall
- removed joint joint_sec_6_right_conn
- removed joint joint_sec_6_right_wall
- removed joint joint_sec_7_left_conn
- removed joint joint_sec_7_left_wall
- removed joint joint_sec_7_right_conn
- removed joint joint_sec_7_right_wall
- removed joint joint_sec_8_left_conn
- removed joint joint_sec_8_left_wall
- removed joint joint_sec_8_right_conn
- removed joint joint_sec_8_right_wall
- removed joint joint_sec_9_left_conn
- removed joint joint_sec_9_left_wall
- removed joint joint_sec_9_right_conn
- removed joint joint_sec_9_right_wall
- added joint joint_1_int_side_0: type fixed, parent base, child 1_int_side_0, origin xyz=0 0 0 rpy=0 0 0
- added joint joint_1_int_side_1: type fixed, parent base, child 1_int_side_1, origin xyz=0 0 0 rpy=0 0 0
- added joint joint_1_int_side_2_left: type fixed, parent base, child 1_int_side_2_left, origin xyz=0 0 0 rpy=0 0 0
- added joint joint_1_int_side_2_right: type fixed, parent base, child 1_int_side_2_right, origin xyz=0 0 0 rpy=0 0 0
- added joint joint_1_int_side_3: type fixed, parent base, child 1_int_side_3, origin xyz=0 0 0 rpy=0 0 0
- added joint joint_2_sec_10_left_wall: type fixed, parent base, child 2_sec_10_left_wall, origin xyz=0 0 0 rpy=0 0 0
- added joint joint_2_sec_10_right_wall: type fixed, parent base, child 2_sec_10_right_wall, origin xyz=0 0 0 rpy=0 0 0
- added joint joint_2_sec_1_left_conn: type fixed, parent base, child 2_sec_1_left_conn, origin xyz=0 0 0 rpy=0 0 0
- added joint joint_2_sec_1_left_wall: type fixed, parent base, child 2_sec_1_left_wall, origin xyz=0 0 0 rpy=0 0 0
- added joint joint_2_sec_1_right_conn: type fixed, parent base, child 2_sec_1_right_conn, origin xyz=0 0 0 rpy=0 0 0
- added joint joint_2_sec_1_right_wall: type fixed, parent base, child 2_sec_1_right_wall, origin xyz=0 0 0 rpy=0 0 0
- added joint joint_2_sec_2_left_conn: type fixed, parent base, child 2_sec_2_left_conn, origin xyz=0 0 0 rpy=0 0 0
- added joint joint_2_sec_2_left_wall: type fixed, parent base, child 2_sec_2_left_wall, origin xyz=0 0 0 rpy=0 0 0
- added joint joint_2_sec_2_right_conn: type fixed, parent base, child 2_sec_2_right_conn, origin xyz=0 0 0 rpy=0 0 0
- added joint joint_2_sec_2_right_wall: type fixed, parent base, child 2_sec_2_right_wall, origin xyz=0 0 0 rpy=0 0 0
- added joint joint_2_sec_3_left_conn: type fixed, parent base, child 2_sec_3_left_conn, origin xyz=0 0 0 rpy=0 0 0
- added joint joint_2_sec_3_left_wall: type fixed, parent base, child 2_sec_3_left_wall, origin xyz=0 0 0 rpy=0 0 0
- added joint joint_2_sec_3_right_conn: type fixed, parent base, child 2_sec_3_right_conn, origin xyz=0 0 0 rpy=0 0 0
- added joint joint_2_sec_3_right_wall: type fixed, parent base, child 2_sec_3_right_wall, origin xyz=0 0 0 rpy=0 0 0
- added joint joint_2_sec_4_left_conn: type fixed, parent base, child 2_sec_4_left_conn, origin xyz=0 0 0 rpy=0 0 0
- added joint joint_2_sec_4_left_wall: type fixed, parent base, child 2_sec_4_left_wall, origin xyz=0 0 0 rpy=0 0 0
- added joint joint_2_sec_4_right_conn: type fixed, parent base, child 2_sec_4_right_conn, origin xyz=0 0 0 rpy=0 0 0
- added joint joint_2_sec_4_right_wall: type fixed, parent base, child 2_sec_4_right_wall, origin xyz=0 0 0 rpy=0 0 0
- added joint joint_2_sec_5_left_conn: type fixed, parent base, child 2_sec_5_left_conn, origin xyz=0 0 0 rpy=0 0 0
- added joint joint_2_sec_5_left_wall: type fixed, parent base, child 2_sec_5_left_wall, origin xyz=0 0 0 rpy=0 0 0
- added joint joint_2_sec_5_right_conn: type fixed, parent base, child 2_sec_5_right_conn, origin xyz=0 0 0 rpy=0 0 0
- added joint joint_2_sec_5_right_wall: type fixed, parent base, child 2_sec_5_right_wall, origin xyz=0 0 0 rpy=0 0 0
- added joint joint_2_sec_6_left_conn: type fixed, parent base, child 2_sec_6_left_conn, origin xyz=0 0 0 rpy=0 0 0
- added joint joint_2_sec_6_left_wall: type fixed, parent base, child 2_sec_6_left_wall, origin xyz=0 0 0 rpy=0 0 0
- added joint joint_2_sec_6_right_conn: type fixed, parent base, child 2_sec_6_right_conn, origin xyz=0 0 0 rpy=0 0 0
- added joint joint_2_sec_6_right_wall: type fixed, parent base, child 2_sec_6_right_wall, origin xyz=0 0 0 rpy=0 0 0
- added joint joint_2_sec_7_left_conn: type fixed, parent base, child 2_sec_7_left_conn, origin xyz=0 0 0 rpy=0 0 0
- added joint joint_2_sec_7_left_wall: type fixed, parent base, child 2_sec_7_left_wall, origin xyz=0 0 0 rpy=0 0 0
- added joint joint_2_sec_7_right_conn: type fixed, parent base, child 2_sec_7_right_conn, origin xyz=0 0 0 rpy=0 0 0
- added joint joint_2_sec_7_right_wall: type fixed, parent base, child 2_sec_7_right_wall, origin xyz=0 0 0 rpy=0 0 0
- added joint joint_2_sec_8_left_conn: type fixed, parent base, child 2_sec_8_left_conn, origin xyz=0 0 0 rpy=0 0 0
- added joint joint_2_sec_8_left_wall: type fixed, parent base, child 2_sec_8_left_wall, origin xyz=0 0 0 rpy=0 0 0
- added joint joint_2_sec_8_right_conn: type fixed, parent base, child 2_sec_8_right_conn, origin xyz=0 0 0 rpy=0 0 0
- added joint joint_2_sec_8_right_wall: type fixed, parent base, child 2_sec_8_right_wall, origin xyz=0 0 0 rpy=0 0 0
- added joint joint_2_sec_9_left_conn: type fixed, parent base, child 2_sec_9_left_conn, origin xyz=0 0 0 rpy=0 0 0
- added joint joint_2_sec_9_left_wall: type fixed, parent base, child 2_sec_9_left_wall, origin xyz=0 0 0 rpy=0 0 0
- added joint joint_2_sec_9_right_conn: type fixed, parent base, child 2_sec_9_right_conn, origin xyz=0 0 0 rpy=0 0 0
- added joint joint_2_sec_9_right_wall: type fixed, parent base, child 2_sec_9_right_wall, origin xyz=0 0 0 rpy=0 0 0
- added joint joint_3_int_side_0_left: type fixed, parent base, child 3_int_side_0_left, origin xyz=0 0 0 rpy=0 0 0
- added joint joint_3_int_side_0_right: type fixed, parent base, child 3_int_side_0_right, origin xyz=0 0 0 rpy=0 0 0
- added joint joint_3_int_side_1_left: type fixed, parent base, child 3_int_side_1_left, origin xyz=0 0 0 rpy=0 0 0
- added joint joint_3_int_side_1_right: type fixed, parent base, child 3_int_side_1_right, origin xyz=0 0 0 rpy=0 0 0
- added joint joint_3_int_side_2: type fixed, parent base, child 3_int_side_2, origin xyz=0 0 0 rpy=0 0 0
- added joint joint_3_int_side_3_left: type fixed, parent base, child 3_int_side_3_left, origin xyz=0 0 0 rpy=0 0 0
- added joint joint_3_int_side_3_right: type fixed, parent base, child 3_int_side_3_right, origin xyz=0 0 0 rpy=0 0 0
- added joint joint_4_sec_10_left_wall: type fixed, parent base, child 4_sec_10_left_wall, origin xyz=0 0 0 rpy=0 0 0
- added joint joint_4_sec_10_right_wall: type fixed, parent base, child 4_sec_10_right_wall, origin xyz=0 0 0 rpy=0 0 0
- added joint joint_4_sec_1_left_conn: type fixed, parent base, child 4_sec_1_left_conn, origin xyz=0 0 0 rpy=0 0 0
- added joint joint_4_sec_1_left_wall: type fixed, parent base, child 4_sec_1_left_wall, origin xyz=0 0 0 rpy=0 0 0
- added joint joint_4_sec_1_right_conn: type fixed, parent base, child 4_sec_1_right_conn, origin xyz=0 0 0 rpy=0 0 0
- added joint joint_4_sec_1_right_wall: type fixed, parent base, child 4_sec_1_right_wall, origin xyz=0 0 0 rpy=0 0 0
- added joint joint_4_sec_2_left_conn: type fixed, parent base, child 4_sec_2_left_conn, origin xyz=0 0 0 rpy=0 0 0
- added joint joint_4_sec_2_left_wall: type fixed, parent base, child 4_sec_2_left_wall, origin xyz=0 0 0 rpy=0 0 0
- added joint joint_4_sec_2_right_conn: type fixed, parent base, child 4_sec_2_right_conn, origin xyz=0 0 0 rpy=0 0 0
- added joint joint_4_sec_2_right_wall: type fixed, parent base, child 4_sec_2_right_wall, origin xyz=0 0 0 rpy=0 0 0
- added joint joint_4_sec_3_left_conn: type fixed, parent base, child 4_sec_3_left_conn, origin xyz=0 0 0 rpy=0 0 0
- added joint joint_4_sec_3_left_wall: type fixed, parent base, child 4_sec_3_left_wall, origin xyz=0 0 0 rpy=0 0 0
- added joint joint_4_sec_3_right_conn: type fixed, parent base, child 4_sec_3_right_conn, origin xyz=0 0 0 rpy=0 0 0
- added joint joint_4_sec_3_right_wall: type fixed, parent base, child 4_sec_3_right_wall, origin xyz=0 0 0 rpy=0 0 0
- added joint joint_4_sec_4_left_conn: type fixed, parent base, child 4_sec_4_left_conn, origin xyz=0 0 0 rpy=0 0 0
- added joint joint_4_sec_4_left_wall: type fixed, parent base, child 4_sec_4_left_wall, origin xyz=0 0 0 rpy=0 0 0
- added joint joint_4_sec_4_right_conn: type fixed, parent base, child 4_sec_4_right_conn, origin xyz=0 0 0 rpy=0 0 0
- added joint joint_4_sec_4_right_wall: type fixed, parent base, child 4_sec_4_right_wall, origin xyz=0 0 0 rpy=0 0 0
- added joint joint_4_sec_5_left_conn: type fixed, parent base, child 4_sec_5_left_conn, origin xyz=0 0 0 rpy=0 0 0
- added joint joint_4_sec_5_left_wall: type fixed, parent base, child 4_sec_5_left_wall, origin xyz=0 0 0 rpy=0 0 0
- added joint joint_4_sec_5_right_conn: type fixed, parent base, child 4_sec_5_right_conn, origin xyz=0 0 0 rpy=0 0 0
- added joint joint_4_sec_5_right_wall: type fixed, parent base, child 4_sec_5_right_wall, origin xyz=0 0 0 rpy=0 0 0
- added joint joint_4_sec_6_left_conn: type fixed, parent base, child 4_sec_6_left_conn, origin xyz=0 0 0 rpy=0 0 0
- added joint joint_4_sec_6_left_wall: type fixed, parent base, child 4_sec_6_left_wall, origin xyz=0 0 0 rpy=0 0 0
- added joint joint_4_sec_6_right_conn: type fixed, parent base, child 4_sec_6_right_conn, origin xyz=0 0 0 rpy=0 0 0
- added joint joint_4_sec_6_right_wall: type fixed, parent base, child 4_sec_6_right_wall, origin xyz=0 0 0 rpy=0 0 0
- added joint joint_4_sec_7_left_conn: type fixed, parent base, child 4_sec_7_left_conn, origin xyz=0 0 0 rpy=0 0 0
- added joint joint_4_sec_7_left_wall: type fixed, parent base, child 4_sec_7_left_wall, origin xyz=0 0 0 rpy=0 0 0
- added joint joint_4_sec_7_right_conn: type fixed, parent base, child 4_sec_7_right_conn, origin xyz=0 0 0 rpy=0 0 0
- added joint joint_4_sec_7_right_wall: type fixed, parent base, child 4_sec_7_right_wall, origin xyz=0 0 0 rpy=0 0 0
- added joint joint_4_sec_8_left_conn: type fixed, parent base, child 4_sec_8_left_conn, origin xyz=0 0 0 rpy=0 0 0
- added joint joint_4_sec_8_left_wall: type fixed, parent base, child 4_sec_8_left_wall, origin xyz=0 0 0 rpy=0 0 0
- added joint joint_4_sec_8_right_conn: type fixed, parent base, child 4_sec_8_right_conn, origin xyz=0 0 0 rpy=0 0 0
- added joint joint_4_sec_8_right_wall: type fixed, parent base, child 4_sec_8_right_wall, origin xyz=0 0 0 rpy=0 0 0
- added joint joint_4_sec_9_left_conn: type fixed, parent base, child 4_sec_9_left_conn, origin xyz=0 0 0 rpy=0 0 0
- added joint joint_4_sec_9_left_wall: type fixed, parent base, child 4_sec_9_left_wall, origin xyz=0 0 0 rpy=0 0 0
- added joint joint_4_sec_9_right_conn: type fixed, parent base, child 4_sec_9_right_conn, origin xyz=0 0 0 rpy=0 0 0
- added joint joint_4_sec_9_right_wall: type fixed, parent base, child 4_sec_9_right_wall, origin xyz=0 0 0 rpy=0 0 0
