Commit message: simulation fixes

File: urdf/random_hall.urdf (robot description, URDF)
Before this commit: robot hallway, 89 links, 88 joints
Links:
- link 2_sec_1_left_conn: geometry collision box size=0.2 1.115 3.0; visual box size=0.2 1.115 3.0
- link 2_sec_1_right_conn: geometry collision box size=0.2 1.115 3.0; visual box size=0.2 1.115 3.0
- link 2_sec_2_left_conn: geometry collision box size=0.2 0.515 3.0; visual box size=0.2 0.515 3.0
- link 2_sec_2_left_wall: geometry collision box size=5.22 0.2 3.0; visual box size=5.22 0.2 3.0
- link 2_sec_2_right_conn: geometry collision box size=0.2 0.515 3.0; visual box size=0.2 0.515 3.0
- link 2_sec_2_right_wall: geometry collision box size=5.22 0.2 3.0; visual box size=5.22 0.2 3.0
- link 2_sec_3_left_conn: geometry collision box size=0.2 0.45 3.0; visual box size=0.2 0.45 3.0
- link 2_sec_3_left_wall: geometry collision box size=3.56 0.2 3.0; visual box size=3.56 0.2 3.0
- link 2_sec_3_right_conn: geometry collision box size=0.2 0.45 3.0; visual box size=0.2 0.45 3.0
- link 2_sec_3_right_wall: geometry collision box size=3.56 0.2 3.0; visual box size=3.56 0.2 3.0
- link 2_sec_4_left_conn: geometry collision box size=0.2 0.665 3.0; visual box size=0.2 0.665 3.0
- link 2_sec_4_left_wall: geometry collision box size=3.88 0.2 3.0; visual box size=3.88 0.2 3.0
- link 2_sec_4_right_conn: geometry collision box size=0.2 0.665 3.0; visual box size=0.2 0.665 3.0
- link 2_sec_4_right_wall: geometry collision box size=3.88 0.2 3.0; visual box size=3.88 0.2 3.0
- link 2_sec_5_left_conn: geometry collision box size=0.2 0.395 3.0; visual box size=0.2 0.395 3.0
- link 2_sec_5_left_wall: geometry collision box size=4.06 0.2 3.0; visual box size=4.06 0.2 3.0
- link 2_sec_5_right_conn: geometry collision box size=0.2 0.395 3.0; visual box size=0.2 0.395 3.0
- link 2_sec_5_right_wall: geometry collision box size=4.06 0.2 3.0; visual box size=4.06 0.2 3.0
- link 2_sec_6_left_conn: geometry collision box size=0.2 0.275 3.0; visual box size=0.2 0.275 3.0
- link 2_sec_6_left_wall: geometry collision box size=6.23 0.2 3.0; visual box size=6.23 0.2 3.0
- link 2_sec_6_right_conn: geometry collision box size=0.2 0.275 3.0; visual box size=0.2 0.275 3.0
- link 2_sec_6_right_wall: geometry collision box size=6.23 0.2 3.0; visual box size=6.23 0.2 3.0
- link 2_sec_7_left_conn: geometry collision box size=0.2 0.285 3.0; visual box size=0.2 0.285 3.0
- link 2_sec_7_left_wall: geometry collision box size=4.48 0.2 3.0; visual box size=4.48 0.2 3.0
- link 2_sec_7_right_conn: geometry collision box size=0.2 0.285 3.0; visual box size=0.2 0.285 3.0
- link 2_sec_7_right_wall: geometry collision box size=4.48 0.2 3.0; visual box size=4.48 0.2 3.0
- link 2_sec_8_left_conn: geometry collision box size=0.2 0.34 3.0; visual box size=0.2 0.34 3.0
- link 2_sec_8_left_wall: geometry collision box size=4.75 0.2 3.0; visual box size=4.75 0.2 3.0
- link 2_sec_8_right_conn: geometry collision box size=0.2 0.34 3.0; visual box size=0.2 0.34 3.0
- link 2_sec_8_right_wall: geometry collision box size=4.75 0.2 3.0; visual box size=4.75 0.2 3.0
- link 2_sec_9_left_conn: geometry collision box size=0.2 0.93 3.0; visual box size=0.2 0.93 3.0
- link 2_sec_9_left_wall: geometry collision box size=6.4 0.2 3.0; visual box size=6.4 0.2 3.0
- link 2_sec_9_right_conn: geometry collision box size=0.2 0.93 3.0; visual box size=0.2 0.93 3.0
- link 2_sec_9_right_wall: geometry collision box size=6.4 0.2 3.0; visual box size=6.4 0.2 3.0
- link 4_sec_1_left_conn: geometry collision box size=0.815 0.2 3.0; visual box size=0.815 0.2 3.0
- link 4_sec_1_right_conn: geometry collision box size=0.815 0.2 3.0; visual box size=0.815 0.2 3.0
- link 4_sec_2_left_conn: geometry collision box size=0.235 0.2 3.0; visual box size=0.235 0.2 3.0
- link 4_sec_2_left_wall: geometry collision box size=0.2 5.01 3.0; visual box size=0.2 5.01 3.0
- link 4_sec_2_right_conn: geometry collision box size=0.235 0.2 3.0; visual box size=0.235 0.2 3.0
- link 4_sec_2_right_wall: geometry collision box size=0.2 5.01 3.0; visual box size=0.2 5.01 3.0
- link 4_sec_3_left_conn: geometry collision box size=0.375 0.2 3.0; visual box size=0.375 0.2 3.0
- link 4_sec_3_left_wall: geometry collision box size=0.2 4.26 3.0; visual box size=0.2 4.26 3.0
- link 4_sec_3_right_conn: geometry collision box size=0.375 0.2 3.0; visual box size=0.375 0.2 3.0
- link 4_sec_3_right_wall: geometry collision box size=0.2 4.26 3.0; visual box size=0.2 4.26 3.0
- link 4_sec_4_left_conn: geometry collision box size=0.72 0.2 3.0; visual box size=0.72 0.2 3.0
- link 4_sec_4_left_wall: geometry collision box size=0.2 7.53 3.0; visual box size=0.2 7.53 3.0
- link 4_sec_4_right_conn: geometry collision box size=0.72 0.2 3.0; visual box size=0.72 0.2 3.0
- link 4_sec_4_right_wall: geometry collision box size=0.2 7.53 3.0; visual box size=0.2 7.53 3.0
- link 4_sec_5_left_wall: geometry collision box size=0.2 5.88 3.0; visual box size=0.2 5.88 3.0
- link 4_sec_5_right_wall: geometry collision box size=0.2 5.88 3.0; visual box size=0.2 5.88 3.0
- link 4_sec_6_left_conn: geometry collision box size=0.305 0.2 3.0; visual box size=0.305 0.2 3.0
- link 4_sec_6_left_wall: geometry collision box size=0.2 5.27 3.0; visual box size=0.2 5.27 3.0
- link 4_sec_6_right_conn: geometry collision box size=0.305 0.2 3.0; visual box size=0.305 0.2 3.0
- link 4_sec_6_right_wall: geometry collision box size=0.2 5.27 3.0; visual box size=0.2 5.27 3.0
- link 4_sec_7_left_conn: geometry collision box size=0.28 0.2 3.0; visual box size=0.28 0.2 3.0
- link 4_sec_7_left_wall: geometry collision box size=0.2 3.5 3.0; visual box size=0.2 3.5 3.0
- link 4_sec_7_right_conn: geometry collision box size=0.28 0.2 3.0; visual box size=0.28 0.2 3.0
- link 4_sec_7_right_wall: geometry collision box size=0.2 3.5 3.0; visual box size=0.2 3.5 3.0
- link 4_sec_8_left_conn: geometry collision box size=0.595 0.2 3.0; visual box size=0.595 0.2 3.0
- link 4_sec_8_left_wall: geometry collision box size=0.2 4.6 3.0; visual box size=0.2 4.6 3.0
- link 4_sec_8_right_conn: geometry collision box size=0.595 0.2 3.0; visual box size=0.595 0.2 3.0
- link 4_sec_8_right_wall: geometry collision box size=0.2 4.6 3.0; visual box size=0.2 4.6 3.0
- link 4_sec_9_left_conn: geometry collision box size=1.055 0.2 3.0; visual box size=1.055 0.2 3.0
- link 4_sec_9_left_wall: geometry collision box size=0.2 5.5 3.0; visual box size=0.2 5.5 3.0
- link 4_sec_9_right_conn: geometry collision box size=1.055 0.2 3.0; visual box size=1.055 0.2 3.0
- link 4_sec_9_right_wall: geometry collision box size=0.2 5.5 3.0; visual box size=0.2 5.5 3.0
- link base: mass 50,0 -> 50.0; geometry collision box size=108.96 114.9 0.2; visual box size=108.96 114.9 0.2

Commit message: fixed symmetry issues from simulation

File: urdf/random_hall.urdf (robot description, URDF)
Before this commit: robot hallway, 89 links, 88 joints
Links:
- removed link 2_sec_10_left_wall
- removed link 2_sec_10_right_wall
- removed link 2_sec_5_left_conn
- removed link 2_sec_5_right_conn
- removed link 2_sec_6_left_conn
- removed link 2_sec_6_left_wall
- removed link 2_sec_6_right_conn
- removed link 2_sec_6_right_wall
- removed link 2_sec_7_left_conn
- removed link 2_sec_7_left_wall
- removed link 2_sec_7_right_conn
- removed link 2_sec_7_right_wall
- removed link 2_sec_8_left_conn
- removed link 2_sec_8_left_wall
- removed link 2_sec_8_right_conn
- removed link 2_sec_8_right_wall
- removed link 2_sec_9_left_conn
- removed link 2_sec_9_left_wall
- removed link 2_sec_9_right_conn
- removed link 2_sec_9_right_wall
- removed link 3_int_side_2
- removed link 3_int_side_3_left
- removed link 3_int_side_3_right
- removed link 4_sec_10_left_wall
- removed link 4_sec_10_right_wall
- removed link 4_sec_5_left_conn
- removed link 4_sec_5_right_conn
- removed link 4_sec_6_left_conn
- removed link 4_sec_6_left_wall
- removed link 4_sec_6_right_conn
- removed link 4_sec_6_right_wall
- removed link 4_sec_7_left_conn
- removed link 4_sec_7_left_wall
- removed link 4_sec_7_right_conn
- removed link 4_sec_7_right_wall
- removed link 4_sec_8_left_conn
- removed link 4_sec_8_left_wall
- removed link 4_sec_8_right_conn
- removed link 4_sec_8_right_wall
- removed link 4_sec_9_left_conn
- removed link 4_sec_9_left_wall
- removed link 4_sec_9_right_conn
- removed link 4_sec_9_right_wall
- added link 3_int_side_2_left; collision box size=0.2 0.7 3.0; visual box size=0.2 0.7 3.0
- added link 3_int_side_2_right; collision box size=0.2 0.7 3.0; visual box size=0.2 0.7 3.0
- added link 3_int_side_3; collision box size=5.9 0.2 3.0; visual box size=5.9 0.2 3.0
- link 2_sec_1_left_conn: geometry collision box size=0.2 0.88 3.0; visual box size=0.2 0.88 3.0
- link 2_sec_1_right_conn: geometry collision box size=0.2 0.88 3.0; visual box size=0.2 0.88 3.0
- link 2_sec_2_left_conn: geometry collision box size=0.2 0.72 3.0; visual box size=0.2 0.72 3.0
- link 2_sec_2_left_wall: geometry collision box size=4.57 0.2 3.0; visual box size=4.57 0.2 3.0
- link 2_sec_2_right_conn: geometry collision box size=0.2 0.72 3.0; visual box size=0.2 0.72 3.0
- link 2_sec_2_right_wall: geometry collision box size=4.57 0.2 3.0; visual box size=4.57 0.2 3.0
- link 2_sec_3_left_conn: geometry collision box size=0.2 0.44 3.0; visual box size=0.2 0.44 3.0
- link 2_sec_3_left_wall: geometry collision box size=5.67 0.2 3.0; visual box size=5.67 0.2 3.0
- link 2_sec_3_right_conn: geometry collision box size=0.2 0.44 3.0; visual box size=0.2 0.44 3.0
- link 2_sec_3_right_wall: geometry collision box size=5.67 0.2 3.0; visual box size=5.67 0.2 3.0
- link 2_sec_4_left_conn: geometry collision box size=0.2 0.6 3.0; visual box size=0.2 0.6 3.0
- link 2_sec_4_left_wall: geometry collision box size=3.69 0.2 3.0; visual box size=3.69 0.2 3.0
- link 2_sec_4_right_conn: geometry collision box size=0.2 0.6 3.0; visual box size=0.2 0.6 3.0
- link 2_sec_4_right_wall: geometry collision box size=3.69 0.2 3.0; visual box size=3.69 0.2 3.0
- link 2_sec_5_left_wall: geometry collision box size=5.0 0.2 3.0; visual box size=5.0 0.2 3.0
- link 2_sec_5_right_wall: geometry collision box size=5.0 0.2 3.0; visual box size=5.0 0.2 3.0
- link 4_sec_1_left_conn: geometry collision box size=0.565 0.2 3.0; visual box size=0.565 0.2 3.0
- link 4_sec_1_right_conn: geometry collision box size=0.565 0.2 3.0; visual box size=0.565 0.2 3.0
- link 4_sec_2_left_conn: geometry collision box size=0.65 0.2 3.0; visual box size=0.65 0.2 3.0
- link 4_sec_2_left_wall: geometry collision box size=0.2 5.94 3.0; visual box size=0.2 5.94 3.0
- link 4_sec_2_right_conn: geometry collision box size=0.65 0.2 3.0; visual box size=0.65 0.2 3.0
- link 4_sec_2_right_wall: geometry collision box size=0.2 5.94 3.0; visual box size=0.2 5.94 3.0
- link 4_sec_3_left_conn: geometry collision box size=0.705 0.2 3.0; visual box size=0.705 0.2 3.0
- link 4_sec_3_left_wall: geometry collision box size=0.2 5.31 3.0; visual box size=0.2 5.31 3.0
- link 4_sec_3_right_conn: geometry collision box size=0.705 0.2 3.0; visual box size=0.705 0.2 3.0
- link 4_sec_3_right_wall: geometry collision box size=0.2 5.31 3.0; visual box size=0.2 5.31 3.0
- link 4_sec_4_left_conn: geometry collision box size=0.51 0.2 3.0; visual box size=0.51 0.2 3.0
- link 4_sec_4_left_wall: geometry collision box size=0.2 3.92 3.0; visual box size=0.2 3.92 3.0
- link 4_sec_4_right_conn: geometry collision box size=0.51 0.2 3.0; visual box size=0.51 0.2 3.0
- link 4_sec_4_right_wall: geometry collision box size=0.2 3.92 3.0; visual box size=0.2 3.92 3.0
- link 4_sec_5_left_wall: geometry collision box size=0.2 5.0 3.0; visual box size=0.2 5.0 3.0
- link 4_sec_5_right_wall: geometry collision box size=0.2 5.0 3.0; visual box size=0.2 5.0 3.0
- link base: geometry collision box size=59.66 62.14 0.2; visual box size=59.66 62.14 0.2
Joints:
- removed joint joint_2_sec_10_left_wall
- removed joint joint_2_sec_10_right_wall
- removed joint joint_2_sec_5_left_conn
- removed joint joint_2_sec_5_right_conn
- removed joint joint_2_sec_6_left_conn
- removed joint joint_2_sec_6_left_wall
- removed joint joint_2_sec_6_right_conn
- removed joint joint_2_sec_6_right_wall
- removed joint joint_2_sec_7_left_conn
- removed joint joint_2_sec_7_left_wall
- removed joint joint_2_sec_7_right_conn
- removed joint joint_2_sec_7_right_wall
- removed joint joint_2_sec_8_left_conn
- removed joint joint_2_sec_8_left_wall
- removed joint joint_2_sec_8_right_conn
- removed joint joint_2_sec_8_right_wall
- removed joint joint_2_sec_9_left_conn
- removed joint joint_2_sec_9_left_wall
- removed joint joint_2_sec_9_right_conn
- removed joint joint_2_sec_9_right_wall
- removed joint joint_3_int_side_2
- removed joint joint_3_int_side_3_left
- removed joint joint_3_int_side_3_right
- removed joint joint_4_sec_10_left_wall
- removed joint joint_4_sec_10_right_wall
- removed joint joint_4_sec_5_left_conn
- removed joint joint_4_sec_5_right_conn
- removed joint joint_4_sec_6_left_conn
- removed joint joint_4_sec_6_left_wall
- removed joint joint_4_sec_6_right_conn
- removed joint joint_4_sec_6_right_wall
- removed joint joint_4_sec_7_left_conn
- removed joint joint_4_sec_7_left_wall
- removed joint joint_4_sec_7_right_conn
- removed joint joint_4_sec_7_right_wall
- removed joint joint_4_sec_8_left_conn
- removed joint joint_4_sec_8_left_wall
- removed joint joint_4_sec_8_right_conn
- removed joint joint_4_sec_8_right_wall
- removed joint joint_4_sec_9_left_conn
- removed joint joint_4_sec_9_left_wall
- removed joint joint_4_sec_9_right_conn
- removed joint joint_4_sec_9_right_wall
- added joint joint_3_int_side_2_left: type fixed, parent base, child 3_int_side_2_left, origin xyz=0 0 0 rpy=0 0 0
- added joint joint_3_int_side_2_right: type fixed, parent base, child 3_int_side_2_right, origin xyz=0 0 0 rpy=0 0 0
- added joint joint_3_int_side_3: type fixed, parent base, child 3_int_side_3, origin xyz=0 0 0 rpy=0 0 0
