Commit message: working hallway and intersection functions!

File: urdf/random_hall.urdf (robot description, URDF)
Before this commit: robot hallway, 49 links, 48 joints
Links:
- removed link 3_int_side_2_left
- removed link 3_int_side_2_right
- removed link 4_sec_4_left_conn
- removed link 4_sec_4_right_conn
- removed link 4_sec_5_left_wall
- removed link 4_sec_5_right_wall
- added link 2_sec_10_left_wall; collision box size=5.0 0.2 3.0; visual box size=5.0 0.2 3.0
- added link 2_sec_10_right_wall; collision box size=5.0 0.2 3.0; visual box size=5.0 0.2 3.0
- added link 2_sec_5_left_conn; collision box size=0.2 0.325 3.0; visual box size=0.2 0.325 3.0
- added link 2_sec_5_right_conn; collision box size=0.2 0.325 3.0; visual box size=0.2 0.325 3.0
- added link 2_sec_6_left_conn; collision box size=0.2 0.59 3.0; visual box size=0.2 0.59 3.0
- added link 2_sec_6_left_wall; collision box size=3.87 0.2 3.0; visual box size=3.87 0.2 3.0
- added link 2_sec_6_right_conn; collision box size=0.2 0.59 3.0; visual box size=0.2 0.59 3.0
- added link 2_sec_6_right_wall; collision box size=3.87 0.2 3.0; visual box size=3.87 0.2 3.0
- added link 2_sec_7_left_conn; collision box size=0.2 0.35 3.0; visual box size=0.2 0.35 3.0
- added link 2_sec_7_left_wall; collision box size=5.87 0.2 3.0; visual box size=5.87 0.2 3.0
- added link 2_sec_7_right_conn; collision box size=0.2 0.35 3.0; visual box size=0.2 0.35 3.0
- added link 2_sec_7_right_wall; collision box size=5.87 0.2 3.0; visual box size=5.87 0.2 3.0
- added link 2_sec_8_left_conn; collision box size=0.2 0.61 3.0; visual box size=0.2 0.61 3.0
- added link 2_sec_8_left_wall; collision box size=4.24 0.2 3.0; visual box size=4.24 0.2 3.0
- added link 2_sec_8_right_conn; collision box size=0.2 0.61 3.0; visual box size=0.2 0.61 3.0
- added link 2_sec_8_right_wall; collision box size=4.24 0.2 3.0; visual box size=4.24 0.2 3.0
- added link 2_sec_9_left_conn; collision box size=0.2 0.465 3.0; visual box size=0.2 0.465 3.0
- added link 2_sec_9_left_wall; collision box size=4.35 0.2 3.0; visual box size=4.35 0.2 3.0
- added link 2_sec_9_right_conn; collision box size=0.2 0.465 3.0; visual box size=0.2 0.465 3.0
- added link 2_sec_9_right_wall; collision box size=4.35 0.2 3.0; visual box size=4.35 0.2 3.0
- added link 3_int_side_2; collision box size=0.2 5.9 3.0; visual box size=0.2 5.9 3.0
- added link 5_int_side_0_left; collision box size=0.2 0.9 3.0; visual box size=0.2 0.9 3.0
- added link 5_int_side_0_right; collision box size=0.2 0.9 3.0; visual box size=0.2 0.9 3.0
- added link 5_int_side_1; collision box size=5.9 0.2 3.0; visual box size=5.9 0.2 3.0
- added link 5_int_side_2; collision box size=0.2 5.9 3.0; visual box size=0.2 5.9 3.0
- added link 5_int_side_3_left; collision box size=0.9 0.2 3.0; visual box size=0.9 0.2 3.0
- added link 5_int_side_3_right; collision box size=0.9 0.2 3.0; visual box size=0.9 0.2 3.0
- added link 6_sec_1_left_conn; collision box size=-0.2 -0.465 3.0; visual box size=-0.2 -0.465 3.0
- added link 6_sec_1_left_wall; collision box size=-5.0 -0.2 3.0; visual box size=-5.0 -0.2 3.0
- added link 6_sec_1_right_conn; collision box size=-0.2 -0.465 3.0; visual box size=-0.2 -0.465 3.0
- added link 6_sec_1_right_wall; collision box size=-5.0 -0.2 3.0; visual box size=-5.0 -0.2 3.0
- added link 6_sec_2_left_conn; collision box size=-0.2 -0.21 3.0; visual box size=-0.2 -0.21 3.0
- added link 6_sec_2_left_wall; collision box size=-5.32 -0.2 3.0; visual box size=-5.32 -0.2 3.0
- added link 6_sec_2_right_conn; collision box size=-0.2 -0.21 3.0; visual box size=-0.2 -0.21 3.0
- added link 6_sec_2_right_wall; collision box size=-5.32 -0.2 3.0; visual box size=-5.32 -0.2 3.0
- added link 6_sec_3_left_conn; collision box size=-0.2 -0.915 3.0; visual box size=-0.2 -0.915 3.0
- added link 6_sec_3_left_wall; collision box size=-3.56 -0.2 3.0; visual box size=-3.56 -0.2 3.0
- added link 6_sec_3_right_conn; collision box size=-0.2 -0.915 3.0; visual box size=-0.2 -0.915 3.0
- added link 6_sec_3_right_wall; collision box size=-3.56 -0.2 3.0; visual box size=-3.56 -0.2 3.0
- added link 6_sec_4_left_conn; collision box size=-0.2 -1.17 3.0; visual box size=-0.2 -1.17 3.0
- added link 6_sec_4_left_wall; collision box size=-3.81 -0.2 3.0; visual box size=-3.81 -0.2 3.0
- added link 6_sec_4_right_conn; collision box size=-0.2 -1.17 3.0; visual box size=-0.2 -1.17 3.0
- added link 6_sec_4_right_wall; collision box size=-3.81 -0.2 3.0; visual box size=-3.81 -0.2 3.0
- added link 6_sec_5_left_wall; collision box size=-5.0 -0.2 3.0; visual box size=-5.0 -0.2 3.0
- added link 6_sec_5_right_wall; collision box size=-5.0 -0.2 3.0; visual box size=-5.0 -0.2 3.0
- link 1_int_side_2_left: geometry collision box size=0.2 0.9 3.0; visual box size=0.2 0.9 3.0
- link 1_int_side_2_right: geometry collision box size=0.2 0.9 3.0; visual box size=0.2 0.9 3.0
- link 2_sec_1_left_conn: geometry collision box size=0.2 0.63 3.0; visual box size=0.2 0.63 3.0
- link 2_sec_1_right_conn: geometry collision box size=0.2 0.63 3.0; visual box size=0.2 0.63 3.0
- link 2_sec_2_left_conn: geometry collision box size=0.2 0.605 3.0; visual box size=0.2 0.605 3.0
- link 2_sec_2_left_wall: geometry collision box size=6.22 0.2 3.0; visual box size=6.22 0.2 3.0
- link 2_sec_2_right_conn: geometry collision box size=0.2 0.605 3.0; visual box size=0.2 0.605 3.0
- link 2_sec_2_right_wall: geometry collision box size=6.22 0.2 3.0; visual box size=6.22 0.2 3.0
- link 2_sec_3_left_conn: geometry collision box size=0.2 0.275 3.0; visual box size=0.2 0.275 3.0
- link 2_sec_3_left_wall: geometry collision box size=4.69 0.2 3.0; visual box size=4.69 0.2 3.0
- link 2_sec_3_right_conn: geometry collision box size=0.2 0.275 3.0; visual box size=0.2 0.275 3.0
- link 2_sec_3_right_wall: geometry collision box size=4.69 0.2 3.0; visual box size=4.69 0.2 3.0
- link 2_sec_4_left_conn: geometry collision box size=0.2 0.36 3.0; visual box size=0.2 0.36 3.0
- link 2_sec_4_left_wall: geometry collision box size=4.84 0.2 3.0; visual box size=4.84 0.2 3.0
- link 2_sec_4_right_conn: geometry collision box size=0.2 0.36 3.0; visual box size=0.2 0.36 3.0
- link 2_sec_4_right_wall: geometry collision box size=4.84 0.2 3.0; visual box size=4.84 0.2 3.0
- link 2_sec_5_left_wall: geometry collision box size=4.34 0.2 3.0; visual box size=4.34 0.2 3.0
- link 2_sec_5_right_wall: geometry collision box size=4.34 0.2 3.0; visual box size=4.34 0.2 3.0
- link 3_int_side_0_left: geometry collision box size=0.2 0.9 3.0; visual box size=0.2 0.9 3.0
- link 3_int_side_0_right: geometry collision box size=0.2 0.9 3.0; visual box size=0.2 0.9 3.0
- link 3_int_side_1_left: geometry collision box size=0.9 0.2 3.0; visual box size=0.9 0.2 3.0
- link 3_int_side_1_right: geometry collision box size=0.9 0.2 3.0; visual box size=0.9 0.2 3.0
- link 4_sec_1_left_conn: geometry collision box size=0.44 0.2 3.0; visual box size=0.44 0.2 3.0
- link 4_sec_1_right_conn: geometry collision box size=0.44 0.2 3.0; visual box size=0.44 0.2 3.0
- link 4_sec_2_left_conn: geometry collision box size=0.295 0.2 3.0; visual box size=0.295 0.2 3.0
- link 4_sec_2_left_wall: geometry collision box size=0.2 3.67 3.0; visual box size=0.2 3.67 3.0
- link 4_sec_2_right_conn: geometry collision box size=0.295 0.2 3.0; visual box size=0.295 0.2 3.0
- link 4_sec_2_right_wall: geometry collision box size=0.2 3.67 3.0; visual box size=0.2 3.67 3.0
- link 4_sec_3_left_conn: geometry collision box size=0.535 0.2 3.0; visual box size=0.535 0.2 3.0
- link 4_sec_3_left_wall: geometry collision box size=0.2 5.94 3.0; visual box size=0.2 5.94 3.0
- link 4_sec_3_right_conn: geometry collision box size=0.535 0.2 3.0; visual box size=0.535 0.2 3.0
- link 4_sec_3_right_wall: geometry collision box size=0.2 5.94 3.0; visual box size=0.2 5.94 3.0
- link 4_sec_4_left_wall: geometry collision box size=0.2 5.0 3.0; visual box size=0.2 5.0 3.0
- link 4_sec_4_right_wall: geometry collision box size=0.2 5.0 3.0; visual box size=0.2 5.0 3.0
- link base: geometry collision box size=51.46 51.02 0.2; visual box size=51.46 51.02 0.2
Joints:
- removed joint joint_3_int_side_2_left
- removed joint joint_3_int_side_2_right
- removed joint joint_4_sec_4_left_conn
- removed joint joint_4_sec_4_right_conn
- removed joint joint_4_sec_5_left_wall
- removed joint joint_4_sec_5_right_wall
- added joint joint_2_sec_10_left_wall: type fixed, parent base, child 2_sec_10_left_wall, origin xyz=0 0 0 rpy=0 0 0
- added joint joint_2_sec_10_right_wall: type fixed, parent base, child 2_sec_10_right_wall, origin xyz=0 0 0 rpy=0 0 0
- added joint joint_2_sec_5_left_conn: type fixed, parent base, child 2_sec_5_left_conn, origin xyz=0 0 0 rpy=0 0 0
- added joint joint_2_sec_5_right_conn: type fixed, parent base, child 2_sec_5_right_conn, origin xyz=0 0 0 rpy=0 0 0
- added joint joint_2_sec_6_left_conn: type fixed, parent base, child 2_sec_6_left_conn, origin xyz=0 0 0 rpy=0 0 0
- added joint joint_2_sec_6_left_wall: type fixed, parent base, child 2_sec_6_left_wall, origin xyz=0 0 0 rpy=0 0 0
- added joint joint_2_sec_6_right_conn: type fixed, parent base, child 2_sec_6_right_conn, origin xyz=0 0 0 rpy=0 0 0
- added joint joint_2_sec_6_right_wall: type fixed, parent base, child 2_sec_6_right_wall, origin xyz=0 0 0 rpy=0 0 0
- added joint joint_2_sec_7_left_conn: type fixed, parent base, child 2_sec_7_left_conn, origin xyz=0 0 0 rpy=0 0 0
- added joint joint_2_sec_7_left_wall: type fixed, parent base, child 2_sec_7_left_wall, origin xyz=0 0 0 rpy=0 0 0
- added joint joint_2_sec_7_right_conn: type fixed, parent base, child 2_sec_7_right_conn, origin xyz=0 0 0 rpy=0 0 0
- added joint joint_2_sec_7_right_wall: type fixed, parent base, child 2_sec_7_right_wall, origin xyz=0 0 0 rpy=0 0 0
- added joint joint_2_sec_8_left_conn: type fixed, parent base, child 2_sec_8_left_conn, origin xyz=0 0 0 rpy=0 0 0
- added joint joint_2_sec_8_left_wall: type fixed, parent base, child 2_sec_8_left_wall, origin xyz=0 0 0 rpy=0 0 0
- added joint joint_2_sec_8_right_conn: type fixed, parent base, child 2_sec_8_right_conn, origin xyz=0 0 0 rpy=0 0 0
- added joint joint_2_sec_8_right_wall: type fixed, parent base, child 2_sec_8_right_wall, origin xyz=0 0 0 rpy=0 0 0
- added joint joint_2_sec_9_left_conn: type fixed, parent base, child 2_sec_9_left_conn, origin xyz=0 0 0 rpy=0 0 0
- added joint joint_2_sec_9_left_wall: type fixed, parent base, child 2_sec_9_left_wall, origin xyz=0 0 0 rpy=0 0 0
- added joint joint_2_sec_9_right_conn: type fixed, parent base, child 2_sec_9_right_conn, origin xyz=0 0 0 rpy=0 0 0
- added joint joint_2_sec_9_right_wall: type fixed, parent base, child 2_sec_9_right_wall, origin xyz=0 0 0 rpy=0 0 0
- added joint joint_3_int_side_2: type fixed, parent base, child 3_int_side_2, origin xyz=0 0 0 rpy=0 0 0
- added joint joint_5_int_side_0_left: type fixed, parent base, child 5_int_side_0_left, origin xyz=0 0 0 rpy=0 0 0
- added joint joint_5_int_side_0_right: type fixed, parent base, child 5_int_side_0_right, origin xyz=0 0 0 rpy=0 0 0
- added joint joint_5_int_side_1: type fixed, parent base, child 5_int_side_1, origin xyz=0 0 0 rpy=0 0 0
- added joint joint_5_int_side_2: type fixed, parent base, child 5_int_side_2, origin xyz=0 0 0 rpy=0 0 0
- added joint joint_5_int_side_3_left: type fixed, parent base, child 5_int_side_3_left, origin xyz=0 0 0 rpy=0 0 0
- added joint joint_5_int_side_3_right: type fixed, parent base, child 5_int_side_3_right, origin xyz=0 0 0 rpy=0 0 0
- added joint joint_6_sec_1_left_conn: type fixed, parent base, child 6_sec_1_left_conn, origin xyz=0 0 0 rpy=0 0 0
- added joint joint_6_sec_1_left_wall: type fixed, parent base, child 6_sec_1_left_wall, origin xyz=0 0 0 rpy=0 0 0
- added joint joint_6_sec_1_right_conn: type fixed, parent base, child 6_sec_1_right_conn, origin xyz=0 0 0 rpy=0 0 0
- added joint joint_6_sec_1_right_wall: type fixed, parent base, child 6_sec_1_right_wall, origin xyz=0 0 0 rpy=0 0 0
- added joint joint_6_sec_2_left_conn: type fixed, parent base, child 6_sec_2_left_conn, origin xyz=0 0 0 rpy=0 0 0
- added joint joint_6_sec_2_left_wall: type fixed, parent base, child 6_sec_2_left_wall, origin xyz=0 0 0 rpy=0 0 0
- added joint joint_6_sec_2_right_conn: type fixed, parent base, child 6_sec_2_right_conn, origin xyz=0 0 0 rpy=0 0 0
- added joint joint_6_sec_2_right_wall: type fixed, parent base, child 6_sec_2_right_wall, origin xyz=0 0 0 rpy=0 0 0
- added joint joint_6_sec_3_left_conn: type fixed, parent base, child 6_sec_3_left_conn, origin xyz=0 0 0 rpy=0 0 0
- added joint joint_6_sec_3_left_wall: type fixed, parent base, child 6_sec_3_left_wall, origin xyz=0 0 0 rpy=0 0 0
- added joint joint_6_sec_3_right_conn: type fixed, parent base, child 6_sec_3_right_conn, origin xyz=0 0 0 rpy=0 0 0
- added joint joint_6_sec_3_right_wall: type fixed, parent base, child 6_sec_3_right_wall, origin xyz=0 0 0 rpy=0 0 0
- added joint joint_6_sec_4_left_conn: type fixed, parent base, child 6_sec_4_left_conn, origin xyz=0 0 0 rpy=0 0 0
- added joint joint_6_sec_4_left_wall: type fixed, parent base, child 6_sec_4_left_wall, origin xyz=0 0 0 rpy=0 0 0
- added joint joint_6_sec_4_right_conn: type fixed, parent base, child 6_sec_4_right_conn, origin xyz=0 0 0 rpy=0 0 0
- added joint joint_6_sec_4_right_wall: type fixed, parent base, child 6_sec_4_right_wall, origin xyz=0 0 0 rpy=0 0 0
- added joint joint_6_sec_5_left_wall: type fixed, parent base, child 6_sec_5_left_wall, origin xyz=0 0 0 rpy=0 0 0
- added joint joint_6_sec_5_right_wall: type fixed, parent base, child 6_sec_5_right_wall, origin xyz=0 0 0 rpy=0 0 0

Commit message: room launch file with person

File: urdf/random_hall.urdf (robot description, URDF)
Before this commit: robot hallway, 88 links, 87 joints
Links:
- link 1_int_side_0: geometry collision box size=0.2 6.4 3.0; visual box size=0.2 6.4 3.0
- link 1_int_side_1: geometry collision box size=6.4 0.2 3.0; visual box size=6.4 0.2 3.0
- link 1_int_side_2_left: geometry collision box size=0.2 1.2 3.0; visual box size=0.2 1.2 3.0
- link 1_int_side_2_right: geometry collision box size=0.2 1.2 3.0; visual box size=0.2 1.2 3.0
- link 1_int_side_3: geometry collision box size=6.4 0.2 3.0; visual box size=6.4 0.2 3.0
- link 2_sec_10_left_wall: geometry collision box size=4.0 0.2 3.0; visual box size=4.0 0.2 3.0
- link 2_sec_10_right_wall: geometry collision box size=4.0 0.2 3.0; visual box size=4.0 0.2 3.0
- link 2_sec_1_left_conn: geometry collision box size=0.2 0.48 3.0; visual box size=0.2 0.48 3.0
- link 2_sec_1_left_wall: geometry collision box size=4.0 0.2 3.0; visual box size=4.0 0.2 3.0
- link 2_sec_1_right_conn: geometry collision box size=0.2 0.48 3.0; visual box size=0.2 0.48 3.0
- link 2_sec_1_right_wall: geometry collision box size=4.0 0.2 3.0; visual box size=4.0 0.2 3.0
- link 2_sec_2_left_conn: geometry collision box size=0.2 1.13 3.0; visual box size=0.2 1.13 3.0
- link 2_sec_2_left_wall: geometry collision box size=3.85 0.2 3.0; visual box size=3.85 0.2 3.0
- link 2_sec_2_right_conn: geometry collision box size=0.2 1.13 3.0; visual box size=0.2 1.13 3.0
- link 2_sec_2_right_wall: geometry collision box size=3.85 0.2 3.0; visual box size=3.85 0.2 3.0
- link 2_sec_3_left_conn: geometry collision box size=0.2 0.27 3.0; visual box size=0.2 0.27 3.0
- link 2_sec_3_left_wall: geometry collision box size=4.55 0.2 3.0; visual box size=4.55 0.2 3.0
- link 2_sec_3_right_conn: geometry collision box size=0.2 0.27 3.0; visual box size=0.2 0.27 3.0
- link 2_sec_3_right_wall: geometry collision box size=4.55 0.2 3.0; visual box size=4.55 0.2 3.0
- link 2_sec_4_left_conn: geometry collision box size=0.2 0.35 3.0; visual box size=0.2 0.35 3.0
- link 2_sec_4_left_wall: geometry collision box size=3.74 0.2 3.0; visual box size=3.74 0.2 3.0
- link 2_sec_4_right_conn: geometry collision box size=0.2 0.35 3.0; visual box size=0.2 0.35 3.0
- link 2_sec_4_right_wall: geometry collision box size=3.74 0.2 3.0; visual box size=3.74 0.2 3.0
- link 2_sec_5_left_conn: geometry collision box size=0.2 0.535 3.0; visual box size=0.2 0.535 3.0
- link 2_sec_5_left_wall: geometry collision box size=5.13 0.2 3.0; visual box size=5.13 0.2 3.0
- link 2_sec_5_right_conn: geometry collision box size=0.2 0.535 3.0; visual box size=0.2 0.535 3.0
- link 2_sec_5_right_wall: geometry collision box size=5.13 0.2 3.0; visual box size=5.13 0.2 3.0
- link 2_sec_6_left_conn: geometry collision box size=0.2 1.065 3.0; visual box size=0.2 1.065 3.0
- link 2_sec_6_left_wall: geometry collision box size=3.46 0.2 3.0; visual box size=3.46 0.2 3.0
- link 2_sec_6_right_conn: geometry collision box size=0.2 1.065 3.0; visual box size=0.2 1.065 3.0
- link 2_sec_6_right_wall: geometry collision box size=3.46 0.2 3.0; visual box size=3.46 0.2 3.0
- link 2_sec_7_left_conn: geometry collision box size=0.2 0.685 3.0; visual box size=0.2 0.685 3.0
- link 2_sec_7_left_wall: geometry collision box size=3.0 0.2 3.0; visual box size=3.0 0.2 3.0
- link 2_sec_7_right_conn: geometry collision box size=0.2 0.685 3.0; visual box size=0.2 0.685 3.0
- link 2_sec_7_right_wall: geometry collision box size=3.0 0.2 3.0; visual box size=3.0 0.2 3.0
- link 2_sec_8_left_conn: geometry collision box size=0.2 1.115 3.0; visual box size=0.2 1.115 3.0
- link 2_sec_8_left_wall: geometry collision box size=2.92 0.2 3.0; visual box size=2.92 0.2 3.0
- link 2_sec_8_right_conn: geometry collision box size=0.2 1.115 3.0; visual box size=0.2 1.115 3.0
- link 2_sec_8_right_wall: geometry collision box size=2.92 0.2 3.0; visual box size=2.92 0.2 3.0
- link 2_sec_9_left_conn: geometry collision box size=0.2 1.13 3.0; visual box size=0.2 1.13 3.0
- link 2_sec_9_left_wall: geometry collision box size=6.06 0.2 3.0; visual box size=6.06 0.2 3.0
- link 2_sec_9_right_conn: geometry collision box size=0.2 1.13 3.0; visual box size=0.2 1.13 3.0
- link 2_sec_9_right_wall: geometry collision box size=6.06 0.2 3.0; visual box size=6.06 0.2 3.0
- link 3_int_side_0_left: geometry collision box size=0.2 1.2 3.0; visual box size=0.2 1.2 3.0
- link 3_int_side_0_right: geometry collision box size=0.2 1.2 3.0; visual box size=0.2 1.2 3.0
- link 3_int_side_1_left: geometry collision box size=1.2 0.2 3.0; visual box size=1.2 0.2 3.0
- link 3_int_side_1_right: geometry collision box size=1.2 0.2 3.0; visual box size=1.2 0.2 3.0
- link 3_int_side_2: geometry collision box size=0.2 6.4 3.0; visual box size=0.2 6.4 3.0
- link 3_int_side_3: geometry collision box size=6.4 0.2 3.0; visual box size=6.4 0.2 3.0
- link 4_sec_1_left_conn: geometry collision box size=1.015 0.2 3.0; visual box size=1.015 0.2 3.0
- link 4_sec_1_left_wall: geometry collision box size=0.2 4.0 3.0; visual box size=0.2 4.0 3.0
- link 4_sec_1_right_conn: geometry collision box size=1.015 0.2 3.0; visual box size=1.015 0.2 3.0
- link 4_sec_1_right_wall: geometry collision box size=0.2 4.0 3.0; visual box size=0.2 4.0 3.0
- link 4_sec_2_left_conn: geometry collision box size=0.36 0.2 3.0; visual box size=0.36 0.2 3.0
- link 4_sec_2_left_wall: geometry collision box size=0.2 3.86 3.0; visual box size=0.2 3.86 3.0
- link 4_sec_2_right_conn: geometry collision box size=0.36 0.2 3.0; visual box size=0.36 0.2 3.0
- link 4_sec_2_right_wall: geometry collision box size=0.2 3.86 3.0; visual box size=0.2 3.86 3.0
- link 4_sec_3_left_conn: geometry collision box size=0.855 0.2 3.0; visual box size=0.855 0.2 3.0
- link 4_sec_3_left_wall: geometry collision box size=0.2 5.53 3.0; visual box size=0.2 5.53 3.0
- link 4_sec_3_right_conn: geometry collision box size=0.855 0.2 3.0; visual box size=0.855 0.2 3.0
- link 4_sec_3_right_wall: geometry collision box size=0.2 5.53 3.0; visual box size=0.2 5.53 3.0
- link 4_sec_4_left_wall: geometry collision box size=0.2 4.0 3.0; visual box size=0.2 4.0 3.0
- link 4_sec_4_right_wall: geometry collision box size=0.2 4.0 3.0; visual box size=0.2 4.0 3.0
- link 5_int_side_0_left: geometry collision box size=0.2 1.2 3.0; visual box size=0.2 1.2 3.0
- link 5_int_side_0_right: geometry collision box size=0.2 1.2 3.0; visual box size=0.2 1.2 3.0
- link 5_int_side_1: geometry collision box size=6.4 0.2 3.0; visual box size=6.4 0.2 3.0
- link 5_int_side_2: geometry collision box size=0.2 6.4 3.0; visual box size=0.2 6.4 3.0
- link 5_int_side_3_left: geometry collision box size=1.2 0.2 3.0; visual box size=1.2 0.2 3.0
- link 5_int_side_3_right: geometry collision box size=1.2 0.2 3.0; visual box size=1.2 0.2 3.0
- link 6_sec_1_left_conn: geometry collision box size=-0.2 -1.11 3.0; visual box size=-0.2 -1.11 3.0
- link 6_sec_1_left_wall: geometry collision box size=-4.0 -0.2 3.0; visual box size=-4.0 -0.2 3.0
- link 6_sec_1_right_conn: geometry collision box size=-0.2 -1.11 3.0; visual box size=-0.2 -1.11 3.0
- link 6_sec_1_right_wall: geometry collision box size=-4.0 -0.2 3.0; visual box size=-4.0 -0.2 3.0
- link 6_sec_2_left_conn: geometry collision box size=-0.2 -0.875 3.0; visual box size=-0.2 -0.875 3.0
- link 6_sec_2_left_wall: geometry collision box size=-5.3 -0.2 3.0; visual box size=-5.3 -0.2 3.0
- link 6_sec_2_right_conn: geometry collision box size=-0.2 -0.875 3.0; visual box size=-0.2 -0.875 3.0
- link 6_sec_2_right_wall: geometry collision box size=-5.3 -0.2 3.0; visual box size=-5.3 -0.2 3.0
- link 6_sec_3_left_conn: geometry collision box size=-0.2 -1.0 3.0; visual box size=-0.2 -1.0 3.0
- link 6_sec_3_left_wall: geometry collision box size=-3.6 -0.2 3.0; visual box size=-3.6 -0.2 3.0
- link 6_sec_3_right_conn: geometry collision box size=-0.2 -1.0 3.0; visual box size=-0.2 -1.0 3.0
- link 6_sec_3_right_wall: geometry collision box size=-3.6 -0.2 3.0; visual box size=-3.6 -0.2 3.0
- link 6_sec_4_left_conn: geometry collision box size=-0.2 -1.235 3.0; visual box size=-0.2 -1.235 3.0
- link 6_sec_4_left_wall: geometry collision box size=-2.65 -0.2 3.0; visual box size=-2.65 -0.2 3.0
- link 6_sec_4_right_conn: geometry collision box size=-0.2 -1.235 3.0; visual box size=-0.2 -1.235 3.0
- link 6_sec_4_right_wall: geometry collision box size=-2.65 -0.2 3.0; visual box size=-2.65 -0.2 3.0
- link 6_sec_5_left_wall: geometry collision box size=-4.0 -0.2 3.0; visual box size=-4.0 -0.2 3.0
- link 6_sec_5_right_wall: geometry collision box size=-4.0 -0.2 3.0; visual box size=-4.0 -0.2 3.0
- link base: geometry collision box size=42.32 47.58 0.2; visual box size=42.32 47.58 0.2
