Commit message: subscribes to bumper value and prints to txt file

File: urdf/random_hall.urdf (robot description, URDF)
Before this commit: robot hallway, 143 links, 142 joints
Links:
- removed link 2_sec_10_left_wall
- removed link 2_sec_10_right_wall
- removed link 2_sec_6_left_conn
- removed link 2_sec_6_right_conn
- removed link 2_sec_7_left_conn
- removed link 2_sec_7_left_wall
- removed link 2_sec_7_right_conn
- removed link 2_sec_7_right_wall
- removed link 2_sec_8_left_conn
- removed link 2_sec_8_left_wall
- removed link 2_sec_8_right_conn
- removed link 2_sec_8_right_wall
- removed link 2_sec_9_left_conn
- removed link 2_sec_9_left_wall
- removed link 2_sec_9_right_conn
- removed link 2_sec_9_right_wall
- removed link 4_sec_5_left_conn
- removed link 4_sec_5_right_conn
- removed link 4_sec_6_left_conn
- removed link 4_sec_6_left_wall
- removed link 4_sec_6_right_conn
- removed link 4_sec_6_right_wall
- removed link 4_sec_7_left_conn
- removed link 4_sec_7_left_wall
- removed link 4_sec_7_right_conn
- removed link 4_sec_7_right_wall
- removed link 4_sec_8_left_conn
- removed link 4_sec_8_left_wall
- removed link 4_sec_8_right_conn
- removed link 4_sec_8_right_wall
- removed link 4_sec_9_left_wall
- removed link 4_sec_9_right_wall
- removed link 7_sec_5_left_conn
- removed link 7_sec_5_right_conn
- removed link 7_sec_6_left_conn
- removed link 7_sec_6_left_wall
- removed link 7_sec_6_right_conn
- removed link 7_sec_6_right_wall
- removed link 7_sec_7_left_conn
- removed link 7_sec_7_left_wall
- removed link 7_sec_7_right_conn
- removed link 7_sec_7_right_wall
- removed link 7_sec_8_left_conn
- removed link 7_sec_8_left_wall
- removed link 7_sec_8_right_conn
- removed link 7_sec_8_right_wall
- removed link 7_sec_9_left_wall
- removed link 7_sec_9_right_wall
- link 2_sec_1_left_conn: geometry collision box size=0.2 0.215 3.0; visual box size=0.2 0.215 3.0
- link 2_sec_1_right_conn: geometry collision box size=0.2 0.215 3.0; visual box size=0.2 0.215 3.0
- link 2_sec_2_left_conn: geometry collision box size=0.2 0.805 3.0; visual box size=0.2 0.805 3.0
- link 2_sec_2_left_wall: geometry collision box size=4.26 0.2 3.0; visual box size=4.26 0.2 3.0
- link 2_sec_2_right_conn: geometry collision box size=0.2 0.805 3.0; visual box size=0.2 0.805 3.0
- link 2_sec_2_right_wall: geometry collision box size=4.26 0.2 3.0; visual box size=4.26 0.2 3.0
- link 2_sec_3_left_conn: geometry collision box size=0.2 0.805 3.0; visual box size=0.2 0.805 3.0
- link 2_sec_3_left_wall: geometry collision box size=2.82 0.2 3.0; visual box size=2.82 0.2 3.0
- link 2_sec_3_right_conn: geometry collision box size=0.2 0.805 3.0; visual box size=0.2 0.805 3.0
- link 2_sec_3_right_wall: geometry collision box size=2.82 0.2 3.0; visual box size=2.82 0.2 3.0
- link 2_sec_4_left_conn: geometry collision box size=0.2 0.99 3.0; visual box size=0.2 0.99 3.0
- link 2_sec_4_left_wall: geometry collision box size=3.34 0.2 3.0; visual box size=3.34 0.2 3.0
- link 2_sec_4_right_conn: geometry collision box size=0.2 0.99 3.0; visual box size=0.2 0.99 3.0
- link 2_sec_4_right_wall: geometry collision box size=3.34 0.2 3.0; visual box size=3.34 0.2 3.0
- link 2_sec_5_left_conn: geometry collision box size=0.2 1.005 3.0; visual box size=0.2 1.005 3.0
- link 2_sec_5_left_wall: geometry collision box size=3.08 0.2 3.0; visual box size=3.08 0.2 3.0
- link 2_sec_5_right_conn: geometry collision box size=0.2 1.005 3.0; visual box size=0.2 1.005 3.0
- link 2_sec_5_right_wall: geometry collision box size=3.08 0.2 3.0; visual box size=3.08 0.2 3.0
- link 2_sec_6_left_wall: geometry collision box size=4.0 0.2 3.0; visual box size=4.0 0.2 3.0
- link 2_sec_6_right_wall: geometry collision box size=4.0 0.2 3.0; visual box size=4.0 0.2 3.0
- link 4_sec_1_left_conn: geometry collision box size=1.11 0.2 3.0; visual box size=1.11 0.2 3.0
- link 4_sec_1_right_conn: geometry collision box size=1.11 0.2 3.0; visual box size=1.11 0.2 3.0
- link 4_sec_2_left_conn: geometry collision box size=1.135 0.2 3.0; visual box size=1.135 0.2 3.0
- link 4_sec_2_left_wall: geometry collision box size=0.2 5.19 3.0; visual box size=0.2 5.19 3.0
- link 4_sec_2_right_conn: geometry collision box size=1.135 0.2 3.0; visual box size=1.135 0.2 3.0
- link 4_sec_2_right_wall: geometry collision box size=0.2 5.19 3.0; visual box size=0.2 5.19 3.0
- link 4_sec_3_left_conn: geometry collision box size=0.615 0.2 3.0; visual box size=0.615 0.2 3.0
- link 4_sec_3_left_wall: geometry collision box size=0.2 3.53 3.0; visual box size=0.2 3.53 3.0
- link 4_sec_3_right_conn: geometry collision box size=0.615 0.2 3.0; visual box size=0.615 0.2 3.0
- link 4_sec_3_right_wall: geometry collision box size=0.2 3.53 3.0; visual box size=0.2 3.53 3.0
- link 4_sec_4_left_conn: geometry collision box size=0.59 0.2 3.0; visual box size=0.59 0.2 3.0
- link 4_sec_4_left_wall: geometry collision box size=0.2 4.95 3.0; visual box size=0.2 4.95 3.0
- link 4_sec_4_right_conn: geometry collision box size=0.59 0.2 3.0; visual box size=0.59 0.2 3.0
- link 4_sec_4_right_wall: geometry collision box size=0.2 4.95 3.0; visual box size=0.2 4.95 3.0
- link 4_sec_5_left_wall: geometry collision box size=0.2 4.0 3.0; visual box size=0.2 4.0 3.0
- link 4_sec_5_right_wall: geometry collision box size=0.2 4.0 3.0; visual box size=0.2 4.0 3.0
- link 6_sec_1_left_conn: geometry collision box size=-0.2 -1.205 3.0; visual box size=-0.2 -1.205 3.0
- link 6_sec_1_right_conn: geometry collision box size=-0.2 -1.205 3.0; visual box size=-0.2 -1.205 3.0
- link 6_sec_2_left_conn: geometry collision box size=-0.2 -0.88 3.0; visual box size=-0.2 -0.88 3.0
- link 6_sec_2_left_wall: geometry collision box size=-5.48 -0.2 3.0; visual box size=-5.48 -0.2 3.0
- link 6_sec_2_right_conn: geometry collision box size=-0.2 -0.88 3.0; visual box size=-0.2 -0.88 3.0
- link 6_sec_2_right_wall: geometry collision box size=-5.48 -0.2 3.0; visual box size=-5.48 -0.2 3.0
- link 6_sec_3_left_conn: geometry collision box size=-0.2 -0.325 3.0; visual box size=-0.2 -0.325 3.0
- link 6_sec_3_left_wall: geometry collision box size=-0.61 -0.2 3.0; visual box size=-0.61 -0.2 3.0
- link 6_sec_3_right_conn: geometry collision box size=-0.2 -0.325 3.0; visual box size=-0.2 -0.325 3.0
- link 6_sec_3_right_wall: geometry collision box size=-0.61 -0.2 3.0; visual box size=-0.61 -0.2 3.0
- link 6_sec_4_left_conn: geometry collision box size=-0.2 -0.4 3.0; visual box size=-0.2 -0.4 3.0
- link 6_sec_4_left_wall: geometry collision box size=-3.83 -0.2 3.0; visual box size=-3.83 -0.2 3.0
- link 6_sec_4_right_conn: geometry collision box size=-0.2 -0.4 3.0; visual box size=-0.2 -0.4 3.0
- link 6_sec_4_right_wall: geometry collision box size=-3.83 -0.2 3.0; visual box size=-3.83 -0.2 3.0
- link 7_sec_1_left_conn: geometry collision box size=0.2 0.4 3.0; visual box size=0.2 0.4 3.0
- link 7_sec_1_right_conn: geometry collision box size=0.2 0.4 3.0; visual box size=0.2 0.4 3.0
- link 7_sec_2_left_wall: geometry collision box size=4.88 0.2 3.0; visual box size=4.88 0.2 3.0
- link 7_sec_2_right_wall: geometry collision box size=4.88 0.2 3.0; visual box size=4.88 0.2 3.0
- link 7_sec_3_left_conn: geometry collision box size=0.2 1.14 3.0; visual box size=0.2 1.14 3.0
- link 7_sec_3_left_wall: geometry collision box size=3.38 0.2 3.0; visual box size=3.38 0.2 3.0
- link 7_sec_3_right_conn: geometry collision box size=0.2 1.14 3.0; visual box size=0.2 1.14 3.0
- link 7_sec_3_right_wall: geometry collision box size=3.38 0.2 3.0; visual box size=3.38 0.2 3.0
- link 7_sec_4_left_conn: geometry collision box size=0.2 0.8 3.0; visual box size=0.2 0.8 3.0
- link 7_sec_4_left_wall: geometry collision box size=3.11 0.2 3.0; visual box size=3.11 0.2 3.0
- link 7_sec_4_right_conn: geometry collision box size=0.2 0.8 3.0; visual box size=0.2 0.8 3.0
- link 7_sec_4_right_wall: geometry collision box size=3.11 0.2 3.0; visual box size=3.11 0.2 3.0
- link 7_sec_5_left_wall: geometry collision box size=4.0 0.2 3.0; visual box size=4.0 0.2 3.0
- link 7_sec_5_right_wall: geometry collision box size=4.0 0.2 3.0; visual box size=4.0 0.2 3.0
Joints:
- removed joint joint_2_sec_10_left_wall
- removed joint joint_2_sec_10_right_wall
- removed joint joint_2_sec_6_left_conn
- removed joint joint_2_sec_6_right_conn
- removed joint joint_2_sec_7_left_conn
- removed joint joint_2_sec_7_left_wall
- removed joint joint_2_sec_7_right_conn
- removed joint joint_2_sec_7_right_wall
- removed joint joint_2_sec_8_left_conn
- removed joint joint_2_sec_8_left_wall
- removed joint joint_2_sec_8_right_conn
- removed joint joint_2_sec_8_right_wall
- removed joint joint_2_sec_9_left_conn
- removed joint joint_2_sec_9_left_wall
- removed joint joint_2_sec_9_right_conn
- removed joint joint_2_sec_9_right_wall
- removed joint joint_4_sec_5_left_conn
- removed joint joint_4_sec_5_right_conn
- removed joint joint_4_sec_6_left_conn
- removed joint joint_4_sec_6_left_wall
- removed joint joint_4_sec_6_right_conn
- removed joint joint_4_sec_6_right_wall
- removed joint joint_4_sec_7_left_conn
- removed joint joint_4_sec_7_left_wall
- removed joint joint_4_sec_7_right_conn
- removed joint joint_4_sec_7_right_wall
- removed joint joint_4_sec_8_left_conn
- removed joint joint_4_sec_8_left_wall
- removed joint joint_4_sec_8_right_conn
- removed joint joint_4_sec_8_right_wall
- removed joint joint_4_sec_9_left_wall
- removed joint joint_4_sec_9_right_wall
- removed joint joint_7_sec_5_left_conn
- removed joint joint_7_sec_5_right_conn
- removed joint joint_7_sec_6_left_conn
- removed joint joint_7_sec_6_left_wall
- removed joint joint_7_sec_6_right_conn
- removed joint joint_7_sec_6_right_wall
- removed joint joint_7_sec_7_left_conn
- removed joint joint_7_sec_7_left_wall
- removed joint joint_7_sec_7_right_conn
- removed joint joint_7_sec_7_right_wall
- removed joint joint_7_sec_8_left_conn
- removed joint joint_7_sec_8_left_wall
- removed joint joint_7_sec_8_right_conn
- removed joint joint_7_sec_8_right_wall
- removed joint joint_7_sec_9_left_wall
- removed joint joint_7_sec_9_right_wall
