Commit message: fixed for lidar direction

File: urdf/random_hall.urdf (robot description, URDF)
Before this commit: robot hallway, 95 links, 94 joints
Links:
- removed link 2_sec_5_left_conn
- removed link 2_sec_5_right_conn
- removed link 2_sec_6_left_wall
- removed link 2_sec_6_right_wall
- removed link 5_int_side_2_left
- removed link 5_int_side_2_right
- removed link 7_sec_1_left_conn
- removed link 7_sec_1_left_wall
- removed link 7_sec_1_right_conn
- removed link 7_sec_1_right_wall
- removed link 7_sec_2_left_conn
- removed link 7_sec_2_left_wall
- removed link 7_sec_2_right_conn
- removed link 7_sec_2_right_wall
- removed link 7_sec_3_left_conn
- removed link 7_sec_3_left_wall
- removed link 7_sec_3_right_conn
- removed link 7_sec_3_right_wall
- removed link 7_sec_4_left_conn
- removed link 7_sec_4_left_wall
- removed link 7_sec_4_right_conn
- removed link 7_sec_4_right_wall
- removed link 7_sec_5_left_wall
- removed link 7_sec_5_right_wall
- added link 4_sec_5_left_conn; collision box size=0.915 0.2 3.0; visual box size=0.915 0.2 3.0
- added link 4_sec_5_right_conn; collision box size=0.915 0.2 3.0; visual box size=0.915 0.2 3.0
- added link 4_sec_6_left_wall; collision box size=0.2 4.0 3.0; visual box size=0.2 4.0 3.0
- added link 4_sec_6_right_wall; collision box size=0.2 4.0 3.0; visual box size=0.2 4.0 3.0
- added link 5_int_side_2; collision box size=0.2 6.4 3.0; visual box size=0.2 6.4 3.0
- added link 6_sec_5_left_conn; collision box size=-0.2 -0.325 3.0; visual box size=-0.2 -0.325 3.0
- added link 6_sec_5_right_conn; collision box size=-0.2 -0.325 3.0; visual box size=-0.2 -0.325 3.0
- added link 6_sec_6_left_conn; collision box size=-0.2 -0.23 3.0; visual box size=-0.2 -0.23 3.0
- added link 6_sec_6_left_wall; collision box size=-2.9 -0.2 3.0; visual box size=-2.9 -0.2 3.0
- added link 6_sec_6_right_conn; collision box size=-0.2 -0.23 3.0; visual box size=-0.2 -0.23 3.0
- added link 6_sec_6_right_wall; collision box size=-2.9 -0.2 3.0; visual box size=-2.9 -0.2 3.0
- added link 6_sec_7_left_conn; collision box size=-0.2 -1.76 3.0; visual box size=-0.2 -1.76 3.0
- added link 6_sec_7_left_wall; collision box size=-3.41 -0.2 3.0; visual box size=-3.41 -0.2 3.0
- added link 6_sec_7_right_conn; collision box size=-0.2 -1.76 3.0; visual box size=-0.2 -1.76 3.0
- added link 6_sec_7_right_wall; collision box size=-3.41 -0.2 3.0; visual box size=-3.41 -0.2 3.0
- added link 6_sec_8_left_conn; collision box size=-0.2 -1.7 3.0; visual box size=-0.2 -1.7 3.0
- added link 6_sec_8_left_wall; collision box size=-2.81 -0.2 3.0; visual box size=-2.81 -0.2 3.0
- added link 6_sec_8_right_conn; collision box size=-0.2 -1.7 3.0; visual box size=-0.2 -1.7 3.0
- added link 6_sec_8_right_wall; collision box size=-2.81 -0.2 3.0; visual box size=-2.81 -0.2 3.0
- added link 6_sec_9_left_wall; collision box size=-4.0 -0.2 3.0; visual box size=-4.0 -0.2 3.0
- added link 6_sec_9_right_wall; collision box size=-4.0 -0.2 3.0; visual box size=-4.0 -0.2 3.0
- added link 7_int_side_0; collision box size=0.2 6.4 3.0; visual box size=0.2 6.4 3.0
- added link 7_int_side_1_left; collision box size=1.2 0.2 3.0; visual box size=1.2 0.2 3.0
- added link 7_int_side_1_right; collision box size=1.2 0.2 3.0; visual box size=1.2 0.2 3.0
- added link 7_int_side_2_left; collision box size=0.2 1.2 3.0; visual box size=0.2 1.2 3.0
- added link 7_int_side_2_right; collision box size=0.2 1.2 3.0; visual box size=0.2 1.2 3.0
- added link 7_int_side_3; collision box size=6.4 0.2 3.0; visual box size=6.4 0.2 3.0
- added link 8_sec_1_left_conn; collision box size=1.185 0.2 3.0; visual box size=1.185 0.2 3.0
- added link 8_sec_1_left_wall; collision box size=0.2 4.0 3.0; visual box size=0.2 4.0 3.0
- added link 8_sec_1_right_conn; collision box size=1.185 0.2 3.0; visual box size=1.185 0.2 3.0
- added link 8_sec_1_right_wall; collision box size=0.2 4.0 3.0; visual box size=0.2 4.0 3.0
- added link 8_sec_2_left_conn; collision box size=1.185 0.2 3.0; visual box size=1.185 0.2 3.0
- added link 8_sec_2_left_wall; collision box size=0.2 2.3 3.0; visual box size=0.2 2.3 3.0
- added link 8_sec_2_right_conn; collision box size=1.185 0.2 3.0; visual box size=1.185 0.2 3.0
- added link 8_sec_2_right_wall; collision box size=0.2 2.3 3.0; visual box size=0.2 2.3 3.0
- added link 8_sec_3_left_wall; collision box size=0.2 4.0 3.0; visual box size=0.2 4.0 3.0
- added link 8_sec_3_right_wall; collision box size=0.2 4.0 3.0; visual box size=0.2 4.0 3.0
- link 2_sec_1_left_conn: geometry collision box size=0.2 0.99 3.0; visual box size=0.2 0.99 3.0
- link 2_sec_1_right_conn: geometry collision box size=0.2 0.99 3.0; visual box size=0.2 0.99 3.0
- link 2_sec_2_left_conn: geometry collision box size=0.2 0.305 3.0; visual box size=0.2 0.305 3.0
- link 2_sec_2_left_wall: geometry collision box size=4.8 0.2 3.0; visual box size=4.8 0.2 3.0
- link 2_sec_2_right_conn: geometry collision box size=0.2 0.305 3.0; visual box size=0.2 0.305 3.0
- link 2_sec_2_right_wall: geometry collision box size=4.8 0.2 3.0; visual box size=4.8 0.2 3.0
- link 2_sec_3_left_conn: geometry collision box size=0.2 0.58 3.0; visual box size=0.2 0.58 3.0
- link 2_sec_3_left_wall: geometry collision box size=3.24 0.2 3.0; visual box size=3.24 0.2 3.0
- link 2_sec_3_right_conn: geometry collision box size=0.2 0.58 3.0; visual box size=0.2 0.58 3.0
- link 2_sec_3_right_wall: geometry collision box size=3.24 0.2 3.0; visual box size=3.24 0.2 3.0
- link 2_sec_4_left_conn: geometry collision box size=0.2 0.715 3.0; visual box size=0.2 0.715 3.0
- link 2_sec_4_left_wall: geometry collision box size=2.42 0.2 3.0; visual box size=2.42 0.2 3.0
- link 2_sec_4_right_conn: geometry collision box size=0.2 0.715 3.0; visual box size=0.2 0.715 3.0
- link 2_sec_4_right_wall: geometry collision box size=2.42 0.2 3.0; visual box size=2.42 0.2 3.0
- link 2_sec_5_left_wall: geometry collision box size=4.0 0.2 3.0; visual box size=4.0 0.2 3.0
- link 2_sec_5_right_wall: geometry collision box size=4.0 0.2 3.0; visual box size=4.0 0.2 3.0
- link 4_sec_1_left_conn: geometry collision box size=0.57 0.2 3.0; visual box size=0.57 0.2 3.0
- link 4_sec_1_right_conn: geometry collision box size=0.57 0.2 3.0; visual box size=0.57 0.2 3.0
- link 4_sec_2_left_conn: geometry collision box size=0.66 0.2 3.0; visual box size=0.66 0.2 3.0
- link 4_sec_2_left_wall: geometry collision box size=0.2 4.53 3.0; visual box size=0.2 4.53 3.0
- link 4_sec_2_right_conn: geometry collision box size=0.66 0.2 3.0; visual box size=0.66 0.2 3.0
- link 4_sec_2_right_wall: geometry collision box size=0.2 4.53 3.0; visual box size=0.2 4.53 3.0
- link 4_sec_3_left_conn: geometry collision box size=1.05 0.2 3.0; visual box size=1.05 0.2 3.0
- link 4_sec_3_left_wall: geometry collision box size=0.2 2.82 3.0; visual box size=0.2 2.82 3.0
- link 4_sec_3_right_conn: geometry collision box size=1.05 0.2 3.0; visual box size=1.05 0.2 3.0
- link 4_sec_3_right_wall: geometry collision box size=0.2 2.82 3.0; visual box size=0.2 2.82 3.0
- link 4_sec_4_left_conn: geometry collision box size=0.425 0.2 3.0; visual box size=0.425 0.2 3.0
- link 4_sec_4_left_wall: geometry collision box size=0.2 3.24 3.0; visual box size=0.2 3.24 3.0
- link 4_sec_4_right_conn: geometry collision box size=0.425 0.2 3.0; visual box size=0.425 0.2 3.0
- link 4_sec_4_right_wall: geometry collision box size=0.2 3.24 3.0; visual box size=0.2 3.24 3.0
- link 4_sec_5_left_wall: geometry collision box size=0.2 5.81 3.0; visual box size=0.2 5.81 3.0
- link 4_sec_5_right_wall: geometry collision box size=0.2 5.81 3.0; visual box size=0.2 5.81 3.0
- link 6_sec_1_left_conn: geometry collision box size=-0.2 -0.365 3.0; visual box size=-0.2 -0.365 3.0
- link 6_sec_1_right_conn: geometry collision box size=-0.2 -0.365 3.0; visual box size=-0.2 -0.365 3.0
- link 6_sec_2_left_conn: geometry collision box size=-0.2 -0.85 3.0; visual box size=-0.2 -0.85 3.0
- link 6_sec_2_left_wall: geometry collision box size=-3.08 -0.2 3.0; visual box size=-3.08 -0.2 3.0
- link 6_sec_2_right_conn: geometry collision box size=-0.2 -0.85 3.0; visual box size=-0.2 -0.85 3.0
- link 6_sec_2_right_wall: geometry collision box size=-3.08 -0.2 3.0; visual box size=-3.08 -0.2 3.0
- link 6_sec_3_left_conn: geometry collision box size=-0.2 -0.87 3.0; visual box size=-0.2 -0.87 3.0
- link 6_sec_3_left_wall: geometry collision box size=-4.12 -0.2 3.0; visual box size=-4.12 -0.2 3.0
- link 6_sec_3_right_conn: geometry collision box size=-0.2 -0.87 3.0; visual box size=-0.2 -0.87 3.0
- link 6_sec_3_right_wall: geometry collision box size=-4.12 -0.2 3.0; visual box size=-4.12 -0.2 3.0
- link 6_sec_4_left_conn: geometry collision box size=-0.2 -0.54 3.0; visual box size=-0.2 -0.54 3.0
- link 6_sec_4_left_wall: geometry collision box size=-2.17 -0.2 3.0; visual box size=-2.17 -0.2 3.0
- link 6_sec_4_right_conn: geometry collision box size=-0.2 -0.54 3.0; visual box size=-0.2 -0.54 3.0
- link 6_sec_4_right_wall: geometry collision box size=-2.17 -0.2 3.0; visual box size=-2.17 -0.2 3.0
- link 6_sec_5_left_wall: geometry collision box size=-2.72 -0.2 3.0; visual box size=-2.72 -0.2 3.0
- link 6_sec_5_right_wall: geometry collision box size=-2.72 -0.2 3.0; visual box size=-2.72 -0.2 3.0
Joints:
- removed joint joint_2_sec_5_left_conn
- removed joint joint_2_sec_5_right_conn
- removed joint joint_2_sec_6_left_wall
- removed joint joint_2_sec_6_right_wall
- removed joint joint_5_int_side_2_left
- removed joint joint_5_int_side_2_right
- removed joint joint_7_sec_1_left_conn
- removed joint joint_7_sec_1_left_wall
- removed joint joint_7_sec_1_right_conn
- removed joint joint_7_sec_1_right_wall
- removed joint joint_7_sec_2_left_conn
- removed joint joint_7_sec_2_left_wall
- removed joint joint_7_sec_2_right_conn
- removed joint joint_7_sec_2_right_wall
- removed joint joint_7_sec_3_left_conn
- removed joint joint_7_sec_3_left_wall
- removed joint joint_7_sec_3_right_conn
- removed joint joint_7_sec_3_right_wall
- removed joint joint_7_sec_4_left_conn
- removed joint joint_7_sec_4_left_wall
- removed joint joint_7_sec_4_right_conn
- removed joint joint_7_sec_4_right_wall
- removed joint joint_7_sec_5_left_wall
- removed joint joint_7_sec_5_right_wall
- added joint joint_4_sec_5_left_conn: type fixed, parent base, child 4_sec_5_left_conn, origin xyz=0 0 0 rpy=0 0 0
- added joint joint_4_sec_5_right_conn: type fixed, parent base, child 4_sec_5_right_conn, origin xyz=0 0 0 rpy=0 0 0
- added joint joint_4_sec_6_left_wall: type fixed, parent base, child 4_sec_6_left_wall, origin xyz=0 0 0 rpy=0 0 0
- added joint joint_4_sec_6_right_wall: type fixed, parent base, child 4_sec_6_right_wall, origin xyz=0 0 0 rpy=0 0 0
- added joint joint_5_int_side_2: type fixed, parent base, child 5_int_side_2, origin xyz=0 0 0 rpy=0 0 0
- added joint joint_6_sec_5_left_conn: type fixed, parent base, child 6_sec_5_left_conn, origin xyz=0 0 0 rpy=0 0 0
- added joint joint_6_sec_5_right_conn: type fixed, parent base, child 6_sec_5_right_conn, origin xyz=0 0 0 rpy=0 0 0
- added joint joint_6_sec_6_left_conn: type fixed, parent base, child 6_sec_6_left_conn, origin xyz=0 0 0 rpy=0 0 0
- added joint joint_6_sec_6_left_wall: type fixed, parent base, child 6_sec_6_left_wall, origin xyz=0 0 0 rpy=0 0 0
- added joint joint_6_sec_6_right_conn: type fixed, parent base, child 6_sec_6_right_conn, origin xyz=0 0 0 rpy=0 0 0
- added joint joint_6_sec_6_right_wall: type fixed, parent base, child 6_sec_6_right_wall, origin xyz=0 0 0 rpy=0 0 0
- added joint joint_6_sec_7_left_conn: type fixed, parent base, child 6_sec_7_left_conn, origin xyz=0 0 0 rpy=0 0 0
- added joint joint_6_sec_7_left_wall: type fixed, parent base, child 6_sec_7_left_wall, origin xyz=0 0 0 rpy=0 0 0
- added joint joint_6_sec_7_right_conn: type fixed, parent base, child 6_sec_7_right_conn, origin xyz=0 0 0 rpy=0 0 0
- added joint joint_6_sec_7_right_wall: type fixed, parent base, child 6_sec_7_right_wall, origin xyz=0 0 0 rpy=0 0 0
- added joint joint_6_sec_8_left_conn: type fixed, parent base, child 6_sec_8_left_conn, origin xyz=0 0 0 rpy=0 0 0
- added joint joint_6_sec_8_left_wall: type fixed, parent base, child 6_sec_8_left_wall, origin xyz=0 0 0 rpy=0 0 0
- added joint joint_6_sec_8_right_conn: type fixed, parent base, child 6_sec_8_right_conn, origin xyz=0 0 0 rpy=0 0 0
- added joint joint_6_sec_8_right_wall: type fixed, parent base, child 6_sec_8_right_wall, origin xyz=0 0 0 rpy=0 0 0
- added joint joint_6_sec_9_left_wall: type fixed, parent base, child 6_sec_9_left_wall, origin xyz=0 0 0 rpy=0 0 0
- added joint joint_6_sec_9_right_wall: type fixed, parent base, child 6_sec_9_right_wall, origin xyz=0 0 0 rpy=0 0 0
- added joint joint_7_int_side_0: type fixed, parent base, child 7_int_side_0, origin xyz=0 0 0 rpy=0 0 0
- added joint joint_7_int_side_1_left: type fixed, parent base, child 7_int_side_1_left, origin xyz=0 0 0 rpy=0 0 0
- added joint joint_7_int_side_1_right: type fixed, parent base, child 7_int_side_1_right, origin xyz=0 0 0 rpy=0 0 0
- added joint joint_7_int_side_2_left: type fixed, parent base, child 7_int_side_2_left, origin xyz=0 0 0 rpy=0 0 0
- added joint joint_7_int_side_2_right: type fixed, parent base, child 7_int_side_2_right, origin xyz=0 0 0 rpy=0 0 0
- added joint joint_7_int_side_3: type fixed, parent base, child 7_int_side_3, origin xyz=0 0 0 rpy=0 0 0
- added joint joint_8_sec_1_left_conn: type fixed, parent base, child 8_sec_1_left_conn, origin xyz=0 0 0 rpy=0 0 0
- added joint joint_8_sec_1_left_wall: type fixed, parent base, child 8_sec_1_left_wall, origin xyz=0 0 0 rpy=0 0 0
- added joint joint_8_sec_1_right_conn: type fixed, parent base, child 8_sec_1_right_conn, origin xyz=0 0 0 rpy=0 0 0
- added joint joint_8_sec_1_right_wall: type fixed, parent base, child 8_sec_1_right_wall, origin xyz=0 0 0 rpy=0 0 0
- added joint joint_8_sec_2_left_conn: type fixed, parent base, child 8_sec_2_left_conn, origin xyz=0 0 0 rpy=0 0 0
- added joint joint_8_sec_2_left_wall: type fixed, parent base, child 8_sec_2_left_wall, origin xyz=0 0 0 rpy=0 0 0
- added joint joint_8_sec_2_right_conn: type fixed, parent base, child 8_sec_2_right_conn, origin xyz=0 0 0 rpy=0 0 0
- added joint joint_8_sec_2_right_wall: type fixed, parent base, child 8_sec_2_right_wall, origin xyz=0 0 0 rpy=0 0 0
- added joint joint_8_sec_3_left_wall: type fixed, parent base, child 8_sec_3_left_wall, origin xyz=0 0 0 rpy=0 0 0
- added joint joint_8_sec_3_right_wall: type fixed, parent base, child 8_sec_3_right_wall, origin xyz=0 0 0 rpy=0 0 0
