Commit message: simulations for navigation parameters

File: urdf/random_hall.urdf (robot description, URDF)
Before this commit: robot hallway, 108 links, 107 joints
Links:
- removed link 2_sec_4_left_conn
- removed link 2_sec_4_right_conn
- removed link 2_sec_5_left_wall
- removed link 2_sec_5_right_wall
- removed link 4_sec_4_left_conn
- removed link 4_sec_4_right_conn
- removed link 4_sec_5_left_conn
- removed link 4_sec_5_left_wall
- removed link 4_sec_5_right_conn
- removed link 4_sec_5_right_wall
- removed link 4_sec_6_left_wall
- removed link 4_sec_6_right_wall
- added link 8_sec_3_left_conn; collision box size=1.09 0.2 3.0; visual box size=1.09 0.2 3.0
- added link 8_sec_3_right_conn; collision box size=1.09 0.2 3.0; visual box size=1.09 0.2 3.0
- added link 8_sec_4_left_conn; collision box size=1.115 0.2 3.0; visual box size=1.115 0.2 3.0
- added link 8_sec_4_left_wall; collision box size=0.2 4.58 3.0; visual box size=0.2 4.58 3.0
- added link 8_sec_4_right_conn; collision box size=1.115 0.2 3.0; visual box size=1.115 0.2 3.0
- added link 8_sec_4_right_wall; collision box size=0.2 4.58 3.0; visual box size=0.2 4.58 3.0
- added link 8_sec_5_left_wall; collision box size=0.2 4.0 3.0; visual box size=0.2 4.0 3.0
- added link 8_sec_5_right_wall; collision box size=0.2 4.0 3.0; visual box size=0.2 4.0 3.0
- link 2_sec_1_left_conn: geometry collision box size=0.2 0.29 3.0; visual box size=0.2 0.29 3.0
- link 2_sec_1_right_conn: geometry collision box size=0.2 0.29 3.0; visual box size=0.2 0.29 3.0
- link 2_sec_2_left_conn: geometry collision box size=0.2 0.595 3.0; visual box size=0.2 0.595 3.0
- link 2_sec_2_left_wall: geometry collision box size=4.69 0.2 3.0; visual box size=4.69 0.2 3.0
- link 2_sec_2_right_conn: geometry collision box size=0.2 0.595 3.0; visual box size=0.2 0.595 3.0
- link 2_sec_2_right_wall: geometry collision box size=4.69 0.2 3.0; visual box size=4.69 0.2 3.0
- link 2_sec_3_left_conn: geometry collision box size=0.2 0.685 3.0; visual box size=0.2 0.685 3.0
- link 2_sec_3_left_wall: geometry collision box size=3.53 0.2 3.0; visual box size=3.53 0.2 3.0
- link 2_sec_3_right_conn: geometry collision box size=0.2 0.685 3.0; visual box size=0.2 0.685 3.0
- link 2_sec_3_right_wall: geometry collision box size=3.53 0.2 3.0; visual box size=3.53 0.2 3.0
- link 2_sec_4_left_wall: geometry collision box size=4.0 0.2 3.0; visual box size=4.0 0.2 3.0
- link 2_sec_4_right_wall: geometry collision box size=4.0 0.2 3.0; visual box size=4.0 0.2 3.0
- link 4_sec_1_left_conn: geometry collision box size=1.38 0.2 3.0; visual box size=1.38 0.2 3.0
- link 4_sec_1_right_conn: geometry collision box size=1.38 0.2 3.0; visual box size=1.38 0.2 3.0
- link 4_sec_2_left_conn: geometry collision box size=0.64 0.2 3.0; visual box size=0.64 0.2 3.0
- link 4_sec_2_left_wall: geometry collision box size=0.2 4.01 3.0; visual box size=0.2 4.01 3.0
- link 4_sec_2_right_conn: geometry collision box size=0.64 0.2 3.0; visual box size=0.64 0.2 3.0
- link 4_sec_2_right_wall: geometry collision box size=0.2 4.01 3.0; visual box size=0.2 4.01 3.0
- link 4_sec_3_left_conn: geometry collision box size=0.94 0.2 3.0; visual box size=0.94 0.2 3.0
- link 4_sec_3_left_wall: geometry collision box size=0.2 2.09 3.0; visual box size=0.2 2.09 3.0
- link 4_sec_3_right_conn: geometry collision box size=0.94 0.2 3.0; visual box size=0.94 0.2 3.0
- link 4_sec_3_right_wall: geometry collision box size=0.2 2.09 3.0; visual box size=0.2 2.09 3.0
- link 4_sec_4_left_wall: geometry collision box size=0.2 4.0 3.0; visual box size=0.2 4.0 3.0
- link 4_sec_4_right_wall: geometry collision box size=0.2 4.0 3.0; visual box size=0.2 4.0 3.0
- link 6_sec_1_left_conn: geometry collision box size=-0.2 -0.65 3.0; visual box size=-0.2 -0.65 3.0
- link 6_sec_1_right_conn: geometry collision box size=-0.2 -0.65 3.0; visual box size=-0.2 -0.65 3.0
- link 6_sec_2_left_conn: geometry collision box size=-0.2 -0.47 3.0; visual box size=-0.2 -0.47 3.0
- link 6_sec_2_left_wall: geometry collision box size=-4.19 -0.2 3.0; visual box size=-4.19 -0.2 3.0
- link 6_sec_2_right_conn: geometry collision box size=-0.2 -0.47 3.0; visual box size=-0.2 -0.47 3.0
- link 6_sec_2_right_wall: geometry collision box size=-4.19 -0.2 3.0; visual box size=-4.19 -0.2 3.0
- link 6_sec_3_left_conn: geometry collision box size=-0.2 -0.485 3.0; visual box size=-0.2 -0.485 3.0
- link 6_sec_3_left_wall: geometry collision box size=-2.49 -0.2 3.0; visual box size=-2.49 -0.2 3.0
- link 6_sec_3_right_conn: geometry collision box size=-0.2 -0.485 3.0; visual box size=-0.2 -0.485 3.0
- link 6_sec_3_right_wall: geometry collision box size=-2.49 -0.2 3.0; visual box size=-2.49 -0.2 3.0
- link 6_sec_4_left_conn: geometry collision box size=-0.2 -0.435 3.0; visual box size=-0.2 -0.435 3.0
- link 6_sec_4_left_wall: geometry collision box size=-3.01 -0.2 3.0; visual box size=-3.01 -0.2 3.0
- link 6_sec_4_right_conn: geometry collision box size=-0.2 -0.435 3.0; visual box size=-0.2 -0.435 3.0
- link 6_sec_4_right_wall: geometry collision box size=-3.01 -0.2 3.0; visual box size=-3.01 -0.2 3.0
- link 6_sec_5_left_conn: geometry collision box size=-0.2 -1.24 3.0; visual box size=-0.2 -1.24 3.0
- link 6_sec_5_left_wall: geometry collision box size=-5.27 -0.2 3.0; visual box size=-5.27 -0.2 3.0
- link 6_sec_5_right_conn: geometry collision box size=-0.2 -1.24 3.0; visual box size=-0.2 -1.24 3.0
- link 6_sec_5_right_wall: geometry collision box size=-5.27 -0.2 3.0; visual box size=-5.27 -0.2 3.0
- link 6_sec_6_left_conn: geometry collision box size=-0.2 -0.83 3.0; visual box size=-0.2 -0.83 3.0
- link 6_sec_6_left_wall: geometry collision box size=-5.4 -0.2 3.0; visual box size=-5.4 -0.2 3.0
- link 6_sec_6_right_conn: geometry collision box size=-0.2 -0.83 3.0; visual box size=-0.2 -0.83 3.0
- link 6_sec_6_right_wall: geometry collision box size=-5.4 -0.2 3.0; visual box size=-5.4 -0.2 3.0
- link 6_sec_7_left_conn: geometry collision box size=-0.2 -1.145 3.0; visual box size=-0.2 -1.145 3.0
- link 6_sec_7_left_wall: geometry collision box size=-3.28 -0.2 3.0; visual box size=-3.28 -0.2 3.0
- link 6_sec_7_right_conn: geometry collision box size=-0.2 -1.145 3.0; visual box size=-0.2 -1.145 3.0
- link 6_sec_7_right_wall: geometry collision box size=-3.28 -0.2 3.0; visual box size=-3.28 -0.2 3.0
- link 6_sec_8_left_conn: geometry collision box size=-0.2 -0.505 3.0; visual box size=-0.2 -0.505 3.0
- link 6_sec_8_left_wall: geometry collision box size=-2.85 -0.2 3.0; visual box size=-2.85 -0.2 3.0
- link 6_sec_8_right_conn: geometry collision box size=-0.2 -0.505 3.0; visual box size=-0.2 -0.505 3.0
- link 6_sec_8_right_wall: geometry collision box size=-2.85 -0.2 3.0; visual box size=-2.85 -0.2 3.0
- link 8_sec_1_left_conn: geometry collision box size=0.375 0.2 3.0; visual box size=0.375 0.2 3.0
- link 8_sec_1_right_conn: geometry collision box size=0.375 0.2 3.0; visual box size=0.375 0.2 3.0
- link 8_sec_2_left_conn: geometry collision box size=0.35 0.2 3.0; visual box size=0.35 0.2 3.0
- link 8_sec_2_left_wall: geometry collision box size=0.2 3.31 3.0; visual box size=0.2 3.31 3.0
- link 8_sec_2_right_conn: geometry collision box size=0.35 0.2 3.0; visual box size=0.35 0.2 3.0
- link 8_sec_2_right_wall: geometry collision box size=0.2 3.31 3.0; visual box size=0.2 3.31 3.0
- link 8_sec_3_left_wall: geometry collision box size=0.2 5.21 3.0; visual box size=0.2 5.21 3.0
- link 8_sec_3_right_wall: geometry collision box size=0.2 5.21 3.0; visual box size=0.2 5.21 3.0
Joints:
- removed joint joint_2_sec_4_left_conn
- removed joint joint_2_sec_4_right_conn
- removed joint joint_2_sec_5_left_wall
- removed joint joint_2_sec_5_right_wall
- removed joint joint_4_sec_4_left_conn
- removed joint joint_4_sec_4_right_conn
- removed joint joint_4_sec_5_left_conn
- removed joint joint_4_sec_5_left_wall
- removed joint joint_4_sec_5_right_conn
- removed joint joint_4_sec_5_right_wall
- removed joint joint_4_sec_6_left_wall
- removed joint joint_4_sec_6_right_wall
- added joint joint_8_sec_3_left_conn: type fixed, parent base, child 8_sec_3_left_conn, origin xyz=0 0 0 rpy=0 0 0
- added joint joint_8_sec_3_right_conn: type fixed, parent base, child 8_sec_3_right_conn, origin xyz=0 0 0 rpy=0 0 0
- added joint joint_8_sec_4_left_conn: type fixed, parent base, child 8_sec_4_left_conn, origin xyz=0 0 0 rpy=0 0 0
- added joint joint_8_sec_4_left_wall: type fixed, parent base, child 8_sec_4_left_wall, origin xyz=0 0 0 rpy=0 0 0
- added joint joint_8_sec_4_right_conn: type fixed, parent base, child 8_sec_4_right_conn, origin xyz=0 0 0 rpy=0 0 0
- added joint joint_8_sec_4_right_wall: type fixed, parent base, child 8_sec_4_right_wall, origin xyz=0 0 0 rpy=0 0 0
- added joint joint_8_sec_5_left_wall: type fixed, parent base, child 8_sec_5_left_wall, origin xyz=0 0 0 rpy=0 0 0
- added joint joint_8_sec_5_right_wall: type fixed, parent base, child 8_sec_5_right_wall, origin xyz=0 0 0 rpy=0 0 0

Commit message: simulations

File: urdf/random_hall.urdf (robot description, URDF)
Before this commit: robot hallway, 104 links, 103 joints
Links:
- removed link 8_sec_4_left_conn
- removed link 8_sec_4_right_conn
- removed link 8_sec_5_left_wall
- removed link 8_sec_5_right_wall
- added link 2_sec_4_left_conn; collision box size=0.2 0.825 3.0; visual box size=0.2 0.825 3.0
- added link 2_sec_4_right_conn; collision box size=0.2 0.825 3.0; visual box size=0.2 0.825 3.0
- added link 2_sec_5_left_wall; collision box size=4.0 0.2 3.0; visual box size=4.0 0.2 3.0
- added link 2_sec_5_right_wall; collision box size=4.0 0.2 3.0; visual box size=4.0 0.2 3.0
- added link 4_sec_4_left_conn; collision box size=0.55 0.2 3.0; visual box size=0.55 0.2 3.0
- added link 4_sec_4_right_conn; collision box size=0.55 0.2 3.0; visual box size=0.55 0.2 3.0
- added link 4_sec_5_left_wall; collision box size=0.2 4.0 3.0; visual box size=0.2 4.0 3.0
- added link 4_sec_5_right_wall; collision box size=0.2 4.0 3.0; visual box size=0.2 4.0 3.0
- added link 6_sec_10_left_wall; collision box size=-4.0 -0.2 3.0; visual box size=-4.0 -0.2 3.0
- added link 6_sec_10_right_wall; collision box size=-4.0 -0.2 3.0; visual box size=-4.0 -0.2 3.0
- added link 6_sec_9_left_conn; collision box size=-0.2 -1.65 3.0; visual box size=-0.2 -1.65 3.0
- added link 6_sec_9_right_conn; collision box size=-0.2 -1.65 3.0; visual box size=-0.2 -1.65 3.0
- link 2_sec_1_left_conn: geometry collision box size=0.2 0.73 3.0; visual box size=0.2 0.73 3.0
- link 2_sec_1_right_conn: geometry collision box size=0.2 0.73 3.0; visual box size=0.2 0.73 3.0
- link 2_sec_2_left_conn: geometry collision box size=0.2 0.29 3.0; visual box size=0.2 0.29 3.0
- link 2_sec_2_left_wall: geometry collision box size=5.72 0.2 3.0; visual box size=5.72 0.2 3.0
- link 2_sec_2_right_conn: geometry collision box size=0.2 0.29 3.0; visual box size=0.2 0.29 3.0
- link 2_sec_2_right_wall: geometry collision box size=5.72 0.2 3.0; visual box size=5.72 0.2 3.0
- link 2_sec_3_left_conn: geometry collision box size=0.2 0.385 3.0; visual box size=0.2 0.385 3.0
- link 2_sec_3_left_wall: geometry collision box size=5.41 0.2 3.0; visual box size=5.41 0.2 3.0
- link 2_sec_3_right_conn: geometry collision box size=0.2 0.385 3.0; visual box size=0.2 0.385 3.0
- link 2_sec_3_right_wall: geometry collision box size=5.41 0.2 3.0; visual box size=5.41 0.2 3.0
- link 2_sec_4_left_wall: geometry collision box size=3.45 0.2 3.0; visual box size=3.45 0.2 3.0
- link 2_sec_4_right_wall: geometry collision box size=3.45 0.2 3.0; visual box size=3.45 0.2 3.0
- link 4_sec_1_left_conn: geometry collision box size=0.905 0.2 3.0; visual box size=0.905 0.2 3.0
- link 4_sec_1_right_conn: geometry collision box size=0.905 0.2 3.0; visual box size=0.905 0.2 3.0
- link 4_sec_2_left_conn: geometry collision box size=0.46 0.2 3.0; visual box size=0.46 0.2 3.0
- link 4_sec_2_left_wall: geometry collision box size=0.2 3.21 3.0; visual box size=0.2 3.21 3.0
- link 4_sec_2_right_conn: geometry collision box size=0.46 0.2 3.0; visual box size=0.46 0.2 3.0
- link 4_sec_2_right_wall: geometry collision box size=0.2 3.21 3.0; visual box size=0.2 3.21 3.0
- link 4_sec_3_left_conn: geometry collision box size=0.295 0.2 3.0; visual box size=0.295 0.2 3.0
- link 4_sec_3_left_wall: geometry collision box size=0.2 2.65 3.0; visual box size=0.2 2.65 3.0
- link 4_sec_3_right_conn: geometry collision box size=0.295 0.2 3.0; visual box size=0.295 0.2 3.0
- link 4_sec_3_right_wall: geometry collision box size=0.2 2.65 3.0; visual box size=0.2 2.65 3.0
- link 4_sec_4_left_wall: geometry collision box size=0.2 3.9 3.0; visual box size=0.2 3.9 3.0
- link 4_sec_4_right_wall: geometry collision box size=0.2 3.9 3.0; visual box size=0.2 3.9 3.0
- link 6_sec_1_left_conn: geometry collision box size=-0.2 -1.07 3.0; visual box size=-0.2 -1.07 3.0
- link 6_sec_1_right_conn: geometry collision box size=-0.2 -1.07 3.0; visual box size=-0.2 -1.07 3.0
- link 6_sec_2_left_conn: geometry collision box size=-0.2 -0.79 3.0; visual box size=-0.2 -0.79 3.0
- link 6_sec_2_left_wall: geometry collision box size=-4.52 -0.2 3.0; visual box size=-4.52 -0.2 3.0
- link 6_sec_2_right_conn: geometry collision box size=-0.2 -0.79 3.0; visual box size=-0.2 -0.79 3.0
- link 6_sec_2_right_wall: geometry collision box size=-4.52 -0.2 3.0; visual box size=-4.52 -0.2 3.0
- link 6_sec_3_left_conn: geometry collision box size=-0.2 -0.515 3.0; visual box size=-0.2 -0.515 3.0
- link 6_sec_3_left_wall: geometry collision box size=-3.73 -0.2 3.0; visual box size=-3.73 -0.2 3.0
- link 6_sec_3_right_conn: geometry collision box size=-0.2 -0.515 3.0; visual box size=-0.2 -0.515 3.0
- link 6_sec_3_right_wall: geometry collision box size=-3.73 -0.2 3.0; visual box size=-3.73 -0.2 3.0
- link 6_sec_4_left_conn: geometry collision box size=-0.2 -0.795 3.0; visual box size=-0.2 -0.795 3.0
- link 6_sec_4_left_wall: geometry collision box size=-5.17 -0.2 3.0; visual box size=-5.17 -0.2 3.0
- link 6_sec_4_right_conn: geometry collision box size=-0.2 -0.795 3.0; visual box size=-0.2 -0.795 3.0
- link 6_sec_4_right_wall: geometry collision box size=-5.17 -0.2 3.0; visual box size=-5.17 -0.2 3.0
- link 6_sec_5_left_conn: geometry collision box size=-0.2 -0.48 3.0; visual box size=-0.2 -0.48 3.0
- link 6_sec_5_left_wall: geometry collision box size=-3.65 -0.2 3.0; visual box size=-3.65 -0.2 3.0
- link 6_sec_5_right_conn: geometry collision box size=-0.2 -0.48 3.0; visual box size=-0.2 -0.48 3.0
- link 6_sec_5_right_wall: geometry collision box size=-3.65 -0.2 3.0; visual box size=-3.65 -0.2 3.0
- link 6_sec_6_left_conn: geometry collision box size=-0.2 -0.51 3.0; visual box size=-0.2 -0.51 3.0
- link 6_sec_6_left_wall: geometry collision box size=-3.82 -0.2 3.0; visual box size=-3.82 -0.2 3.0
- link 6_sec_6_right_conn: geometry collision box size=-0.2 -0.51 3.0; visual box size=-0.2 -0.51 3.0
- link 6_sec_6_right_wall: geometry collision box size=-3.82 -0.2 3.0; visual box size=-3.82 -0.2 3.0
- link 6_sec_7_left_conn: geometry collision box size=-0.2 -0.35 3.0; visual box size=-0.2 -0.35 3.0
- link 6_sec_7_left_wall: geometry collision box size=-4.77 -0.2 3.0; visual box size=-4.77 -0.2 3.0
- link 6_sec_7_right_conn: geometry collision box size=-0.2 -0.35 3.0; visual box size=-0.2 -0.35 3.0
- link 6_sec_7_right_wall: geometry collision box size=-4.77 -0.2 3.0; visual box size=-4.77 -0.2 3.0
- link 6_sec_8_left_conn: geometry collision box size=-0.2 -0.91 3.0; visual box size=-0.2 -0.91 3.0
- link 6_sec_8_left_wall: geometry collision box size=-4.24 -0.2 3.0; visual box size=-4.24 -0.2 3.0
- link 6_sec_8_right_conn: geometry collision box size=-0.2 -0.91 3.0; visual box size=-0.2 -0.91 3.0
- link 6_sec_8_right_wall: geometry collision box size=-4.24 -0.2 3.0; visual box size=-4.24 -0.2 3.0
- link 6_sec_9_left_wall: geometry collision box size=-4.86 -0.2 3.0; visual box size=-4.86 -0.2 3.0
- link 6_sec_9_right_wall: geometry collision box size=-4.86 -0.2 3.0; visual box size=-4.86 -0.2 3.0
- link 8_sec_1_left_conn: geometry collision box size=1.07 0.2 3.0; visual box size=1.07 0.2 3.0
- link 8_sec_1_right_conn: geometry collision box size=1.07 0.2 3.0; visual box size=1.07 0.2 3.0
- link 8_sec_2_left_conn: geometry collision box size=0.345 0.2 3.0; visual box size=0.345 0.2 3.0
- link 8_sec_2_left_wall: geometry collision box size=0.2 5.39 3.0; visual box size=0.2 5.39 3.0
- link 8_sec_2_right_conn: geometry collision box size=0.345 0.2 3.0; visual box size=0.345 0.2 3.0
- link 8_sec_2_right_wall: geometry collision box size=0.2 5.39 3.0; visual box size=0.2 5.39 3.0
- link 8_sec_3_left_conn: geometry collision box size=0.925 0.2 3.0; visual box size=0.925 0.2 3.0
- link 8_sec_3_left_wall: geometry collision box size=0.2 3.92 3.0; visual box size=0.2 3.92 3.0
- link 8_sec_3_right_conn: geometry collision box size=0.925 0.2 3.0; visual box size=0.925 0.2 3.0
- link 8_sec_3_right_wall: geometry collision box size=0.2 3.92 3.0; visual box size=0.2 3.92 3.0
- link 8_sec_4_left_wall: geometry collision box size=0.2 4.0 3.0; visual box size=0.2 4.0 3.0
- link 8_sec_4_right_wall: geometry collision box size=0.2 4.0 3.0; visual box size=0.2 4.0 3.0
Joints:
- removed joint joint_8_sec_4_left_conn
- removed joint joint_8_sec_4_right_conn
- removed joint joint_8_sec_5_left_wall
- removed joint joint_8_sec_5_right_wall
- added joint joint_2_sec_4_left_conn: type fixed, parent base, child 2_sec_4_left_conn, origin xyz=0 0 0 rpy=0 0 0
- added joint joint_2_sec_4_right_conn: type fixed, parent base, child 2_sec_4_right_conn, origin xyz=0 0 0 rpy=0 0 0
- added joint joint_2_sec_5_left_wall: type fixed, parent base, child 2_sec_5_left_wall, origin xyz=0 0 0 rpy=0 0 0
- added joint joint_2_sec_5_right_wall: type fixed, parent base, child 2_sec_5_right_wall, origin xyz=0 0 0 rpy=0 0 0
- added joint joint_4_sec_4_left_conn: type fixed, parent base, child 4_sec_4_left_conn, origin xyz=0 0 0 rpy=0 0 0
- added joint joint_4_sec_4_right_conn: type fixed, parent base, child 4_sec_4_right_conn, origin xyz=0 0 0 rpy=0 0 0
- added joint joint_4_sec_5_left_wall: type fixed, parent base, child 4_sec_5_left_wall, origin xyz=0 0 0 rpy=0 0 0
- added joint joint_4_sec_5_right_wall: type fixed, parent base, child 4_sec_5_right_wall, origin xyz=0 0 0 rpy=0 0 0
- added joint joint_6_sec_10_left_wall: type fixed, parent base, child 6_sec_10_left_wall, origin xyz=0 0 0 rpy=0 0 0
- added joint joint_6_sec_10_right_wall: type fixed, parent base, child 6_sec_10_right_wall, origin xyz=0 0 0 rpy=0 0 0
- added joint joint_6_sec_9_left_conn: type fixed, parent base, child 6_sec_9_left_conn, origin xyz=0 0 0 rpy=0 0 0
- added joint joint_6_sec_9_right_conn: type fixed, parent base, child 6_sec_9_right_conn, origin xyz=0 0 0 rpy=0 0 0
