Commit message: second round of simulation testing

File: urdf/random_hall.urdf (robot description, URDF)
Before this commit: robot hallway, 112 links, 111 joints
Links:
- removed link 6_sec_10_left_wall
- removed link 6_sec_10_right_wall
- removed link 6_sec_6_left_conn
- removed link 6_sec_6_right_conn
- removed link 6_sec_7_left_conn
- removed link 6_sec_7_left_wall
- removed link 6_sec_7_right_conn
- removed link 6_sec_7_right_wall
- removed link 6_sec_8_left_conn
- removed link 6_sec_8_left_wall
- removed link 6_sec_8_right_conn
- removed link 6_sec_8_right_wall
- removed link 6_sec_9_left_conn
- removed link 6_sec_9_left_wall
- removed link 6_sec_9_right_conn
- removed link 6_sec_9_right_wall
- link 2_sec_1_left_conn: geometry collision box size=0.2 1.375 3.0; visual box size=0.2 1.375 3.0
- link 2_sec_1_right_conn: geometry collision box size=0.2 1.375 3.0; visual box size=0.2 1.375 3.0
- link 2_sec_2_left_conn: geometry collision box size=0.2 0.465 3.0; visual box size=0.2 0.465 3.0
- link 2_sec_2_left_wall: geometry collision box size=3.44 0.2 3.0; visual box size=3.44 0.2 3.0
- link 2_sec_2_right_conn: geometry collision box size=0.2 0.465 3.0; visual box size=0.2 0.465 3.0
- link 2_sec_2_right_wall: geometry collision box size=3.44 0.2 3.0; visual box size=3.44 0.2 3.0
- link 2_sec_3_left_conn: geometry collision box size=0.2 1.11 3.0; visual box size=0.2 1.11 3.0
- link 2_sec_3_left_wall: geometry collision box size=4.01 0.2 3.0; visual box size=4.01 0.2 3.0
- link 2_sec_3_right_conn: geometry collision box size=0.2 1.11 3.0; visual box size=0.2 1.11 3.0
- link 2_sec_3_right_wall: geometry collision box size=4.01 0.2 3.0; visual box size=4.01 0.2 3.0
- link 2_sec_4_left_conn: geometry collision box size=0.2 0.2 3.0; visual box size=0.2 0.2 3.0
- link 2_sec_4_left_wall: geometry collision box size=4.45 0.2 3.0; visual box size=4.45 0.2 3.0
- link 2_sec_4_right_conn: geometry collision box size=0.2 0.2 3.0; visual box size=0.2 0.2 3.0
- link 2_sec_4_right_wall: geometry collision box size=4.45 0.2 3.0; visual box size=4.45 0.2 3.0
- link 4_sec_1_left_conn: geometry collision box size=0.37 0.2 3.0; visual box size=0.37 0.2 3.0
- link 4_sec_1_right_conn: geometry collision box size=0.37 0.2 3.0; visual box size=0.37 0.2 3.0
- link 4_sec_2_left_conn: geometry collision box size=0.685 0.2 3.0; visual box size=0.685 0.2 3.0
- link 4_sec_2_left_wall: geometry collision box size=0.2 4.53 3.0; visual box size=0.2 4.53 3.0
- link 4_sec_2_right_conn: geometry collision box size=0.685 0.2 3.0; visual box size=0.685 0.2 3.0
- link 4_sec_2_right_wall: geometry collision box size=0.2 4.53 3.0; visual box size=0.2 4.53 3.0
- link 4_sec_3_left_conn: geometry collision box size=0.52 0.2 3.0; visual box size=0.52 0.2 3.0
- link 4_sec_3_left_wall: geometry collision box size=0.2 4.4 3.0; visual box size=0.2 4.4 3.0
- link 4_sec_3_right_conn: geometry collision box size=0.52 0.2 3.0; visual box size=0.52 0.2 3.0
- link 4_sec_3_right_wall: geometry collision box size=0.2 4.4 3.0; visual box size=0.2 4.4 3.0
- link 4_sec_4_left_conn: geometry collision box size=0.535 0.2 3.0; visual box size=0.535 0.2 3.0
- link 4_sec_4_left_wall: geometry collision box size=0.2 5.68 3.0; visual box size=0.2 5.68 3.0
- link 4_sec_4_right_conn: geometry collision box size=0.535 0.2 3.0; visual box size=0.535 0.2 3.0
- link 4_sec_4_right_wall: geometry collision box size=0.2 5.68 3.0; visual box size=0.2 5.68 3.0
- link 6_sec_1_left_conn: geometry collision box size=-0.2 -1.64 3.0; visual box size=-0.2 -1.64 3.0
- link 6_sec_1_right_conn: geometry collision box size=-0.2 -1.64 3.0; visual box size=-0.2 -1.64 3.0
- link 6_sec_2_left_conn: geometry collision box size=-0.2 -1.225 3.0; visual box size=-0.2 -1.225 3.0
- link 6_sec_2_left_wall: geometry collision box size=-2.86 -0.2 3.0; visual box size=-2.86 -0.2 3.0
- link 6_sec_2_right_conn: geometry collision box size=-0.2 -1.225 3.0; visual box size=-0.2 -1.225 3.0
- link 6_sec_2_right_wall: geometry collision box size=-2.86 -0.2 3.0; visual box size=-2.86 -0.2 3.0
- link 6_sec_3_left_conn: geometry collision box size=-0.2 -0.475 3.0; visual box size=-0.2 -0.475 3.0
- link 6_sec_3_left_wall: geometry collision box size=-3.02 -0.2 3.0; visual box size=-3.02 -0.2 3.0
- link 6_sec_3_right_conn: geometry collision box size=-0.2 -0.475 3.0; visual box size=-0.2 -0.475 3.0
- link 6_sec_3_right_wall: geometry collision box size=-3.02 -0.2 3.0; visual box size=-3.02 -0.2 3.0
- link 6_sec_4_left_conn: geometry collision box size=-0.2 -0.735 3.0; visual box size=-0.2 -0.735 3.0
- link 6_sec_4_left_wall: geometry collision box size=-2.43 -0.2 3.0; visual box size=-2.43 -0.2 3.0
- link 6_sec_4_right_conn: geometry collision box size=-0.2 -0.735 3.0; visual box size=-0.2 -0.735 3.0
- link 6_sec_4_right_wall: geometry collision box size=-2.43 -0.2 3.0; visual box size=-2.43 -0.2 3.0
- link 6_sec_5_left_conn: geometry collision box size=-0.2 -0.355 3.0; visual box size=-0.2 -0.355 3.0
- link 6_sec_5_left_wall: geometry collision box size=-2.87 -0.2 3.0; visual box size=-2.87 -0.2 3.0
- link 6_sec_5_right_conn: geometry collision box size=-0.2 -0.355 3.0; visual box size=-0.2 -0.355 3.0
- link 6_sec_5_right_wall: geometry collision box size=-2.87 -0.2 3.0; visual box size=-2.87 -0.2 3.0
- link 6_sec_6_left_wall: geometry collision box size=-4.0 -0.2 3.0; visual box size=-4.0 -0.2 3.0
- link 6_sec_6_right_wall: geometry collision box size=-4.0 -0.2 3.0; visual box size=-4.0 -0.2 3.0
- link 8_sec_1_left_conn: geometry collision box size=0.955 0.2 3.0; visual box size=0.955 0.2 3.0
- link 8_sec_1_right_conn: geometry collision box size=0.955 0.2 3.0; visual box size=0.955 0.2 3.0
- link 8_sec_2_left_conn: geometry collision box size=1.84 0.2 3.0; visual box size=1.84 0.2 3.0
- link 8_sec_2_left_wall: geometry collision box size=0.2 3.21 3.0; visual box size=0.2 3.21 3.0
- link 8_sec_2_right_conn: geometry collision box size=1.84 0.2 3.0; visual box size=1.84 0.2 3.0
- link 8_sec_2_right_wall: geometry collision box size=0.2 3.21 3.0; visual box size=0.2 3.21 3.0
- link 8_sec_3_left_conn: geometry collision box size=1.085 0.2 3.0; visual box size=1.085 0.2 3.0
- link 8_sec_3_left_wall: geometry collision box size=0.2 2.6 3.0; visual box size=0.2 2.6 3.0
- link 8_sec_3_right_conn: geometry collision box size=1.085 0.2 3.0; visual box size=1.085 0.2 3.0
- link 8_sec_3_right_wall: geometry collision box size=0.2 2.6 3.0; visual box size=0.2 2.6 3.0
Joints:
- removed joint joint_6_sec_10_left_wall
- removed joint joint_6_sec_10_right_wall
- removed joint joint_6_sec_6_left_conn
- removed joint joint_6_sec_6_right_conn
- removed joint joint_6_sec_7_left_conn
- removed joint joint_6_sec_7_left_wall
- removed joint joint_6_sec_7_right_conn
- removed joint joint_6_sec_7_right_wall
- removed joint joint_6_sec_8_left_conn
- removed joint joint_6_sec_8_left_wall
- removed joint joint_6_sec_8_right_conn
- removed joint joint_6_sec_8_right_wall
- removed joint joint_6_sec_9_left_conn
- removed joint joint_6_sec_9_left_wall
- removed joint joint_6_sec_9_right_conn
- removed joint joint_6_sec_9_right_wall

Commit message: closest point lidar method

File: urdf/random_hall.urdf (robot description, URDF)
Before this commit: robot hallway, 96 links, 95 joints
Links:
- added link 2_sec_5_left_conn; collision box size=0.2 0.23 3.0; visual box size=0.2 0.23 3.0
- added link 2_sec_5_right_conn; collision box size=0.2 0.23 3.0; visual box size=0.2 0.23 3.0
- added link 2_sec_6_left_conn; collision box size=0.2 0.655 3.0; visual box size=0.2 0.655 3.0
- added link 2_sec_6_left_wall; collision box size=4.21 0.2 3.0; visual box size=4.21 0.2 3.0
- added link 2_sec_6_right_conn; collision box size=0.2 0.655 3.0; visual box size=0.2 0.655 3.0
- added link 2_sec_6_right_wall; collision box size=4.21 0.2 3.0; visual box size=4.21 0.2 3.0
- added link 2_sec_7_left_wall; collision box size=4.0 0.2 3.0; visual box size=4.0 0.2 3.0
- added link 2_sec_7_right_wall; collision box size=4.0 0.2 3.0; visual box size=4.0 0.2 3.0
- added link 4_sec_5_left_conn; collision box size=0.685 0.2 3.0; visual box size=0.685 0.2 3.0
- added link 4_sec_5_right_conn; collision box size=0.685 0.2 3.0; visual box size=0.685 0.2 3.0
- added link 4_sec_6_left_wall; collision box size=0.2 4.0 3.0; visual box size=0.2 4.0 3.0
- added link 4_sec_6_right_wall; collision box size=0.2 4.0 3.0; visual box size=0.2 4.0 3.0
- added link 6_sec_10_left_conn; collision box size=-0.2 -0.745 3.0; visual box size=-0.2 -0.745 3.0
- added link 6_sec_10_left_wall; collision box size=-3.15 -0.2 3.0; visual box size=-3.15 -0.2 3.0
- added link 6_sec_10_right_conn; collision box size=-0.2 -0.745 3.0; visual box size=-0.2 -0.745 3.0
- added link 6_sec_10_right_wall; collision box size=-3.15 -0.2 3.0; visual box size=-3.15 -0.2 3.0
- added link 6_sec_11_left_wall; collision box size=-4.0 -0.2 3.0; visual box size=-4.0 -0.2 3.0
- added link 6_sec_11_right_wall; collision box size=-4.0 -0.2 3.0; visual box size=-4.0 -0.2 3.0
- added link 6_sec_6_left_conn; collision box size=-0.2 -0.42 3.0; visual box size=-0.2 -0.42 3.0
- added link 6_sec_6_right_conn; collision box size=-0.2 -0.42 3.0; visual box size=-0.2 -0.42 3.0
- added link 6_sec_7_left_conn; collision box size=-0.2 -1.295 3.0; visual box size=-0.2 -1.295 3.0
- added link 6_sec_7_left_wall; collision box size=-4.38 -0.2 3.0; visual box size=-4.38 -0.2 3.0
- added link 6_sec_7_right_conn; collision box size=-0.2 -1.295 3.0; visual box size=-0.2 -1.295 3.0
- added link 6_sec_7_right_wall; collision box size=-4.38 -0.2 3.0; visual box size=-4.38 -0.2 3.0
- added link 6_sec_8_left_conn; collision box size=-0.2 -0.485 3.0; visual box size=-0.2 -0.485 3.0
- added link 6_sec_8_left_wall; collision box size=-4.88 -0.2 3.0; visual box size=-4.88 -0.2 3.0
- added link 6_sec_8_right_conn; collision box size=-0.2 -0.485 3.0; visual box size=-0.2 -0.485 3.0
- added link 6_sec_8_right_wall; collision box size=-4.88 -0.2 3.0; visual box size=-4.88 -0.2 3.0
- added link 6_sec_9_left_conn; collision box size=-0.2 -0.8 3.0; visual box size=-0.2 -0.8 3.0
- added link 6_sec_9_left_wall; collision box size=-1.08 -0.2 3.0; visual box size=-1.08 -0.2 3.0
- added link 6_sec_9_right_conn; collision box size=-0.2 -0.8 3.0; visual box size=-0.2 -0.8 3.0
- added link 6_sec_9_right_wall; collision box size=-1.08 -0.2 3.0; visual box size=-1.08 -0.2 3.0
- added link 8_sec_4_left_conn; collision box size=1.18 0.2 3.0; visual box size=1.18 0.2 3.0
- added link 8_sec_4_right_conn; collision box size=1.18 0.2 3.0; visual box size=1.18 0.2 3.0
- added link 8_sec_5_left_wall; collision box size=0.2 4.0 3.0; visual box size=0.2 4.0 3.0
- added link 8_sec_5_right_wall; collision box size=0.2 4.0 3.0; visual box size=0.2 4.0 3.0
- link 2_sec_1_left_conn: geometry collision box size=0.2 1.17 3.0; visual box size=0.2 1.17 3.0
- link 2_sec_1_right_conn: geometry collision box size=0.2 1.17 3.0; visual box size=0.2 1.17 3.0
- link 2_sec_2_left_conn: geometry collision box size=0.2 0.425 3.0; visual box size=0.2 0.425 3.0
- link 2_sec_2_left_wall: geometry collision box size=4.95 0.2 3.0; visual box size=4.95 0.2 3.0
- link 2_sec_2_right_conn: geometry collision box size=0.2 0.425 3.0; visual box size=0.2 0.425 3.0
- link 2_sec_2_right_wall: geometry collision box size=4.95 0.2 3.0; visual box size=4.95 0.2 3.0
- link 2_sec_3_left_conn: geometry collision box size=0.2 0.535 3.0; visual box size=0.2 0.535 3.0
- link 2_sec_3_left_wall: geometry collision box size=5.55 0.2 3.0; visual box size=5.55 0.2 3.0
- link 2_sec_3_right_conn: geometry collision box size=0.2 0.535 3.0; visual box size=0.2 0.535 3.0
- link 2_sec_3_right_wall: geometry collision box size=5.55 0.2 3.0; visual box size=5.55 0.2 3.0
- link 2_sec_4_left_conn: geometry collision box size=0.2 1.705 3.0; visual box size=0.2 1.705 3.0
- link 2_sec_4_left_wall: geometry collision box size=4.4 0.2 3.0; visual box size=4.4 0.2 3.0
- link 2_sec_4_right_conn: geometry collision box size=0.2 1.705 3.0; visual box size=0.2 1.705 3.0
- link 2_sec_4_right_wall: geometry collision box size=4.4 0.2 3.0; visual box size=4.4 0.2 3.0
- link 2_sec_5_left_wall: geometry collision box size=2.18 0.2 3.0; visual box size=2.18 0.2 3.0
- link 2_sec_5_right_wall: geometry collision box size=2.18 0.2 3.0; visual box size=2.18 0.2 3.0
- link 4_sec_1_left_conn: geometry collision box size=0.355 0.2 3.0; visual box size=0.355 0.2 3.0
- link 4_sec_1_right_conn: geometry collision box size=0.355 0.2 3.0; visual box size=0.355 0.2 3.0
- link 4_sec_2_left_conn: geometry collision box size=0.23 0.2 3.0; visual box size=0.23 0.2 3.0
- link 4_sec_2_left_wall: geometry collision box size=0.2 5.66 3.0; visual box size=0.2 5.66 3.0
- link 4_sec_2_right_conn: geometry collision box size=0.23 0.2 3.0; visual box size=0.23 0.2 3.0
- link 4_sec_2_right_wall: geometry collision box size=0.2 5.66 3.0; visual box size=0.2 5.66 3.0
- link 4_sec_3_left_conn: geometry collision box size=0.875 0.2 3.0; visual box size=0.875 0.2 3.0
- link 4_sec_3_left_wall: geometry collision box size=0.2 3.55 3.0; visual box size=0.2 3.55 3.0
- link 4_sec_3_right_conn: geometry collision box size=0.875 0.2 3.0; visual box size=0.875 0.2 3.0
- link 4_sec_3_right_wall: geometry collision box size=0.2 3.55 3.0; visual box size=0.2 3.55 3.0
- link 4_sec_4_left_conn: geometry collision box size=0.205 0.2 3.0; visual box size=0.205 0.2 3.0
- link 4_sec_4_left_wall: geometry collision box size=0.2 5.05 3.0; visual box size=0.2 5.05 3.0
- link 4_sec_4_right_conn: geometry collision box size=0.205 0.2 3.0; visual box size=0.205 0.2 3.0
- link 4_sec_4_right_wall: geometry collision box size=0.2 5.05 3.0; visual box size=0.2 5.05 3.0
- link 4_sec_5_left_wall: geometry collision box size=0.2 4.48 3.0; visual box size=0.2 4.48 3.0
- link 4_sec_5_right_wall: geometry collision box size=0.2 4.48 3.0; visual box size=0.2 4.48 3.0
- link 6_sec_1_left_conn: geometry collision box size=-0.2 -1.7 3.0; visual box size=-0.2 -1.7 3.0
- link 6_sec_1_right_conn: geometry collision box size=-0.2 -1.7 3.0; visual box size=-0.2 -1.7 3.0
- link 6_sec_2_left_conn: geometry collision box size=-0.2 -0.705 3.0; visual box size=-0.2 -0.705 3.0
- link 6_sec_2_left_wall: geometry collision box size=-3.71 -0.2 3.0; visual box size=-3.71 -0.2 3.0
- link 6_sec_2_right_conn: geometry collision box size=-0.2 -0.705 3.0; visual box size=-0.2 -0.705 3.0
- link 6_sec_2_right_wall: geometry collision box size=-3.71 -0.2 3.0; visual box size=-3.71 -0.2 3.0
- link 6_sec_3_left_conn: geometry collision box size=-0.2 -0.845 3.0; visual box size=-0.2 -0.845 3.0
- link 6_sec_3_left_wall: geometry collision box size=-2.73 -0.2 3.0; visual box size=-2.73 -0.2 3.0
- link 6_sec_3_right_conn: geometry collision box size=-0.2 -0.845 3.0; visual box size=-0.2 -0.845 3.0
- link 6_sec_3_right_wall: geometry collision box size=-2.73 -0.2 3.0; visual box size=-2.73 -0.2 3.0
- link 6_sec_4_left_conn: geometry collision box size=-0.2 -0.695 3.0; visual box size=-0.2 -0.695 3.0
- link 6_sec_4_left_wall: geometry collision box size=-4.23 -0.2 3.0; visual box size=-4.23 -0.2 3.0
- link 6_sec_4_right_conn: geometry collision box size=-0.2 -0.695 3.0; visual box size=-0.2 -0.695 3.0
- link 6_sec_4_right_wall: geometry collision box size=-4.23 -0.2 3.0; visual box size=-4.23 -0.2 3.0
- link 6_sec_5_left_conn: geometry collision box size=-0.2 -0.44 3.0; visual box size=-0.2 -0.44 3.0
- link 6_sec_5_left_wall: geometry collision box size=-2.86 -0.2 3.0; visual box size=-2.86 -0.2 3.0
- link 6_sec_5_right_conn: geometry collision box size=-0.2 -0.44 3.0; visual box size=-0.2 -0.44 3.0
- link 6_sec_5_right_wall: geometry collision box size=-2.86 -0.2 3.0; visual box size=-2.86 -0.2 3.0
- link 6_sec_6_left_wall: geometry collision box size=-6.19 -0.2 3.0; visual box size=-6.19 -0.2 3.0
- link 6_sec_6_right_wall: geometry collision box size=-6.19 -0.2 3.0; visual box size=-6.19 -0.2 3.0
- link 8_sec_1_left_conn: geometry collision box size=1.6 0.2 3.0; visual box size=1.6 0.2 3.0
- link 8_sec_1_right_conn: geometry collision box size=1.6 0.2 3.0; visual box size=1.6 0.2 3.0
- link 8_sec_2_left_conn: geometry collision box size=0.78 0.2 3.0; visual box size=0.78 0.2 3.0
- link 8_sec_2_left_wall: geometry collision box size=0.2 3.73 3.0; visual box size=0.2 3.73 3.0
- link 8_sec_2_right_conn: geometry collision box size=0.78 0.2 3.0; visual box size=0.78 0.2 3.0
- link 8_sec_2_right_wall: geometry collision box size=0.2 3.73 3.0; visual box size=0.2 3.73 3.0
- link 8_sec_3_left_conn: geometry collision box size=0.36 0.2 3.0; visual box size=0.36 0.2 3.0
- link 8_sec_3_left_wall: geometry collision box size=0.2 4.16 3.0; visual box size=0.2 4.16 3.0
- link 8_sec_3_right_conn: geometry collision box size=0.36 0.2 3.0; visual box size=0.36 0.2 3.0
- link 8_sec_3_right_wall: geometry collision box size=0.2 4.16 3.0; visual box size=0.2 4.16 3.0
- link 8_sec_4_left_wall: geometry collision box size=0.2 5.39 3.0; visual box size=0.2 5.39 3.0
- link 8_sec_4_right_wall: geometry collision box size=0.2 5.39 3.0; visual box size=0.2 5.39 3.0
- link base: geometry collision box size=1000 1000 0.2; visual box size=1000 1000 0.2
Joints:
- added joint joint_2_sec_5_left_conn: type fixed, parent base, child 2_sec_5_left_conn, origin xyz=0 0 0 rpy=0 0 0
- added joint joint_2_sec_5_right_conn: type fixed, parent base, child 2_sec_5_right_conn, origin xyz=0 0 0 rpy=0 0 0
- added joint joint_2_sec_6_left_conn: type fixed, parent base, child 2_sec_6_left_conn, origin xyz=0 0 0 rpy=0 0 0
- added joint joint_2_sec_6_left_wall: type fixed, parent base, child 2_sec_6_left_wall, origin xyz=0 0 0 rpy=0 0 0
- added joint joint_2_sec_6_right_conn: type fixed, parent base, child 2_sec_6_right_conn, origin xyz=0 0 0 rpy=0 0 0
- added joint joint_2_sec_6_right_wall: type fixed, parent base, child 2_sec_6_right_wall, origin xyz=0 0 0 rpy=0 0 0
- added joint joint_2_sec_7_left_wall: type fixed, parent base, child 2_sec_7_left_wall, origin xyz=0 0 0 rpy=0 0 0
- added joint joint_2_sec_7_right_wall: type fixed, parent base, child 2_sec_7_right_wall, origin xyz=0 0 0 rpy=0 0 0
- added joint joint_4_sec_5_left_conn: type fixed, parent base, child 4_sec_5_left_conn, origin xyz=0 0 0 rpy=0 0 0
- added joint joint_4_sec_5_right_conn: type fixed, parent base, child 4_sec_5_right_conn, origin xyz=0 0 0 rpy=0 0 0
- added joint joint_4_sec_6_left_wall: type fixed, parent base, child 4_sec_6_left_wall, origin xyz=0 0 0 rpy=0 0 0
- added joint joint_4_sec_6_right_wall: type fixed, parent base, child 4_sec_6_right_wall, origin xyz=0 0 0 rpy=0 0 0
- added joint joint_6_sec_10_left_conn: type fixed, parent base, child 6_sec_10_left_conn, origin xyz=0 0 0 rpy=0 0 0
- added joint joint_6_sec_10_left_wall: type fixed, parent base, child 6_sec_10_left_wall, origin xyz=0 0 0 rpy=0 0 0
- added joint joint_6_sec_10_right_conn: type fixed, parent base, child 6_sec_10_right_conn, origin xyz=0 0 0 rpy=0 0 0
- added joint joint_6_sec_10_right_wall: type fixed, parent base, child 6_sec_10_right_wall, origin xyz=0 0 0 rpy=0 0 0
- added joint joint_6_sec_11_left_wall: type fixed, parent base, child 6_sec_11_left_wall, origin xyz=0 0 0 rpy=0 0 0
- added joint joint_6_sec_11_right_wall: type fixed, parent base, child 6_sec_11_right_wall, origin xyz=0 0 0 rpy=0 0 0
- added joint joint_6_sec_6_left_conn: type fixed, parent base, child 6_sec_6_left_conn, origin xyz=0 0 0 rpy=0 0 0
- added joint joint_6_sec_6_right_conn: type fixed, parent base, child 6_sec_6_right_conn, origin xyz=0 0 0 rpy=0 0 0
- added joint joint_6_sec_7_left_conn: type fixed, parent base, child 6_sec_7_left_conn, origin xyz=0 0 0 rpy=0 0 0
- added joint joint_6_sec_7_left_wall: type fixed, parent base, child 6_sec_7_left_wall, origin xyz=0 0 0 rpy=0 0 0
- added joint joint_6_sec_7_right_conn: type fixed, parent base, child 6_sec_7_right_conn, origin xyz=0 0 0 rpy=0 0 0
- added joint joint_6_sec_7_right_wall: type fixed, parent base, child 6_sec_7_right_wall, origin xyz=0 0 0 rpy=0 0 0
- added joint joint_6_sec_8_left_conn: type fixed, parent base, child 6_sec_8_left_conn, origin xyz=0 0 0 rpy=0 0 0
- added joint joint_6_sec_8_left_wall: type fixed, parent base, child 6_sec_8_left_wall, origin xyz=0 0 0 rpy=0 0 0
- added joint joint_6_sec_8_right_conn: type fixed, parent base, child 6_sec_8_right_conn, origin xyz=0 0 0 rpy=0 0 0
- added joint joint_6_sec_8_right_wall: type fixed, parent base, child 6_sec_8_right_wall, origin xyz=0 0 0 rpy=0 0 0
- added joint joint_6_sec_9_left_conn: type fixed, parent base, child 6_sec_9_left_conn, origin xyz=0 0 0 rpy=0 0 0
- added joint joint_6_sec_9_left_wall: type fixed, parent base, child 6_sec_9_left_wall, origin xyz=0 0 0 rpy=0 0 0
- added joint joint_6_sec_9_right_conn: type fixed, parent base, child 6_sec_9_right_conn, origin xyz=0 0 0 rpy=0 0 0
- added joint joint_6_sec_9_right_wall: type fixed, parent base, child 6_sec_9_right_wall, origin xyz=0 0 0 rpy=0 0 0
- added joint joint_8_sec_4_left_conn: type fixed, parent base, child 8_sec_4_left_conn, origin xyz=0 0 0 rpy=0 0 0
- added joint joint_8_sec_4_right_conn: type fixed, parent base, child 8_sec_4_right_conn, origin xyz=0 0 0 rpy=0 0 0
- added joint joint_8_sec_5_left_wall: type fixed, parent base, child 8_sec_5_left_wall, origin xyz=0 0 0 rpy=0 0 0
- added joint joint_8_sec_5_right_wall: type fixed, parent base, child 8_sec_5_right_wall, origin xyz=0 0 0 rpy=0 0 0
