Commit message: second round of simulations

File: urdf/random_hall.urdf (robot description, URDF)
Before this commit: robot hallway, 132 links, 131 joints
Links:
- removed link 6_sec_10_left_conn
- removed link 6_sec_10_left_wall
- removed link 6_sec_10_right_conn
- removed link 6_sec_10_right_wall
- removed link 6_sec_11_left_wall
- removed link 6_sec_11_right_wall
- removed link 6_sec_9_left_conn
- removed link 6_sec_9_right_conn
- removed link 8_sec_4_left_conn
- removed link 8_sec_4_right_conn
- removed link 8_sec_5_left_wall
- removed link 8_sec_5_right_wall
- added link 2_sec_10_left_wall; collision box size=4.0 0.2 3.0; visual box size=4.0 0.2 3.0
- added link 2_sec_10_right_wall; collision box size=4.0 0.2 3.0; visual box size=4.0 0.2 3.0
- added link 2_sec_7_left_conn; collision box size=0.2 0.38 3.0; visual box size=0.2 0.38 3.0
- added link 2_sec_7_right_conn; collision box size=0.2 0.38 3.0; visual box size=0.2 0.38 3.0
- added link 2_sec_8_left_conn; collision box size=0.2 0.445 3.0; visual box size=0.2 0.445 3.0
- added link 2_sec_8_left_wall; collision box size=4.45 0.2 3.0; visual box size=4.45 0.2 3.0
- added link 2_sec_8_right_conn; collision box size=0.2 0.445 3.0; visual box size=0.2 0.445 3.0
- added link 2_sec_8_right_wall; collision box size=4.45 0.2 3.0; visual box size=4.45 0.2 3.0
- added link 2_sec_9_left_conn; collision box size=0.2 0.645 3.0; visual box size=0.2 0.645 3.0
- added link 2_sec_9_left_wall; collision box size=5.11 0.2 3.0; visual box size=5.11 0.2 3.0
- added link 2_sec_9_right_conn; collision box size=0.2 0.645 3.0; visual box size=0.2 0.645 3.0
- added link 2_sec_9_right_wall; collision box size=5.11 0.2 3.0; visual box size=5.11 0.2 3.0
- link 1_int_side_0: geometry collision box size=0.2 3.9 3.0; visual box size=0.2 3.9 3.0
- link 1_int_side_1: geometry collision box size=3.9 0.2 3.0; visual box size=3.9 0.2 3.0
- link 1_int_side_2_left: geometry collision box size=0.2 0.7 3.0; visual box size=0.2 0.7 3.0
- link 1_int_side_2_right: geometry collision box size=0.2 0.7 3.0; visual box size=0.2 0.7 3.0
- link 1_int_side_3: geometry collision box size=3.9 0.2 3.0; visual box size=3.9 0.2 3.0
- link 2_sec_1_left_conn: geometry collision box size=0.2 0.46 3.0; visual box size=0.2 0.46 3.0
- link 2_sec_1_right_conn: geometry collision box size=0.2 0.46 3.0; visual box size=0.2 0.46 3.0
- link 2_sec_2_left_conn: geometry collision box size=0.2 0.34 3.0; visual box size=0.2 0.34 3.0
- link 2_sec_2_left_wall: geometry collision box size=2.65 0.2 3.0; visual box size=2.65 0.2 3.0
- link 2_sec_2_right_conn: geometry collision box size=0.2 0.34 3.0; visual box size=0.2 0.34 3.0
- link 2_sec_2_right_wall: geometry collision box size=2.65 0.2 3.0; visual box size=2.65 0.2 3.0
- link 2_sec_3_left_conn: geometry collision box size=0.2 0.295 3.0; visual box size=0.2 0.295 3.0
- link 2_sec_3_left_wall: geometry collision box size=4.76 0.2 3.0; visual box size=4.76 0.2 3.0
- link 2_sec_3_right_conn: geometry collision box size=0.2 0.295 3.0; visual box size=0.2 0.295 3.0
- link 2_sec_3_right_wall: geometry collision box size=4.76 0.2 3.0; visual box size=4.76 0.2 3.0
- link 2_sec_4_left_conn: geometry collision box size=0.2 0.27 3.0; visual box size=0.2 0.27 3.0
- link 2_sec_4_left_wall: geometry collision box size=4.62 0.2 3.0; visual box size=4.62 0.2 3.0
- link 2_sec_4_right_conn: geometry collision box size=0.2 0.27 3.0; visual box size=0.2 0.27 3.0
- link 2_sec_4_right_wall: geometry collision box size=4.62 0.2 3.0; visual box size=4.62 0.2 3.0
- link 2_sec_5_left_conn: geometry collision box size=0.2 0.415 3.0; visual box size=0.2 0.415 3.0
- link 2_sec_5_left_wall: geometry collision box size=3.36 0.2 3.0; visual box size=3.36 0.2 3.0
- link 2_sec_5_right_conn: geometry collision box size=0.2 0.415 3.0; visual box size=0.2 0.415 3.0
- link 2_sec_5_right_wall: geometry collision box size=3.36 0.2 3.0; visual box size=3.36 0.2 3.0
- link 2_sec_6_left_conn: geometry collision box size=0.2 0.32 3.0; visual box size=0.2 0.32 3.0
- link 2_sec_6_left_wall: geometry collision box size=3.77 0.2 3.0; visual box size=3.77 0.2 3.0
- link 2_sec_6_right_conn: geometry collision box size=0.2 0.32 3.0; visual box size=0.2 0.32 3.0
- link 2_sec_6_right_wall: geometry collision box size=3.77 0.2 3.0; visual box size=3.77 0.2 3.0
- link 2_sec_7_left_wall: geometry collision box size=3.49 0.2 3.0; visual box size=3.49 0.2 3.0
- link 2_sec_7_right_wall: geometry collision box size=3.49 0.2 3.0; visual box size=3.49 0.2 3.0
- link 3_int_side_0_left: geometry collision box size=0.2 0.7 3.0; visual box size=0.2 0.7 3.0
- link 3_int_side_0_right: geometry collision box size=0.2 0.7 3.0; visual box size=0.2 0.7 3.0
- link 3_int_side_1_left: geometry collision box size=0.7 0.2 3.0; visual box size=0.7 0.2 3.0
- link 3_int_side_1_right: geometry collision box size=0.7 0.2 3.0; visual box size=0.7 0.2 3.0
- link 3_int_side_2: geometry collision box size=0.2 3.9 3.0; visual box size=0.2 3.9 3.0
- link 3_int_side_3: geometry collision box size=3.9 0.2 3.0; visual box size=3.9 0.2 3.0
- link 4_sec_1_left_conn: geometry collision box size=0.39 0.2 3.0; visual box size=0.39 0.2 3.0
- link 4_sec_1_right_conn: geometry collision box size=0.39 0.2 3.0; visual box size=0.39 0.2 3.0
- link 4_sec_2_left_conn: geometry collision box size=0.64 0.2 3.0; visual box size=0.64 0.2 3.0
- link 4_sec_2_left_wall: geometry collision box size=0.2 1.75 3.0; visual box size=0.2 1.75 3.0
- link 4_sec_2_right_conn: geometry collision box size=0.64 0.2 3.0; visual box size=0.64 0.2 3.0
- link 4_sec_2_right_wall: geometry collision box size=0.2 1.75 3.0; visual box size=0.2 1.75 3.0
- link 4_sec_3_left_conn: geometry collision box size=0.21 0.2 3.0; visual box size=0.21 0.2 3.0
- link 4_sec_3_left_wall: geometry collision box size=0.2 4.03 3.0; visual box size=0.2 4.03 3.0
- link 4_sec_3_right_conn: geometry collision box size=0.21 0.2 3.0; visual box size=0.21 0.2 3.0
- link 4_sec_3_right_wall: geometry collision box size=0.2 4.03 3.0; visual box size=0.2 4.03 3.0
- link 4_sec_4_left_conn: geometry collision box size=0.72 0.2 3.0; visual box size=0.72 0.2 3.0
- link 4_sec_4_left_wall: geometry collision box size=0.2 3.62 3.0; visual box size=0.2 3.62 3.0
- link 4_sec_4_right_conn: geometry collision box size=0.72 0.2 3.0; visual box size=0.72 0.2 3.0
- link 4_sec_4_right_wall: geometry collision box size=0.2 3.62 3.0; visual box size=0.2 3.62 3.0
- link 4_sec_5_left_conn: geometry collision box size=0.46 0.2 3.0; visual box size=0.46 0.2 3.0
- link 4_sec_5_left_wall: geometry collision box size=0.2 5.12 3.0; visual box size=0.2 5.12 3.0
- link 4_sec_5_right_conn: geometry collision box size=0.46 0.2 3.0; visual box size=0.46 0.2 3.0
- link 4_sec_5_right_wall: geometry collision box size=0.2 5.12 3.0; visual box size=0.2 5.12 3.0
- link 5_int_side_0_left: geometry collision box size=0.2 0.7 3.0; visual box size=0.2 0.7 3.0
- link 5_int_side_0_right: geometry collision box size=0.2 0.7 3.0; visual box size=0.2 0.7 3.0
- link 5_int_side_1: geometry collision box size=3.9 0.2 3.0; visual box size=3.9 0.2 3.0
- link 5_int_side_2: geometry collision box size=0.2 3.9 3.0; visual box size=0.2 3.9 3.0
- link 5_int_side_3_left: geometry collision box size=0.7 0.2 3.0; visual box size=0.7 0.2 3.0
- link 5_int_side_3_right: geometry collision box size=0.7 0.2 3.0; visual box size=0.7 0.2 3.0
- link 6_sec_1_left_conn: geometry collision box size=-0.2 -0.615 3.0; visual box size=-0.2 -0.615 3.0
- link 6_sec_1_right_conn: geometry collision box size=-0.2 -0.615 3.0; visual box size=-0.2 -0.615 3.0
- link 6_sec_2_left_conn: geometry collision box size=-0.2 -0.73 3.0; visual box size=-0.2 -0.73 3.0
- link 6_sec_2_left_wall: geometry collision box size=-5.03 -0.2 3.0; visual box size=-5.03 -0.2 3.0
- link 6_sec_2_right_conn: geometry collision box size=-0.2 -0.73 3.0; visual box size=-0.2 -0.73 3.0
- link 6_sec_2_right_wall: geometry collision box size=-5.03 -0.2 3.0; visual box size=-5.03 -0.2 3.0
- link 6_sec_3_left_conn: geometry collision box size=-0.2 -0.71 3.0; visual box size=-0.2 -0.71 3.0
- link 6_sec_3_left_wall: geometry collision box size=-6.15 -0.2 3.0; visual box size=-6.15 -0.2 3.0
- link 6_sec_3_right_conn: geometry collision box size=-0.2 -0.71 3.0; visual box size=-0.2 -0.71 3.0
- link 6_sec_3_right_wall: geometry collision box size=-6.15 -0.2 3.0; visual box size=-6.15 -0.2 3.0
- link 6_sec_4_left_conn: geometry collision box size=-0.2 -0.615 3.0; visual box size=-0.2 -0.615 3.0
- link 6_sec_4_left_wall: geometry collision box size=-3.41 -0.2 3.0; visual box size=-3.41 -0.2 3.0
- link 6_sec_4_right_conn: geometry collision box size=-0.2 -0.615 3.0; visual box size=-0.2 -0.615 3.0
- link 6_sec_4_right_wall: geometry collision box size=-3.41 -0.2 3.0; visual box size=-3.41 -0.2 3.0
- link 6_sec_5_left_conn: geometry collision box size=-0.2 -0.645 3.0; visual box size=-0.2 -0.645 3.0
- link 6_sec_5_left_wall: geometry collision box size=-4.95 -0.2 3.0; visual box size=-4.95 -0.2 3.0
- link 6_sec_5_right_conn: geometry collision box size=-0.2 -0.645 3.0; visual box size=-0.2 -0.645 3.0
- link 6_sec_5_right_wall: geometry collision box size=-4.95 -0.2 3.0; visual box size=-4.95 -0.2 3.0
- link 6_sec_6_left_conn: geometry collision box size=-0.2 -0.275 3.0; visual box size=-0.2 -0.275 3.0
- link 6_sec_6_left_wall: geometry collision box size=-4.26 -0.2 3.0; visual box size=-4.26 -0.2 3.0
- link 6_sec_6_right_conn: geometry collision box size=-0.2 -0.275 3.0; visual box size=-0.2 -0.275 3.0
- link 6_sec_6_right_wall: geometry collision box size=-4.26 -0.2 3.0; visual box size=-4.26 -0.2 3.0
- link 6_sec_7_left_conn: geometry collision box size=-0.2 -0.86 3.0; visual box size=-0.2 -0.86 3.0
- link 6_sec_7_left_wall: geometry collision box size=-3.95 -0.2 3.0; visual box size=-3.95 -0.2 3.0
- link 6_sec_7_right_conn: geometry collision box size=-0.2 -0.86 3.0; visual box size=-0.2 -0.86 3.0
- link 6_sec_7_right_wall: geometry collision box size=-3.95 -0.2 3.0; visual box size=-3.95 -0.2 3.0
- link 6_sec_8_left_conn: geometry collision box size=-0.2 -0.36 3.0; visual box size=-0.2 -0.36 3.0
- link 6_sec_8_left_wall: geometry collision box size=-4.58 -0.2 3.0; visual box size=-4.58 -0.2 3.0
- link 6_sec_8_right_conn: geometry collision box size=-0.2 -0.36 3.0; visual box size=-0.2 -0.36 3.0
- link 6_sec_8_right_wall: geometry collision box size=-4.58 -0.2 3.0; visual box size=-4.58 -0.2 3.0
- link 6_sec_9_left_wall: geometry collision box size=-4.0 -0.2 3.0; visual box size=-4.0 -0.2 3.0
- link 6_sec_9_right_wall: geometry collision box size=-4.0 -0.2 3.0; visual box size=-4.0 -0.2 3.0
- link 7_int_side_0: geometry collision box size=0.2 3.9 3.0; visual box size=0.2 3.9 3.0
- link 7_int_side_1_left: geometry collision box size=0.7 0.2 3.0; visual box size=0.7 0.2 3.0
- link 7_int_side_1_right: geometry collision box size=0.7 0.2 3.0; visual box size=0.7 0.2 3.0
- link 7_int_side_2_left: geometry collision box size=0.2 0.7 3.0; visual box size=0.2 0.7 3.0
- link 7_int_side_2_right: geometry collision box size=0.2 0.7 3.0; visual box size=0.2 0.7 3.0
- link 7_int_side_3: geometry collision box size=3.9 0.2 3.0; visual box size=3.9 0.2 3.0
- link 8_sec_1_left_conn: geometry collision box size=0.505 0.2 3.0; visual box size=0.505 0.2 3.0
- link 8_sec_1_right_conn: geometry collision box size=0.505 0.2 3.0; visual box size=0.505 0.2 3.0
- link 8_sec_2_left_conn: geometry collision box size=0.495 0.2 3.0; visual box size=0.495 0.2 3.0
- link 8_sec_2_left_wall: geometry collision box size=0.2 3.42 3.0; visual box size=0.2 3.42 3.0
- link 8_sec_2_right_conn: geometry collision box size=0.495 0.2 3.0; visual box size=0.495 0.2 3.0
- link 8_sec_2_right_wall: geometry collision box size=0.2 3.42 3.0; visual box size=0.2 3.42 3.0
- link 8_sec_3_left_conn: geometry collision box size=0.21 0.2 3.0; visual box size=0.21 0.2 3.0
- link 8_sec_3_left_wall: geometry collision box size=0.2 4.53 3.0; visual box size=0.2 4.53 3.0
- link 8_sec_3_right_conn: geometry collision box size=0.21 0.2 3.0; visual box size=0.21 0.2 3.0
- link 8_sec_3_right_wall: geometry collision box size=0.2 4.53 3.0; visual box size=0.2 4.53 3.0
- link 8_sec_4_left_wall: geometry collision box size=0.2 4.0 3.0; visual box size=0.2 4.0 3.0
- link 8_sec_4_right_wall: geometry collision box size=0.2 4.0 3.0; visual box size=0.2 4.0 3.0
Joints:
- removed joint joint_6_sec_10_left_conn
- removed joint joint_6_sec_10_left_wall
- removed joint joint_6_sec_10_right_conn
- removed joint joint_6_sec_10_right_wall
- removed joint joint_6_sec_11_left_wall
- removed joint joint_6_sec_11_right_wall
- removed joint joint_6_sec_9_left_conn
- removed joint joint_6_sec_9_right_conn
- removed joint joint_8_sec_4_left_conn
- removed joint joint_8_sec_4_right_conn
- removed joint joint_8_sec_5_left_wall
- removed joint joint_8_sec_5_right_wall
- added joint joint_2_sec_10_left_wall: type fixed, parent base, child 2_sec_10_left_wall, origin xyz=0 0 0 rpy=0 0 0
- added joint joint_2_sec_10_right_wall: type fixed, parent base, child 2_sec_10_right_wall, origin xyz=0 0 0 rpy=0 0 0
- added joint joint_2_sec_7_left_conn: type fixed, parent base, child 2_sec_7_left_conn, origin xyz=0 0 0 rpy=0 0 0
- added joint joint_2_sec_7_right_conn: type fixed, parent base, child 2_sec_7_right_conn, origin xyz=0 0 0 rpy=0 0 0
- added joint joint_2_sec_8_left_conn: type fixed, parent base, child 2_sec_8_left_conn, origin xyz=0 0 0 rpy=0 0 0
- added joint joint_2_sec_8_left_wall: type fixed, parent base, child 2_sec_8_left_wall, origin xyz=0 0 0 rpy=0 0 0
- added joint joint_2_sec_8_right_conn: type fixed, parent base, child 2_sec_8_right_conn, origin xyz=0 0 0 rpy=0 0 0
- added joint joint_2_sec_8_right_wall: type fixed, parent base, child 2_sec_8_right_wall, origin xyz=0 0 0 rpy=0 0 0
- added joint joint_2_sec_9_left_conn: type fixed, parent base, child 2_sec_9_left_conn, origin xyz=0 0 0 rpy=0 0 0
- added joint joint_2_sec_9_left_wall: type fixed, parent base, child 2_sec_9_left_wall, origin xyz=0 0 0 rpy=0 0 0
- added joint joint_2_sec_9_right_conn: type fixed, parent base, child 2_sec_9_right_conn, origin xyz=0 0 0 rpy=0 0 0
- added joint joint_2_sec_9_right_wall: type fixed, parent base, child 2_sec_9_right_wall, origin xyz=0 0 0 rpy=0 0 0
