Commit message: third round of simulations

File: urdf/random_hall.urdf (robot description, URDF)
Before this commit: robot hallway, 132 links, 131 joints
Links:
- removed link 2_sec_10_left_wall
- removed link 2_sec_10_right_wall
- removed link 2_sec_5_left_conn
- removed link 2_sec_5_right_conn
- removed link 2_sec_6_left_conn
- removed link 2_sec_6_left_wall
- removed link 2_sec_6_right_conn
- removed link 2_sec_6_right_wall
- removed link 2_sec_7_left_conn
- removed link 2_sec_7_left_wall
- removed link 2_sec_7_right_conn
- removed link 2_sec_7_right_wall
- removed link 2_sec_8_left_conn
- removed link 2_sec_8_left_wall
- removed link 2_sec_8_right_conn
- removed link 2_sec_8_right_wall
- removed link 2_sec_9_left_conn
- removed link 2_sec_9_left_wall
- removed link 2_sec_9_right_conn
- removed link 2_sec_9_right_wall
- removed link 4_sec_5_left_conn
- removed link 4_sec_5_right_conn
- removed link 4_sec_6_left_wall
- removed link 4_sec_6_right_wall
- removed link 6_sec_8_left_conn
- removed link 6_sec_8_right_conn
- removed link 6_sec_9_left_wall
- removed link 6_sec_9_right_wall
- removed link 8_sec_3_left_conn
- removed link 8_sec_3_right_conn
- removed link 8_sec_4_left_wall
- removed link 8_sec_4_right_wall
- link 2_sec_1_left_conn: geometry collision box size=0.2 0.205 3.0; visual box size=0.2 0.205 3.0
- link 2_sec_1_right_conn: geometry collision box size=0.2 0.205 3.0; visual box size=0.2 0.205 3.0
- link 2_sec_2_left_conn: geometry collision box size=0.2 0.295 3.0; visual box size=0.2 0.295 3.0
- link 2_sec_2_left_wall: geometry collision box size=3.1 0.2 3.0; visual box size=3.1 0.2 3.0
- link 2_sec_2_right_conn: geometry collision box size=0.2 0.295 3.0; visual box size=0.2 0.295 3.0
- link 2_sec_2_right_wall: geometry collision box size=3.1 0.2 3.0; visual box size=3.1 0.2 3.0
- link 2_sec_3_left_conn: geometry collision box size=0.2 0.61 3.0; visual box size=0.2 0.61 3.0
- link 2_sec_3_left_wall: geometry collision box size=2.4 0.2 3.0; visual box size=2.4 0.2 3.0
- link 2_sec_3_right_conn: geometry collision box size=0.2 0.61 3.0; visual box size=0.2 0.61 3.0
- link 2_sec_3_right_wall: geometry collision box size=2.4 0.2 3.0; visual box size=2.4 0.2 3.0
- link 2_sec_4_left_conn: geometry collision box size=0.2 0.7 3.0; visual box size=0.2 0.7 3.0
- link 2_sec_4_left_wall: geometry collision box size=5.2 0.2 3.0; visual box size=5.2 0.2 3.0
- link 2_sec_4_right_conn: geometry collision box size=0.2 0.7 3.0; visual box size=0.2 0.7 3.0
- link 2_sec_4_right_wall: geometry collision box size=5.2 0.2 3.0; visual box size=5.2 0.2 3.0
- link 2_sec_5_left_wall: geometry collision box size=4.0 0.2 3.0; visual box size=4.0 0.2 3.0
- link 2_sec_5_right_wall: geometry collision box size=4.0 0.2 3.0; visual box size=4.0 0.2 3.0
- link 4_sec_1_left_conn: geometry collision box size=0.69 0.2 3.0; visual box size=0.69 0.2 3.0
- link 4_sec_1_right_conn: geometry collision box size=0.69 0.2 3.0; visual box size=0.69 0.2 3.0
- link 4_sec_2_left_conn: geometry collision box size=0.21 0.2 3.0; visual box size=0.21 0.2 3.0
- link 4_sec_2_left_wall: geometry collision box size=0.2 4.12 3.0; visual box size=0.2 4.12 3.0
- link 4_sec_2_right_conn: geometry collision box size=0.21 0.2 3.0; visual box size=0.21 0.2 3.0
- link 4_sec_2_right_wall: geometry collision box size=0.2 4.12 3.0; visual box size=0.2 4.12 3.0
- link 4_sec_3_left_conn: geometry collision box size=0.405 0.2 3.0; visual box size=0.405 0.2 3.0
- link 4_sec_3_left_wall: geometry collision box size=0.2 3.99 3.0; visual box size=0.2 3.99 3.0
- link 4_sec_3_right_conn: geometry collision box size=0.405 0.2 3.0; visual box size=0.405 0.2 3.0
- link 4_sec_3_right_wall: geometry collision box size=0.2 3.99 3.0; visual box size=0.2 3.99 3.0
- link 4_sec_4_left_conn: geometry collision box size=0.495 0.2 3.0; visual box size=0.495 0.2 3.0
- link 4_sec_4_left_wall: geometry collision box size=0.2 4.25 3.0; visual box size=0.2 4.25 3.0
- link 4_sec_4_right_conn: geometry collision box size=0.495 0.2 3.0; visual box size=0.495 0.2 3.0
- link 4_sec_4_right_wall: geometry collision box size=0.2 4.25 3.0; visual box size=0.2 4.25 3.0
- link 4_sec_5_left_wall: geometry collision box size=0.2 4.0 3.0; visual box size=0.2 4.0 3.0
- link 4_sec_5_right_wall: geometry collision box size=0.2 4.0 3.0; visual box size=0.2 4.0 3.0
- link 6_sec_1_left_conn: geometry collision box size=-0.2 -0.7 3.0; visual box size=-0.2 -0.7 3.0
- link 6_sec_1_right_conn: geometry collision box size=-0.2 -0.7 3.0; visual box size=-0.2 -0.7 3.0
- link 6_sec_2_left_conn: geometry collision box size=-0.2 -0.545 3.0; visual box size=-0.2 -0.545 3.0
- link 6_sec_2_left_wall: geometry collision box size=-4.72 -0.2 3.0; visual box size=-4.72 -0.2 3.0
- link 6_sec_2_right_conn: geometry collision box size=-0.2 -0.545 3.0; visual box size=-0.2 -0.545 3.0
- link 6_sec_2_right_wall: geometry collision box size=-4.72 -0.2 3.0; visual box size=-4.72 -0.2 3.0
- link 6_sec_3_left_conn: geometry collision box size=-0.2 -0.23 3.0; visual box size=-0.2 -0.23 3.0
- link 6_sec_3_left_wall: geometry collision box size=-5.6 -0.2 3.0; visual box size=-5.6 -0.2 3.0
- link 6_sec_3_right_conn: geometry collision box size=-0.2 -0.23 3.0; visual box size=-0.2 -0.23 3.0
- link 6_sec_3_right_wall: geometry collision box size=-5.6 -0.2 3.0; visual box size=-5.6 -0.2 3.0
- link 6_sec_4_left_conn: geometry collision box size=-0.2 -0.39 3.0; visual box size=-0.2 -0.39 3.0
- link 6_sec_4_left_wall: geometry collision box size=-3.37 -0.2 3.0; visual box size=-3.37 -0.2 3.0
- link 6_sec_4_right_conn: geometry collision box size=-0.2 -0.39 3.0; visual box size=-0.2 -0.39 3.0
- link 6_sec_4_right_wall: geometry collision box size=-3.37 -0.2 3.0; visual box size=-3.37 -0.2 3.0
- link 6_sec_5_left_conn: geometry collision box size=-0.2 -0.67 3.0; visual box size=-0.2 -0.67 3.0
- link 6_sec_5_left_wall: geometry collision box size=-2.25 -0.2 3.0; visual box size=-2.25 -0.2 3.0
- link 6_sec_5_right_conn: geometry collision box size=-0.2 -0.67 3.0; visual box size=-0.2 -0.67 3.0
- link 6_sec_5_right_wall: geometry collision box size=-2.25 -0.2 3.0; visual box size=-2.25 -0.2 3.0
- link 6_sec_6_left_conn: geometry collision box size=-0.2 -0.41 3.0; visual box size=-0.2 -0.41 3.0
- link 6_sec_6_left_wall: geometry collision box size=-2.52 -0.2 3.0; visual box size=-2.52 -0.2 3.0
- link 6_sec_6_right_conn: geometry collision box size=-0.2 -0.41 3.0; visual box size=-0.2 -0.41 3.0
- link 6_sec_6_right_wall: geometry collision box size=-2.52 -0.2 3.0; visual box size=-2.52 -0.2 3.0
- link 6_sec_7_left_conn: geometry collision box size=-0.2 -0.395 3.0; visual box size=-0.2 -0.395 3.0
- link 6_sec_7_left_wall: geometry collision box size=-2.91 -0.2 3.0; visual box size=-2.91 -0.2 3.0
- link 6_sec_7_right_conn: geometry collision box size=-0.2 -0.395 3.0; visual box size=-0.2 -0.395 3.0
- link 6_sec_7_right_wall: geometry collision box size=-2.91 -0.2 3.0; visual box size=-2.91 -0.2 3.0
- link 6_sec_8_left_wall: geometry collision box size=-4.0 -0.2 3.0; visual box size=-4.0 -0.2 3.0
- link 6_sec_8_right_wall: geometry collision box size=-4.0 -0.2 3.0; visual box size=-4.0 -0.2 3.0
- link 8_sec_1_left_conn: geometry collision box size=0.37 0.2 3.0; visual box size=0.37 0.2 3.0
- link 8_sec_1_right_conn: geometry collision box size=0.37 0.2 3.0; visual box size=0.37 0.2 3.0
- link 8_sec_2_left_conn: geometry collision box size=0.37 0.2 3.0; visual box size=0.37 0.2 3.0
- link 8_sec_2_left_wall: geometry collision box size=0.2 3.77 3.0; visual box size=0.2 3.77 3.0
- link 8_sec_2_right_conn: geometry collision box size=0.37 0.2 3.0; visual box size=0.37 0.2 3.0
- link 8_sec_2_right_wall: geometry collision box size=0.2 3.77 3.0; visual box size=0.2 3.77 3.0
- link 8_sec_3_left_wall: geometry collision box size=0.2 4.0 3.0; visual box size=0.2 4.0 3.0
- link 8_sec_3_right_wall: geometry collision box size=0.2 4.0 3.0; visual box size=0.2 4.0 3.0
Joints:
- removed joint joint_2_sec_10_left_wall
- removed joint joint_2_sec_10_right_wall
- removed joint joint_2_sec_5_left_conn
- removed joint joint_2_sec_5_right_conn
- removed joint joint_2_sec_6_left_conn
- removed joint joint_2_sec_6_left_wall
- removed joint joint_2_sec_6_right_conn
- removed joint joint_2_sec_6_right_wall
- removed joint joint_2_sec_7_left_conn
- removed joint joint_2_sec_7_left_wall
- removed joint joint_2_sec_7_right_conn
- removed joint joint_2_sec_7_right_wall
- removed joint joint_2_sec_8_left_conn
- removed joint joint_2_sec_8_left_wall
- removed joint joint_2_sec_8_right_conn
- removed joint joint_2_sec_8_right_wall
- removed joint joint_2_sec_9_left_conn
- removed joint joint_2_sec_9_left_wall
- removed joint joint_2_sec_9_right_conn
- removed joint joint_2_sec_9_right_wall
- removed joint joint_4_sec_5_left_conn
- removed joint joint_4_sec_5_right_conn
- removed joint joint_4_sec_6_left_wall
- removed joint joint_4_sec_6_right_wall
- removed joint joint_6_sec_8_left_conn
- removed joint joint_6_sec_8_right_conn
- removed joint joint_6_sec_9_left_wall
- removed joint joint_6_sec_9_right_wall
- removed joint joint_8_sec_3_left_conn
- removed joint joint_8_sec_3_right_conn
- removed joint joint_8_sec_4_left_wall
- removed joint joint_8_sec_4_right_wall

Commit message: ran simulation for presentation

File: urdf/random_hall.urdf (robot description, URDF)
Before this commit: robot hallway, 100 links, 99 joints
Links:
- added link 2_sec_10_left_wall; collision box size=4.0 0.2 3.0; visual box size=4.0 0.2 3.0
- added link 2_sec_10_right_wall; collision box size=4.0 0.2 3.0; visual box size=4.0 0.2 3.0
- added link 2_sec_5_left_conn; collision box size=0.2 0.57 3.0; visual box size=0.2 0.57 3.0
- added link 2_sec_5_right_conn; collision box size=0.2 0.57 3.0; visual box size=0.2 0.57 3.0
- added link 2_sec_6_left_conn; collision box size=0.2 0.535 3.0; visual box size=0.2 0.535 3.0
- added link 2_sec_6_left_wall; collision box size=3.18 0.2 3.0; visual box size=3.18 0.2 3.0
- added link 2_sec_6_right_conn; collision box size=0.2 0.535 3.0; visual box size=0.2 0.535 3.0
- added link 2_sec_6_right_wall; collision box size=3.18 0.2 3.0; visual box size=3.18 0.2 3.0
- added link 2_sec_7_left_conn; collision box size=0.2 0.465 3.0; visual box size=0.2 0.465 3.0
- added link 2_sec_7_left_wall; collision box size=5.61 0.2 3.0; visual box size=5.61 0.2 3.0
- added link 2_sec_7_right_conn; collision box size=0.2 0.465 3.0; visual box size=0.2 0.465 3.0
- added link 2_sec_7_right_wall; collision box size=5.61 0.2 3.0; visual box size=5.61 0.2 3.0
- added link 2_sec_8_left_conn; collision box size=0.2 0.405 3.0; visual box size=0.2 0.405 3.0
- added link 2_sec_8_left_wall; collision box size=5.36 0.2 3.0; visual box size=5.36 0.2 3.0
- added link 2_sec_8_right_conn; collision box size=0.2 0.405 3.0; visual box size=0.2 0.405 3.0
- added link 2_sec_8_right_wall; collision box size=5.36 0.2 3.0; visual box size=5.36 0.2 3.0
- added link 2_sec_9_left_conn; collision box size=0.2 0.425 3.0; visual box size=0.2 0.425 3.0
- added link 2_sec_9_left_wall; collision box size=3.16 0.2 3.0; visual box size=3.16 0.2 3.0
- added link 2_sec_9_right_conn; collision box size=0.2 0.425 3.0; visual box size=0.2 0.425 3.0
- added link 2_sec_9_right_wall; collision box size=3.16 0.2 3.0; visual box size=3.16 0.2 3.0
- added link 4_sec_5_left_conn; collision box size=0.495 0.2 3.0; visual box size=0.495 0.2 3.0
- added link 4_sec_5_right_conn; collision box size=0.495 0.2 3.0; visual box size=0.495 0.2 3.0
- added link 4_sec_6_left_wall; collision box size=0.2 4.0 3.0; visual box size=0.2 4.0 3.0
- added link 4_sec_6_right_wall; collision box size=0.2 4.0 3.0; visual box size=0.2 4.0 3.0
- link 2_sec_1_left_conn: geometry collision box size=0.2 0.53 3.0; visual box size=0.2 0.53 3.0
- link 2_sec_1_right_conn: geometry collision box size=0.2 0.53 3.0; visual box size=0.2 0.53 3.0
- link 2_sec_2_left_conn: geometry collision box size=0.2 0.37 3.0; visual box size=0.2 0.37 3.0
- link 2_sec_2_left_wall: geometry collision box size=5.09 0.2 3.0; visual box size=5.09 0.2 3.0
- link 2_sec_2_right_conn: geometry collision box size=0.2 0.37 3.0; visual box size=0.2 0.37 3.0
- link 2_sec_2_right_wall: geometry collision box size=5.09 0.2 3.0; visual box size=5.09 0.2 3.0
- link 2_sec_3_left_conn: geometry collision box size=0.2 0.29 3.0; visual box size=0.2 0.29 3.0
- link 2_sec_3_left_wall: geometry collision box size=4.33 0.2 3.0; visual box size=4.33 0.2 3.0
- link 2_sec_3_right_conn: geometry collision box size=0.2 0.29 3.0; visual box size=0.2 0.29 3.0
- link 2_sec_3_right_wall: geometry collision box size=4.33 0.2 3.0; visual box size=4.33 0.2 3.0
- link 2_sec_4_left_conn: geometry collision box size=0.2 0.48 3.0; visual box size=0.2 0.48 3.0
- link 2_sec_4_left_wall: geometry collision box size=3.99 0.2 3.0; visual box size=3.99 0.2 3.0
- link 2_sec_4_right_conn: geometry collision box size=0.2 0.48 3.0; visual box size=0.2 0.48 3.0
- link 2_sec_4_right_wall: geometry collision box size=3.99 0.2 3.0; visual box size=3.99 0.2 3.0
- link 2_sec_5_left_wall: geometry collision box size=4.05 0.2 3.0; visual box size=4.05 0.2 3.0
- link 2_sec_5_right_wall: geometry collision box size=4.05 0.2 3.0; visual box size=4.05 0.2 3.0
- link 4_sec_1_left_conn: geometry collision box size=0.7 0.2 3.0; visual box size=0.7 0.2 3.0
- link 4_sec_1_right_conn: geometry collision box size=0.7 0.2 3.0; visual box size=0.7 0.2 3.0
- link 4_sec_2_left_conn: geometry collision box size=0.46 0.2 3.0; visual box size=0.46 0.2 3.0
- link 4_sec_2_left_wall: geometry collision box size=0.2 5.06 3.0; visual box size=0.2 5.06 3.0
- link 4_sec_2_right_conn: geometry collision box size=0.46 0.2 3.0; visual box size=0.46 0.2 3.0
- link 4_sec_2_right_wall: geometry collision box size=0.2 5.06 3.0; visual box size=0.2 5.06 3.0
- link 4_sec_3_left_conn: geometry collision box size=0.26 0.2 3.0; visual box size=0.26 0.2 3.0
- link 4_sec_3_left_wall: geometry collision box size=0.2 4.19 3.0; visual box size=0.2 4.19 3.0
- link 4_sec_3_right_conn: geometry collision box size=0.26 0.2 3.0; visual box size=0.26 0.2 3.0
- link 4_sec_3_right_wall: geometry collision box size=0.2 4.19 3.0; visual box size=0.2 4.19 3.0
- link 4_sec_4_left_conn: geometry collision box size=0.315 0.2 3.0; visual box size=0.315 0.2 3.0
- link 4_sec_4_left_wall: geometry collision box size=0.2 4.57 3.0; visual box size=0.2 4.57 3.0
- link 4_sec_4_right_conn: geometry collision box size=0.315 0.2 3.0; visual box size=0.315 0.2 3.0
- link 4_sec_4_right_wall: geometry collision box size=0.2 4.57 3.0; visual box size=0.2 4.57 3.0
- link 4_sec_5_left_wall: geometry collision box size=0.2 2.59 3.0; visual box size=0.2 2.59 3.0
- link 4_sec_5_right_wall: geometry collision box size=0.2 2.59 3.0; visual box size=0.2 2.59 3.0
- link 6_sec_1_left_conn: geometry collision box size=-0.2 -0.615 3.0; visual box size=-0.2 -0.615 3.0
- link 6_sec_1_right_conn: geometry collision box size=-0.2 -0.615 3.0; visual box size=-0.2 -0.615 3.0
- link 6_sec_2_left_conn: geometry collision box size=-0.2 -0.52 3.0; visual box size=-0.2 -0.52 3.0
- link 6_sec_2_left_wall: geometry collision box size=-3.47 -0.2 3.0; visual box size=-3.47 -0.2 3.0
- link 6_sec_2_right_conn: geometry collision box size=-0.2 -0.52 3.0; visual box size=-0.2 -0.52 3.0
- link 6_sec_2_right_wall: geometry collision box size=-3.47 -0.2 3.0; visual box size=-3.47 -0.2 3.0
- link 6_sec_3_left_conn: geometry collision box size=-0.2 -0.225 3.0; visual box size=-0.2 -0.225 3.0
- link 6_sec_3_left_wall: geometry collision box size=-3.14 -0.2 3.0; visual box size=-3.14 -0.2 3.0
- link 6_sec_3_right_conn: geometry collision box size=-0.2 -0.225 3.0; visual box size=-0.2 -0.225 3.0
- link 6_sec_3_right_wall: geometry collision box size=-3.14 -0.2 3.0; visual box size=-3.14 -0.2 3.0
- link 6_sec_4_left_conn: geometry collision box size=-0.2 -0.8 3.0; visual box size=-0.2 -0.8 3.0
- link 6_sec_4_left_wall: geometry collision box size=-4.01 -0.2 3.0; visual box size=-4.01 -0.2 3.0
- link 6_sec_4_right_conn: geometry collision box size=-0.2 -0.8 3.0; visual box size=-0.2 -0.8 3.0
- link 6_sec_4_right_wall: geometry collision box size=-4.01 -0.2 3.0; visual box size=-4.01 -0.2 3.0
- link 6_sec_5_left_conn: geometry collision box size=-0.2 -0.305 3.0; visual box size=-0.2 -0.305 3.0
- link 6_sec_5_left_wall: geometry collision box size=-2.65 -0.2 3.0; visual box size=-2.65 -0.2 3.0
- link 6_sec_5_right_conn: geometry collision box size=-0.2 -0.305 3.0; visual box size=-0.2 -0.305 3.0
- link 6_sec_5_right_wall: geometry collision box size=-2.65 -0.2 3.0; visual box size=-2.65 -0.2 3.0
- link 6_sec_6_left_conn: geometry collision box size=-0.2 -0.815 3.0; visual box size=-0.2 -0.815 3.0
- link 6_sec_6_left_wall: geometry collision box size=-0.67 -0.2 3.0; visual box size=-0.67 -0.2 3.0
- link 6_sec_6_right_conn: geometry collision box size=-0.2 -0.815 3.0; visual box size=-0.2 -0.815 3.0
- link 6_sec_6_right_wall: geometry collision box size=-0.67 -0.2 3.0; visual box size=-0.67 -0.2 3.0
- link 6_sec_7_left_conn: geometry collision box size=-0.2 -0.23 3.0; visual box size=-0.2 -0.23 3.0
- link 6_sec_7_left_wall: geometry collision box size=-1.08 -0.2 3.0; visual box size=-1.08 -0.2 3.0
- link 6_sec_7_right_conn: geometry collision box size=-0.2 -0.23 3.0; visual box size=-0.2 -0.23 3.0
- link 6_sec_7_right_wall: geometry collision box size=-1.08 -0.2 3.0; visual box size=-1.08 -0.2 3.0
- link 8_sec_1_left_conn: geometry collision box size=0.41 0.2 3.0; visual box size=0.41 0.2 3.0
- link 8_sec_1_right_conn: geometry collision box size=0.41 0.2 3.0; visual box size=0.41 0.2 3.0
- link 8_sec_2_left_conn: geometry collision box size=0.41 0.2 3.0; visual box size=0.41 0.2 3.0
- link 8_sec_2_left_wall: geometry collision box size=0.2 3.12 3.0; visual box size=0.2 3.12 3.0
- link 8_sec_2_right_conn: geometry collision box size=0.41 0.2 3.0; visual box size=0.41 0.2 3.0
- link 8_sec_2_right_wall: geometry collision box size=0.2 3.12 3.0; visual box size=0.2 3.12 3.0
Joints:
- added joint joint_2_sec_10_left_wall: type fixed, parent base, child 2_sec_10_left_wall, origin xyz=0 0 0 rpy=0 0 0
- added joint joint_2_sec_10_right_wall: type fixed, parent base, child 2_sec_10_right_wall, origin xyz=0 0 0 rpy=0 0 0
- added joint joint_2_sec_5_left_conn: type fixed, parent base, child 2_sec_5_left_conn, origin xyz=0 0 0 rpy=0 0 0
- added joint joint_2_sec_5_right_conn: type fixed, parent base, child 2_sec_5_right_conn, origin xyz=0 0 0 rpy=0 0 0
- added joint joint_2_sec_6_left_conn: type fixed, parent base, child 2_sec_6_left_conn, origin xyz=0 0 0 rpy=0 0 0
- added joint joint_2_sec_6_left_wall: type fixed, parent base, child 2_sec_6_left_wall, origin xyz=0 0 0 rpy=0 0 0
- added joint joint_2_sec_6_right_conn: type fixed, parent base, child 2_sec_6_right_conn, origin xyz=0 0 0 rpy=0 0 0
- added joint joint_2_sec_6_right_wall: type fixed, parent base, child 2_sec_6_right_wall, origin xyz=0 0 0 rpy=0 0 0
- added joint joint_2_sec_7_left_conn: type fixed, parent base, child 2_sec_7_left_conn, origin xyz=0 0 0 rpy=0 0 0
- added joint joint_2_sec_7_left_wall: type fixed, parent base, child 2_sec_7_left_wall, origin xyz=0 0 0 rpy=0 0 0
- added joint joint_2_sec_7_right_conn: type fixed, parent base, child 2_sec_7_right_conn, origin xyz=0 0 0 rpy=0 0 0
- added joint joint_2_sec_7_right_wall: type fixed, parent base, child 2_sec_7_right_wall, origin xyz=0 0 0 rpy=0 0 0
- added joint joint_2_sec_8_left_conn: type fixed, parent base, child 2_sec_8_left_conn, origin xyz=0 0 0 rpy=0 0 0
- added joint joint_2_sec_8_left_wall: type fixed, parent base, child 2_sec_8_left_wall, origin xyz=0 0 0 rpy=0 0 0
- added joint joint_2_sec_8_right_conn: type fixed, parent base, child 2_sec_8_right_conn, origin xyz=0 0 0 rpy=0 0 0
- added joint joint_2_sec_8_right_wall: type fixed, parent base, child 2_sec_8_right_wall, origin xyz=0 0 0 rpy=0 0 0
- added joint joint_2_sec_9_left_conn: type fixed, parent base, child 2_sec_9_left_conn, origin xyz=0 0 0 rpy=0 0 0
- added joint joint_2_sec_9_left_wall: type fixed, parent base, child 2_sec_9_left_wall, origin xyz=0 0 0 rpy=0 0 0
- added joint joint_2_sec_9_right_conn: type fixed, parent base, child 2_sec_9_right_conn, origin xyz=0 0 0 rpy=0 0 0
- added joint joint_2_sec_9_right_wall: type fixed, parent base, child 2_sec_9_right_wall, origin xyz=0 0 0 rpy=0 0 0
- added joint joint_4_sec_5_left_conn: type fixed, parent base, child 4_sec_5_left_conn, origin xyz=0 0 0 rpy=0 0 0
- added joint joint_4_sec_5_right_conn: type fixed, parent base, child 4_sec_5_right_conn, origin xyz=0 0 0 rpy=0 0 0
- added joint joint_4_sec_6_left_wall: type fixed, parent base, child 4_sec_6_left_wall, origin xyz=0 0 0 rpy=0 0 0
- added joint joint_4_sec_6_right_wall: type fixed, parent base, child 4_sec_6_right_wall, origin xyz=0 0 0 rpy=0 0 0
